File: narra 0805design/narra 0805design.sch (KiCad schematic (older format))
At the start: 8 parts

Commit message: Added a soldering pad and protection resistors to the LED0805 design
Parts:
- added J1: P1_rows, Measurement_Points:Measurement_Point_Square-SMD-Pad_Small, symbol TEST_1P
- added J2: P2_columns, Measurement_Points:Measurement_Point_Square-SMD-Pad_Small, symbol TEST_1P
- added R1, R2, R3, R4, R5, R6, R7, R8: 37, Resistors_SMD:R_0805, symbol R
Connections:
- net Columns_anode: now also J2.1
- net Rows_cathode: now also J1.1, R1.2, R2.2, R3.2, R4.2, R5.2, R6.2, R7.2, R8.2; no longer D1.1 (K), D2.1 (K), D3.1 (K), D4.1 (K), D5.1 (K), D6.1 (K), D7.1 (K), D8.1 (K)
- new net: D1.1 (K), R1.1
- new net: D2.1 (K), R2.1
- new net: D3.1 (K), R3.1
- new net: D4.1 (K), R4.1
- new net: D5.1 (K), R5.1
- new net: D6.1 (K), R6.1
- new net: D7.1 (K), R7.1
- new net: D8.1 (K), R8.1
Changed lines of the file:
@@
 LIBS:contrib
 LIBS:valves
+LIBS:narra 0805design-cache
 EELAYER 25 0
 EELAYER END
@@
 $EndComp
 Wire Wire Line
-	2800 1600 2550 1600
-Wire Wire Line
-	2550 1300 2550 3700
-Wire Wire Line
-	2550 3700 2800 3700
-Wire Wire Line
-	2800 3400 2550 3400
-Connection ~ 2550 3400
-Wire Wire Line
-	2800 3100 2550 3100
-Connection ~ 2550 3100
-Wire Wire Line
-	2800 2800 2550 2800
-Connection ~ 2550 2800
-Wire Wire Line
-	2800 2500 2550 2500
-Connection ~ 2550 2500
-Wire Wire Line
-	2800 2200 2550 2200
-Connection ~ 2550 2200
-Wire Wire Line
-	2550 1900 2800 1900
-Connection ~ 2550 1900
-Wire Wire Line
 	3100 1600 3350 1600
 Wire Wire Line
@@
 	3100 1900 3350 1900
 Connection ~ 3350 1900
-Connection ~ 2550 1600
 Connection ~ 3350 3700
 Text Label 3700 3700 0    60   ~ 0
 Columns_anode
-Text Label 2550 1300 0    60   ~ 0
+Text Label 1800 1600 2    60   ~ 0
 Rows_cathode
+$Comp
+L TEST_1P J1
+U 1 1 58DF58BA
+P 2550 1300
+F 0 "J1" H 2550 1570 50  0000 C CNN
+F 1 "P1_rows" H 2550 1500 50  0000 C CNN
+F 2 "Measurement_Points:Measurement_Point_Square-SMD-Pad_Small" H 2750 1300 50  0001 C CNN
+F 3 "" H 2750 1300 50  0001 C CNN
+	1    2550 1300
+	1    0    0    -1
+$EndComp
+$Comp
+L TEST_1P J2
+U 1 1 58DF592F
+P 3700 3850
+F 0 "J2" H 3700 4120 50  0000 C CNN
+F 1 "P2_columns" H 3700 4050 50  0000 C CNN
+F 2 "Measurement_Points:Measurement_Point_Square-SMD-Pad_Small" H 3900 3850 50  0001 C CNN
+F 3 "" H 3900 3850 50  0001 C CNN
+	1    3700 3850
+	-1   0    0    1
+$EndComp
+$Comp
+L R R1
+U 1 1 58DF6766
+P 2200 1600
+F 0 "R1" V 2280 1600 50  0000 C CNN
+F 1 "37" V 2200 1600 50  0000 C CNN
+F 2 "Resistors_SMD:R_0805" V 2130 1600 50  0001 C CNN
+F 3 "" H 2200 1600 50  0001 C CNN
+	1    2200 1600
+	0    1    1    0
+$EndComp
+$Comp
+L R R2
+U 1 1 58DF6ACF
+P 2200 1900
+F 0 "R2" V 2280 1900 50  0000 C CNN
+F 1 "37" V 2200 1900 50  0000 C CNN
+F 2 "Resistors_SMD:R_0805" V 2130 1900 50  0001 C CNN
+F 3 "" H 2200 1900 50  0001 C CNN
+	1    2200 1900
+	0    1    1    0
+$EndComp
+$Comp
+L R R3
+U 1 1 58DF73C1
+P 2200 2200
+F 0 "R3" V 2280 2200 50  0000 C CNN
+F 1 "37" V 2200 2200 50  0000 C CNN
+F 2 "Resistors_SMD:R_0805" V 2130 2200 50  0001 C CNN
+F 3 "" H 2200 2200 50  0001 C CNN
+	1    2200 2200
+	0    1    1    0
+$EndComp
+$Comp
+L R R4
+U 1 1 58DF73C7
+P 2200 2500
+F 0 "R4" V 2280 2500 50  0000 C CNN
+F 1 "37" V 2200 2500 50  0000 C CNN
+F 2 "Resistors_SMD:R_0805" V 2130 2500 50  0001 C CNN
+F 3 "" H 2200 2500 50  0001 C CNN
+	1    2200 2500
+	0    1    1    0
+$EndComp
+$Comp
+L R R5
+U 1 1 58DF74D9
+P 2200 2800
+F 0 "R5" V 2280 2800 50  0000 C CNN
+F 1 "37" V 2200 2800 50  0000 C CNN
+F 2 "Resistors_SMD:R_0805" V 2130 2800 50  0001 C CNN
+F 3 "" H 2200 2800 50  0001 C CNN
+	1    2200 2800
+	0    1    1    0
+$EndComp
+$Comp
+L R R6
+U 1 1 58DF74DF
+P 2200 3100
+F 0 "R6" V 2280 3100 50  0000 C CNN
+F 1 "37" V 2200 3100 50  0000 C CNN
+F 2 "Resistors_SMD:R_0805" V 2130 3100 50  0001 C CNN
+F 3 "" H 2200 3100 50  0001 C CNN
+	1    2200 3100
+	0    1    1    0
+$EndComp
+$Comp
+L R R7
+U 1 1 58DF74E5
+P 2200 3400
+F 0 "R7" V 2280 3400 50  0000 C CNN
+F 1 "37" V 2200 3400 50  0000 C CNN
+F 2 "Resistors_SMD:R_0805" V 2130 3400 50  0001 C CNN
+F 3 "" H 2200 3400 50  0001 C CNN
+	1    2200 3400
+	0    1    1    0
+$EndComp
+$Comp
+L R R8
+U 1 1 58DF74EB
+P 2200 3700
+F 0 "R8" V 2280 3700 50  0000 C CNN
+F 1 "37" V 2200 3700 50  0000 C CNN
+F 2 "Resistors_SMD:R_0805" V 2130 3700 50  0001 C CNN
+F 3 "" H 2200 3700 50  0001 C CNN
+	1    2200 3700
+	0    1    1    0
+$EndComp
+Wire Wire Line
+	2350 1600 2800 1600
+Wire Wire Line
+	2350 1900 2800 1900
+Wire Wire Line
+	2350 2200 2800 2200
+Wire Wire Line
+	2350 2500 2800 2500
+Wire Wire Line
+	2350 2800 2800 2800
+Wire Wire Line
+	2350 3100 2800 3100
+Wire Wire Line
+	2350 3400 2800 3400
+Wire Wire Line
+	2350 3700 2800 3700
+Wire Wire Line
+	1800 1300 1800 3700
+Wire Wire Line
+	1800 3400 2050 3400
+Wire Wire Line
+	2050 3100 1800 3100
+Connection ~ 1800 3100
+Wire Wire Line
+	2050 2800 1800 2800
+Connection ~ 1800 2800
+Wire Wire Line
+	2050 2500 1800 2500
+Connection ~ 1800 2500
+Wire Wire Line
+	2050 2200 1800 2200
+Connection ~ 1800 2200
+Wire Wire Line
+	2050 1900 1800 1900
+Connection ~ 1800 1900
+Wire Wire Line
+	2050 1600 1800 1600
+Wire Wire Line
+	1800 1300 2550 1300
+Connection ~ 1800 1600
+Wire Wire Line
+	1800 3700 2050 3700
+Connection ~ 1800 3400
+Wire Wire Line
+	3700 3700 3700 3850
 $EndSCHEMATC

Commit message: Modified schematic and board level design ========================================= -Added gndref symbol to schematic -Expanded board edge so as to add clearance to edge from anode traces. -Connected copper fill zone to cathode connection point in order to provide a low inductance and resistance path for current. -Deleted traces to cathode connection point from the protection resistors.
Connections:
- net Rows_cathode: no longer J1.1, R1.2, R2.2, R3.2, R4.2, R5.2, R6.2, R7.2, R8.2
- new net GNDREF: J1.1, R1.2, R2.2, R3.2, R4.2, R5.2, R6.2, R7.2, R8.2
Other:
- moved on the sheet: D1, D2, D3, D4, D5, D6, D7, D8, J1, J2, R1, R2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

Commit message: Changed SMD resistor footprint to through-hole type.
Parts:
- J1: value P1_rows -> Rows
- J2: value P2_columns -> Columns
- R1, R2, R3, R4, R5, R6, R7, R8: footprint Resistors_SMD:R_0805 -> Resistors_THT:R_Axial_DIN0207_L6.3mm_D2.5mm_P7.62mm_Horizontal
Connections:
- net Columns_anode renamed C
Changed lines of the file:
@@
 LIBS:valves
 LIBS:narra 0805design-cache
-EELAYER 26 0
+EELAYER 25 0
 EELAYER END
 $Descr A4 11693 8268
@@
 $EndComp
 Text Label 6700 4850 0    60   ~ 0
-Columns_anode
+C
 Text Label 4750 2800 2    60   ~ 0
-Rows_cathode
+R
 $Comp
 L TEST_1P J1
@@
 P 5550 2450
 F 0 "J1" H 5550 2720 50  0000 C CNN
-F 1 "P1_rows" H 5550 2650 50  0000 C CNN
+F 1 "Rows" H 5550 2650 50  0000 C CNN
 F 2 "Measurement_Points:Measurement_Point_Square-SMD-Pad_Small" H 5750 2450 50  0001 C CNN
 F 3 "" H 5750 2450 50  0001 C CNN
@@
 P 6700 5000
 F 0 "J2" H 6700 5270 50  0000 C CNN
-F 1 "P2_columns" H 6700 5200 50  0000 C CNN
+F 1 "Columns" H 6700 5200 50  0000 C CNN
 F 2 "Measurement_Points:Measurement_Point_Square-SMD-Pad_Small" H 6900 5000 50  0001 C CNN
 F 3 "" H 6900 5000 50  0001 C CNN
@@
 F 0 "R1" V 5280 2750 50  0000 C CNN
 F 1 "37" V 5200 2750 50  0000 C CNN
-F 2 "Resistors_SMD:R_0805" V 5130 2750 50  0001 C CNN
+F 2 "Resistors_THT:R_Axial_DIN0207_L6.3mm_D2.5mm_P7.62mm_Horizontal" V 5130 2750 50  0001 C CNN
 F 3 "" H 5200 2750 50  0001 C CNN
 	1    5200 2750
@@
 F 0 "R2" V 5280 3050 50  0000 C CNN
 F 1 "37" V 5200 3050 50  0000 C CNN
-F 2 "Resistors_SMD:R_0805" V 5130 3050 50  0001 C CNN
+F 2 "Resistors_THT:R_Axial_DIN0207_L6.3mm_D2.5mm_P7.62mm_Horizontal" V 5130 3050 50  0001 C CNN
 F 3 "" H 5200 3050 50  0001 C CNN
 	1    5200 3050
@@
 F 0 "R3" V 5280 3350 50  0000 C CNN
 F 1 "37" V 5200 3350 50  0000 C CNN
-F 2 "Resistors_SMD:R_0805" V 5130 3350 50  0001 C CNN
+F 2 "Resistors_THT:R_Axial_DIN0207_L6.3mm_D2.5mm_P7.62mm_Horizontal" V 5130 3350 50  0001 C CNN
 F 3 "" H 5200 3350 50  0001 C CNN
 	1    5200 3350
@@
 F 0 "R4" V 5280 3650 50  0000 C CNN
 F 1 "37" V 5200 3650 50  0000 C CNN
-F 2 "Resistors_SMD:R_0805" V 5130 3650 50  0001 C CNN
+F 2 "Resistors_THT:R_Axial_DIN0207_L6.3mm_D2.5mm_P7.62mm_Horizontal" V 5130 3650 50  0001 C CNN
 F 3 "" H 5200 3650 50  0001 C CNN
 	1    5200 3650
@@
 F 0 "R5" V 5280 3950 50  0000 C CNN
 F 1 "37" V 5200 3950 50  0000 C CNN
-F 2 "Resistors_SMD:R_0805" V 5130 3950 50  0001 C CNN
+F 2 "Resistors_THT:R_Axial_DIN0207_L6.3mm_D2.5mm_P7.62mm_Horizontal" V 5130 3950 50  0001 C CNN
 F 3 "" H 5200 3950 50  0001 C CNN
 	1    5200 3950
@@
 F 0 "R6" V 5280 4250 50  0000 C CNN
 F 1 "37" V 5200 4250 50  0000 C CNN
-F 2 "Resistors_SMD:R_0805" V 5130 4250 50  0001 C CNN
+F 2 "Resistors_THT:R_Axial_DIN0207_L6.3mm_D2.5mm_P7.62mm_Horizontal" V 5130 4250 50  0001 C CNN
 F 3 "" H 5200 4250 50  0001 C CNN
 	1    5200 4250
@@
 F 0 "R7" V 5280 4550 50  0000 C CNN
 F 1 "37" V 5200 4550 50  0000 C CNN
-F 2 "Resistors_SMD:R_0805" V 5130 4550 50  0001 C CNN
+F 2 "Resistors_THT:R_Axial_DIN0207_L6.3mm_D2.5mm_P7.62mm_Horizontal" V 5130 4550 50  0001 C CNN
 F 3 "" H 5200 4550 50  0001 C CNN
 	1    5200 4550
@@
 F 0 "R8" V 5280 4850 50  0000 C CNN
 F 1 "37" V 5200 4850 50  0000 C CNN
-F 2 "Resistors_SMD:R_0805" V 5130 4850 50  0001 C CNN
+F 2 "Resistors_THT:R_Axial_DIN0207_L6.3mm_D2.5mm_P7.62mm_Horizontal" V 5130 4850 50  0001 C CNN
 F 3 "" H 5200 4850 50  0001 C CNN
 	1    5200 4850
@@
 $EndComp
 $Comp
-L GNDREF #PWR?
+L GNDREF #PWR01
 U 1 1 58E21BBF
 P 4600 2500
-F 0 "#PWR?" H 4600 2250 50  0001 C CNN
+F 0 "#PWR01" H 4600 2250 50  0001 C CNN
 F 1 "GNDREF" H 4600 2350 50  0000 C CNN
 F 2 "" H 4600 2500 50  0001 C CNN
