File: narra 0805design/narra 0805design.kicad_pcb (KiCad board)
At the start: 2 copper layers, 6 x 41 mm, 8 parts

Commit message: Added a soldering pad and protection resistors to the LED0805 design
Parts:
- added J1: P1_rows, Measurement_Points:Measurement_Point_Square-SMD-Pad_Small, F.Cu at (125.3, 119.1)
- added J2: P2_columns, Measurement_Points:Measurement_Point_Square-SMD-Pad_Small, F.Cu at (162.8, 118.6)
- added R1: 37, Resistors_SMD:R_0805, F.Cu at (129.9, 120.9)
- added R2: 37, Resistors_SMD:R_0805, F.Cu at (134.0, 120.9)
- added R3: 37, Resistors_SMD:R_0805, F.Cu at (138.0, 120.9)
- added R4: 37, Resistors_SMD:R_0805, F.Cu at (142.1, 120.9)
- added R5: 37, Resistors_SMD:R_0805, F.Cu at (146.2, 120.9)
- added R6: 37, Resistors_SMD:R_0805, F.Cu at (150.2, 120.9)
- added R7: 37, Resistors_SMD:R_0805, F.Cu at (154.4, 120.9)
- added R8: 37, Resistors_SMD:R_0805, F.Cu at (158.6, 120.9)
- moved D1 63.6 mm to (130.3, 116.5), turned to 90 degrees
- moved D2 60.1 mm to (134.6, 116.5), turned to 90 degrees
- moved D3 57.1 mm to (138.7, 116.5), turned to 90 degrees
- moved D4 54.6 mm to (142.7, 116.5), turned to 90 degrees
- moved D5 52.9 mm to (146.8, 116.5), turned to 90 degrees
- moved D8 52.3 mm to (159.1, 116.5), turned to 90 degrees
- moved D6 51.9 mm to (150.9, 116.5), turned to 90 degrees
- moved D7 51.6 mm to (154.9, 116.5), turned to 90 degrees
Connections:
- D1 pad 1: /Rows_cathode -> Net-(D1-Pad1)
- D2 pad 1: /Rows_cathode -> Net-(D2-Pad1)
- D3 pad 1: /Rows_cathode -> Net-(D3-Pad1)
- D4 pad 1: /Rows_cathode -> Net-(D4-Pad1)
- D5 pad 1: /Rows_cathode -> Net-(D5-Pad1)
- D6 pad 1: /Rows_cathode -> Net-(D6-Pad1)
- D7 pad 1: /Rows_cathode -> Net-(D7-Pad1)
- D8 pad 1: /Rows_cathode -> Net-(D8-Pad1)
Routing:
- net Net-(D1-Pad1): track 0.00 -> 3.62 mm
- net Net-(D8-Pad1): track 0.00 -> 3.53 mm
- net Net-(D7-Pad1): track 0.00 -> 3.53 mm
- net Net-(D6-Pad1): track 0.00 -> 3.48 mm
- net Net-(D5-Pad1): track 0.00 -> 3.48 mm
- net Net-(D4-Pad1): track 0.00 -> 3.48 mm
- net Net-(D3-Pad1): track 0.00 -> 3.48 mm
- net Net-(D2-Pad1): track 0.00 -> 3.48 mm
- net /Rows_cathode: track 46.7 -> 49.7 mm
Other:
- board size 6 x 41 mm -> 43.2 x 10.2 mm
- rule pad_to_mask_clearance: 0.2 -> 0

Commit message: Modified schematic and board level design ========================================= -Added gndref symbol to schematic -Expanded board edge so as to add clearance to edge from anode traces. -Connected copper fill zone to cathode connection point in order to provide a low inductance and resistance path for current. -Deleted traces to cathode connection point from the protection resistors.
Routing:
- net /Rows_cathode: track 49.7 -> 0.00 mm
- added copper zone on F.Cu, net /Rows_cathode
- removed copper zone on F.Cu, net (none)
Other:
- board size 43.2 x 10.2 mm -> 43.2 x 10.9 mm
Changed lines of the file:
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@@
-(kicad_pcb (version 4) (host pcbnew 4.0.6-e0-6349~53~ubuntu16.04.1)
+(kicad_pcb (version 20170123) (host pcbnew no-vcs-found-9c2ebf3~58~ubuntu16.04.1)
   (general
     (links 24)
     (no_connects 0)
-    (area 122.30288 113.487999 165.889 123.748001)
+    (area 122.301 112.720577 165.9065 123.748001)
     (thickness 1.6)
-    (drawings 5)
-    (tracks 60)
+    (drawings 4)
+    (tracks 35)
     (zones 0)
     (modules 18)
@@
       (hpglpenspeed 20)
       (hpglpendiameter 15)
-      (hpglpenoverlay 2)
       (psnegative false)
       (psa4output false)
@@
     )
   )
-  (gr_line (start 122.428 123.698) (end 122.682 123.698) (angle 90) (layer Edge.Cuts) (width 0.1))
-  (gr_line (start 122.428 113.538) (end 122.428 123.698) (angle 90) (layer Edge.Cuts) (width 0.1))
-  (gr_line (start 165.608 113.538) (end 122.428 113.538) (angle 90) (layer Edge.Cuts) (width 0.1))
-  (gr_line (start 165.608 123.698) (end 165.608 113.538) (angle 90) (layer Edge.Cuts) (width 0.1))
+  (gr_line (start 165.608 112.776) (end 122.428 112.776) (layer Edge.Cuts) (width 0.1))
+  (gr_line (start 165.608 123.698) (end 165.608 112.776) (layer Edge.Cuts) (width 0.1))
+  (gr_line (start 122.428 112.776) (end 122.428 123.698) (layer Edge.Cuts) (width 0.1))
   (gr_line (start 122.428 123.698) (end 165.608 123.698) (angle 90) (layer Edge.Cuts) (width 0.1))
   (segment (start 159.131 115.359) (end 159.131 114.046) (width 0.25) (layer F.Cu) (net 1))
@@
   (segment (start 159.573 120.904) (end 159.573 118.001) (width 0.25) (layer F.Cu) (net 9))
   (segment (start 159.573 118.001) (end 159.131 117.559) (width 0.25) (layer F.Cu) (net 9))
-  (segment (start 128.96592 120.94464) (end 128.96592 122.682) (width 0.25) (layer F.Cu) (net 10))
-  (segment (start 128.96592 122.682) (end 129.032 122.682) (width 0.25) (layer F.Cu) (net 10))
-  (segment (start 133.035 120.904) (end 133.035 122.682) (width 0.25) (layer F.Cu) (net 10))
-  (segment (start 133.035 122.682) (end 132.842 122.682) (width 0.25) (layer F.Cu) (net 10))
-  (segment (start 137.099 120.904) (end 137.099 122.682) (width 0.25) (layer F.Cu) (net 10))
-  (segment (start 137.099 122.682) (end 137.16 122.682) (width 0.25) (layer F.Cu) (net 10))
-  (segment (start 141.163 120.904) (end 141.163 122.682) (width 0.25) (layer F.Cu) (net 10))
-  (segment (start 141.163 122.682) (end 141.224 122.682) (width 0.25) (layer F.Cu) (net 10))
-  (segment (start 145.227 120.904) (end 145.227 122.682) (width 0.25) (layer F.Cu) (net 10))
-  (segment (start 145.227 122.682) (end 145.034 122.682) (width 0.25) (layer F.Cu) (net 10))
-  (segment (start 149.291 120.904) (end 149.291 122.682) (width 0.25) (layer F.Cu) (net 10))
-  (segment (start 149.291 122.682) (end 149.352 122.682) (width 0.25) (layer F.Cu) (net 10))
-  (segment (start 153.482 120.904) (end 153.482 122.682) (width 0.25) (layer F.Cu) (net 10))
-  (segment (start 153.482 122.682) (end 153.416 122.682) (width 0.25) (layer F.Cu) (net 10))
-  (segment (start 125.27788 119.1006) (end 125.27788 122.48388) (width 0.25) (layer F.Cu) (net 10))
-  (segment (start 155.895 122.682) (end 157.673 120.904) (width 0.25) (layer F.Cu) (net 10))
-  (segment (start 125.476 122.682) (end 129.032 122.682) (width 0.25) (layer F.Cu) (net 10))
-  (segment (start 129.032 122.682) (end 132.842 122.682) (width 0.25) (layer F.Cu) (net 10))
-  (segment (start 132.842 122.682) (end 137.16 122.682) (width 0.25) (layer F.Cu) (net 10))
-  (segment (start 137.16 122.682) (end 141.224 122.682) (width 0.25) (layer F.Cu) (net 10))
-  (segment (start 141.224 122.682) (end 145.034 122.682) (width 0.25) (layer F.Cu) (net 10))
-  (segment (start 145.034 122.682) (end 149.352 122.682) (width 0.25) (layer F.Cu) (net 10))
-  (segment (start 149.352 122.682) (end 153.416 122.682) (width 0.25) (layer F.Cu) (net 10))
-  (segment (start 153.416 122.682) (end 155.895 122.682) (width 0.25) (layer F.Cu) (net 10))
-  (segment (start 125.27788 122.48388) (end 125.476 122.682) (width 0.25) (layer F.Cu) (net 10))
-  (zone (net 0) (net_name "") (layer F.Cu) (hatch edge 0.508)
+  (zone (net 10) (net_name /Rows_cathode) (layer F.Cu) (hatch edge 0.508)
     (connect_pads (clearance 0.508))
     (min_thickness 0.254)
@@
     (polygon
       (pts
-        (xy 165.608 113.538) (xy 165.608 123.698) (xy 122.428 123.698) (xy 122.428 113.538)
+        (xy 165.481 112.720577) (xy 165.608 123.642577) (xy 122.428 123.642577) (xy 122.301 112.720577)
       )
     )
