File: narra 0805design/narra 0805design.kicad_pcb (KiCad board)
At the start: 2 copper layers, 61 x 11.7 mm, 18 parts, among them J1 Rows, J2 Columns

Commit message: made a footprint to match the dimensions of the actual chip for the 5050 design
Parts:
- moved D8 0.28 mm to (208.0, 88.5)
Routing:
- net /C: track 56.6 -> 59.5 mm
Other:
- board text added: "+"
