File: narra 0805design/narra 0805design.kicad_pcb (KiCad board)
At the start: 2 copper layers, 43.2 x 10.9 mm, 18 parts, among them J1 P1_rows, J2 P2_columns

Commit message: Changed SMD resistor footprint to through-hole type.
Parts:
- J1: value P1_rows -> Rows
- J2: value P2_columns -> Columns
- R1, R2, R3, R4, R5, R6, R7, R8: footprint Resistors_SMD:R_0805 -> Resistors_THT:R_Axial_DIN0207_L6.3mm_D2.5mm_P7.62mm_Horizontal
- moved R8 58.5 mm to (204.7, 84.8), turned to 270 degrees
- moved D8 56.5 mm to (208.3, 88.6), turned to 270 degrees
- moved R6 54.4 mm to (191.0, 84.8), turned to 270 degrees
- moved D7 53.9 mm to (201.2, 88.6)
- moved J2 52.5 mm to (208.3, 92.5), turned to 0 degrees
- moved R7 51.7 mm to (197.6, 92.5), turned to 90 degrees
- moved D6 51.6 mm to (194.3, 88.6), turned to 270 degrees
- moved R4 49.3 mm to (175.8, 84.8), turned to 270 degrees
- moved D5 48.8 mm to (186.9, 88.6)
- moved R5 46.8 mm to (183.4, 92.5), turned to 90 degrees
- moved D4 46.2 mm to (179.6, 88.6), turned to 270 degrees
- moved R2 45.5 mm to (161.8, 84.8), turned to 270 degrees
- moved D3 43.6 mm to (172.2, 88.6)
- moved J1 42.9 mm to (151.1, 84.8), turned to 0 degrees
- moved R3 41.8 mm to (168.7, 92.5), turned to 90 degrees
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Connections:
- net /Columns_anode renamed /C
- net /Rows_cathode renamed GNDREF
Routing:
- net GNDREF: track 0.00 -> 119.6 mm
- net /C: track 46.8 -> 56.6 mm
- net Net-(D4-Pad1): track 3.48 -> 6.37 mm
- net Net-(D5-Pad1): track 3.48 -> 6.27 mm
- net Net-(D3-Pad1): track 3.48 -> 6.27 mm
- net Net-(D8-Pad1): track 3.53 -> 6.27 mm
- net Net-(D7-Pad1): track 3.53 -> 6.27 mm
- net Net-(D2-Pad1): track 3.48 -> 6.01 mm
- net Net-(D1-Pad1): track 3.62 -> 6.01 mm
- net Net-(D6-Pad1): track 3.48 -> 5.86 mm
Other:
- board size 43.2 x 10.9 mm -> 61 x 11.7 mm

Commit message: finalise matrix column design prior to meshing design
Parts:
- moved R8 0.63 mm to (204.1, 84.8)
Routing:
- net GNDREF: track 119.6 -> 0.00 mm
- net /C: track 56.6 -> 59.3 mm
- net Net-(D7-Pad1): track 6.27 -> 5.60 mm
- net Net-(D4-Pad1): track 6.37 -> 5.70 mm
- net Net-(D3-Pad1): track 6.27 -> 5.60 mm
- net Net-(D2-Pad1): track 6.01 -> 5.34 mm
- net Net-(D5-Pad1): track 6.27 -> 5.67 mm
- net Net-(D1-Pad1): track 6.01 -> 5.42 mm
- net Net-(D6-Pad1): track 5.86 -> 5.34 mm
