File: drivers/ND-01/ND01 output.sch (KiCad schematic (older format))
At the start: 13 parts, among them J10 CONN_01X08, J11 CONN_01X08, J12 CONN_01X08, J13 CONN_01X08, J14 CONN_01X08, J15 CONN_01X08, J16 CONN_01X08, J4 CONN_01X08, J5 CONN_01X08, J6 CONN_01X08, J7 CONN_01X08, J8 CONN_01X08, J9 CONN_01X08

Commit message: Add 2088xS LED dot matrix documentation pictures
Changed lines of the file:
@@
 	5300 900  5400 900
 Wire Bus Line
-	5400 900  5400 950
-Wire Bus Line
-	5400 950  5400 1050
-Wire Bus Line
-	5400 1050 5400 1150
-Wire Bus Line
-	5400 1150 5400 1250
-Wire Bus Line
-	5400 1250 5400 1350
-Wire Bus Line
-	5400 1350 5400 1450
-Wire Bus Line
-	5400 1450 5400 1550
-Wire Bus Line
-	5400 1550 5400 1650
-Wire Bus Line
-	5400 1650 5400 1800
+	5400 900  5400 1800
 $Comp
 L CONN_01X08 J4
@@
 	1200 2500 1500 2500
 Wire Bus Line
-	1500 2500 1500 2550
-Wire Bus Line
-	1500 2550 1500 2650
-Wire Bus Line
-	1500 2650 1500 2750
-Wire Bus Line
-	1500 2750 1500 2850
-Wire Bus Line
-	1500 2850 1500 2950
-Wire Bus Line
-	1500 2950 1500 3050
-Wire Bus Line
-	1500 3050 1500 3150
-Wire Bus Line
-	1500 3150 1500 3250
-Wire Bus Line
-	1500 3250 1500 3400
+	1500 2500 1500 3400
 $Comp
 L CONN_01X08 J5
@@
 	2900 2500 3200 2500
 Wire Bus Line
-	3200 2500 3200 2550
-Wire Bus Line
-	3200 2550 3200 2650
-Wire Bus Line
-	3200 2650 3200 2750
-Wire Bus Line
-	3200 2750 3200 2850
-Wire Bus Line
-	3200 2850 3200 2950
-Wire Bus Line
-	3200 2950 3200 3050
-Wire Bus Line
-	3200 3050 3200 3150
-Wire Bus Line
-	3200 3150 3200 3250
-Wire Bus Line
-	3200 3250 3200 3400
+	3200 2500 3200 3400
 $Comp
 L CONN_01X08 J6
@@
 	4600 2500 4900 2500
 Wire Bus Line
-	4900 2500 4900 2550
-Wire Bus Line
-	4900 2550 4900 2650
-Wire Bus Line
-	4900 2650 4900 2750
-Wire Bus Line
-	4900 2750 4900 2850
-Wire Bus Line
-	4900 2850 4900 2950
-Wire Bus Line
-	4900 2950 4900 3050
-Wire Bus Line
-	4900 3050 4900 3150
-Wire Bus Line
-	4900 3150 4900 3250
-Wire Bus Line
-	4900 3250 4900 3400
+	4900 2500 4900 3400
 $Comp
 L CONN_01X08 J7
@@
 	6200 2500 6500 2500
 Wire Bus Line
-	6500 2500 6500 2550
-Wire Bus Line
-	6500 2550 6500 2650
-Wire Bus Line
-	6500 2650 6500 2750
-Wire Bus Line
-	6500 2750 6500 2850
-Wire Bus Line
-	6500 2850 6500 2950
-Wire Bus Line
-	6500 2950 6500 3050
-Wire Bus Line
-	6500 3050 6500 3150
-Wire Bus Line
-	6500 3150 6500 3250
-Wire Bus Line
-	6500 3250 6500 3400
+	6500 2500 6500 3400
 $Comp
 L CONN_01X08 J8
@@
 	7750 2500 8050 2500
 Wire Bus Line
-	8050 2500 8050 2550
-Wire Bus Line
-	8050 2550 8050 2650
-Wire Bus Line
-	8050 2650 8050 2750
-Wire Bus Line
-	8050 2750 8050 2850
-Wire Bus Line
-	8050 2850 8050 2950
-Wire Bus Line
-	8050 2950 8050 3050
-Wire Bus Line
-	8050 3050 8050 3150
-Wire Bus Line
-	8050 3150 8050 3250
-Wire Bus Line
-	8050 3250 8050 3400
+	8050 2500 8050 3400
 $Comp
 L CONN_01X08 J9
@@
 	9300 2500 9600 2500
 Wire Bus Line
-	9600 2500 9600 2550
-Wire Bus Line
-	9600 2550 9600 2650
-Wire Bus Line
-	9600 2650 9600 2750
-Wire Bus Line
-	9600 2750 9600 2850
-Wire Bus Line
-	9600 2850 9600 2950
-Wire Bus Line
-	9600 2950 9600 3050
-Wire Bus Line
-	9600 3050 9600 3150
-Wire Bus Line
-	9600 3150 9600 3250
-Wire Bus Line
-	9600 3250 9600 3400
+	9600 2500 9600 3400
 $Comp
 L CONN_01X08 J10
@@
 	1200 4050 1500 4050
 Wire Bus Line
-	1500 4050 1500 4100
-Wire Bus Line
-	1500 4100 1500 4200
-Wire Bus Line
-	1500 4200 1500 4300
-Wire Bus Line
-	1500 4300 1500 4400
-Wire Bus Line
-	1500 4400 1500 4500
-Wire Bus Line
-	1500 4500 1500 4600
-Wire Bus Line
-	1500 4600 1500 4700
-Wire Bus Line
-	1500 4700 1500 4800
-Wire Bus Line
-	1500 4800 1500 4950
+	1500 4050 1500 4950
 $Comp
 L CONN_01X08 J11
@@
 	2900 4050 3200 4050
 Wire Bus Line
-	3200 4050 3200 4100
-Wire Bus Line
-	3200 4100 3200 4200
-Wire Bus Line
-	3200 4200 3200 4300
-Wire Bus Line
-	3200 4300 3200 4400
-Wire Bus Line
-	3200 4400 3200 4500
-Wire Bus Line
-	3200 4500 3200 4600
-Wire Bus Line
-	3200 4600 3200 4700
-Wire Bus Line
-	3200 4700 3200 4800
-Wire Bus Line
-	3200 4800 3200 4950
+	3200 4050 3200 4950
 $Comp
 L CONN_01X08 J12
@@
 	4600 4050 4900 4050
 Wire Bus Line
-	4900 4050 4900 4100
-Wire Bus Line
-	4900 4100 4900 4200
-Wire Bus Line
-	4900 4200 4900 4300
-Wire Bus Line
-	4900 4300 4900 4400
-Wire Bus Line
-	4900 4400 4900 4500
-Wire Bus Line
-	4900 4500 4900 4600
-Wire Bus Line
-	4900 4600 4900 4700
-Wire Bus Line
-	4900 4700 4900 4800
-Wire Bus Line
-	4900 4800 4900 4950
+	4900 4050 4900 4950
 $Comp
 L CONN_01X08 J13
@@
 	6200 4050 6500 4050
 Wire Bus Line
-	6500 4050 6500 4100
-Wire Bus Line
-	6500 4100 6500 4200
-Wire Bus Line
-	6500 4200 6500 4300
-Wire Bus Line
-	6500 4300 6500 4400
-Wire Bus Line
-	6500 4400 6500 4500
-Wire Bus Line
-	6500 4500 6500 4600
-Wire Bus Line
-	6500 4600 6500 4700
-Wire Bus Line
-	6500 4700 6500 4800
-Wire Bus Line
-	6500 4800 6500 4950
+	6500 4050 6500 4950
 $Comp
 L CONN_01X08 J14
@@
 	7750 4050 8050 4050
 Wire Bus Line
-	8050 4050 8050 4100
-Wire Bus Line
-	8050 4100 8050 4200
-Wire Bus Line
-	8050 4200 8050 4300
-Wire Bus Line
-	8050 4300 8050 4400
-Wire Bus Line
-	8050 4400 8050 4500
-Wire Bus Line
-	8050 4500 8050 4600
-Wire Bus Line
-	8050 4600 8050 4700
-Wire Bus Line
-	8050 4700 8050 4800
-Wire Bus Line
-	8050 4800 8050 4950
+	8050 4050 8050 4950
 $Comp
 L CONN_01X08 J15
@@
 	9300 4050 9600 4050
 Wire Bus Line
-	9600 4050 9600 4100
-Wire Bus Line
-	9600 4100 9600 4200
-Wire Bus Line
-	9600 4200 9600 4300
-Wire Bus Line
-	9600 4300 9600 4400
-Wire Bus Line
-	9600 4400 9600 4500
-Wire Bus Line
-	9600 4500 9600 4600
-Wire Bus Line
-	9600 4600 9600 4700
-Wire Bus Line
-	9600 4700 9600 4800
-Wire Bus Line
-	9600 4800 9600 4950
+	9600 4050 9600 4950
 $Comp
 L CONN_01X08 J16

Commit message: Add separate driver uses to schematic
Parts:
- added M?: MATRIX, pochi:Dot_matrix_CC_2088-AS, symbol MATRIX
Connections:
- net C0: now also M?.c0 (COL0)
- net C1: now also M?.C1 (COL1)
- net C10: now also M?.c12 (COL12)
- net C11: now also M?.c13 (COL13)
- net C12: now also M?.c14 (COL14)
- net C13: now also M?.c15 (COL15)
- net C16: now also M?.c16 (COL16)
- net C17: now also M?.c17 (COL17)
- net C18: now also M?.c18 (COL18)
- net C19: now also M?.c19 (COL19)
- net C2: now also M?.c2 (COL2)
- net C20: now also M?.c20 (COL20)
- net C21: now also M?.c21 (COL21)
- net C22: now also M?.c22 (COL22)
- net C23: now also M?.c23 (COL23)
- net C24: now also M?.c26 (COL26)
- net C25: now also M?.c27 (COL27)
- net C26: now also M?.c28 (COL28)
- net C27: now also M?.c29 (COL29)
- net C28: now also M?.c30 (COL30)
- net C29: now also M?.c31 (COL31)
- net C3: now also M?.c3 (COL3)
- net C4: now also M?.c4 (COL4)
- net C5: now also M?.c5 (COL5)
- net C6: now also M?.c6 (COL6)
- net C7: now also M?.c7 (COL7)
- net C8: now also M?.c10 (COL10)
- net C9: now also M?.c11 (COL11)
- net R0: now also M?.r0 (ROW0)
- net R1: now also M?.r1 (ROW1)
- net R2: now also M?.r2 (ROW2)
- net R3: now also M?.r3 (ROW3)
- net R4: now also M?.r4 (ROW4)
- net R5: now also M?.r5 (ROW5)
- net R6: now also M?.r6 (ROW6)
- net R7: now also M?.r7 (ROW7)
Other:
- note added: "COLUMN OUTPUTS(For external driver use)"
- note added: "MATRIX OUTPUT(For device driver use)"
- note added: "ROW OUTPUTS(For external driver use)"
- note removed: "COLUMN OUTPUTS"
- note removed: "ROW OUTPUTS"
- moved on the sheet: J10, J11, J12, J13, J14, J15, J16, J5, J6, J7, J8, J9

Commit message: Add protection resistors
Parts:
- added R? (x8): R, symbol R
Connections:
- net R0: now also R?.1; no longer M?.r0 (ROW0)
- net R1: now also R?.1; no longer M?.r1 (ROW1)
- net R2: now also R?.1; no longer M?.r2 (ROW2)
- net R3: now also R?.1; no longer M?.r3 (ROW3)
- net R4: now also R?.1; no longer M?.r4 (ROW4)
- net R5: now also R?.1; no longer M?.r5 (ROW5)
- net R6: now also R?.1; no longer M?.r6 (ROW6)
- net R7: now also R?.1; no longer M?.r7 (ROW7)
- new net: M?.r0 (ROW0), R?.2
- new net: M?.r1 (ROW1), R?.2
- new net: M?.r2 (ROW2), R?.2
- new net: M?.r3 (ROW3), R?.2
- new net: M?.r4 (ROW4), R?.2
- new net: M?.r5 (ROW5), R?.2
- new net: M?.r6 (ROW6), R?.2
- new net: M?.r7 (ROW7), R?.2
Other:
- moved on the sheet: M?
Changed lines of the file:
@@
 EESchema Schematic File Version 2
-LIBS:ND-01-rescue
 LIBS:power
 LIBS:device
@@
 	500  2050 11200 2050
 Entry Wire Line
-	1650 5400 1750 5500
-Entry Wire Line
 	1650 5500 1750 5600
 Entry Wire Line
@@
 	1650 6100 1750 6200
 Entry Wire Line
-	1650 6400 1750 6500
+	1650 6200 1750 6300
 Entry Wire Line
 	1650 6500 1750 6600
@@
 Entry Wire Line
 	1650 7100 1750 7200
+Entry Wire Line
+	1650 7200 1750 7300
 Wire Bus Line
-	1650 7250 1650 6300
+	1650 7350 1650 6400
 Wire Bus Line
-	1650 6300 1500 6300
+	1650 6400 1500 6400
 Wire Bus Line
-	1650 6200 1650 5300
+	1650 6300 1650 5400
 Wire Bus Line
-	1650 5300 1500 5300
+	1650 5400 1500 5400
+Entry Wire Line
+	3150 6300 3250 6200
 Entry Wire Line
 	3150 6200 3250 6100
@@
 	3150 5600 3250 5500
 Entry Wire Line
-	3150 5500 3250 5400
-Entry Wire Line
-	3150 6500 3250 6400
-Entry Wire Line
 	3150 6600 3250 6500
 Entry Wire Line
@@
 Entry Wire Line
 	3150 7200 3250 7100
+Entry Wire Line
+	3150 7300 3250 7200
 Wire Bus Line
-	3250 7250 3250 6250
+	3250 7350 3250 6350
 Wire Bus Line
-	3250 6250 3400 6250
+	3250 6350 3400 6350
 Wire Bus Line
-	3250 6200 3250 5250
+	3250 6300 3250 5350
 Wire Bus Line
-	3250 5250 3400 5250
-Text HLabel 1500 5300 0    39   Input ~ 0
+	3250 5350 3400 5350
+Text HLabel 1500 5400 0    39   Input ~ 0
 COL[0:7]
-Text HLabel 1500 6300 0    39   Input ~ 0
+Text HLabel 1500 6400 0    39   Input ~ 0
 COL[8:15]
-Text HLabel 3400 5250 2    39   Input ~ 0
+Text HLabel 3400 5350 2    39   Input ~ 0
 COL[16:23]
-Text HLabel 3400 6250 2    39   Input ~ 0
+Text HLabel 3400 6350 2    39   Input ~ 0
 COL[24:31]
 Wire Wire Line
-	1850 5500 1750 5500
-Wire Wire Line
 	1850 5600 1750 5600
 Wire Wire Line
@@
 	1850 6200 1750 6200
 Wire Wire Line
-	1850 6500 1750 6500
+	1850 6300 1750 6300
 Wire Wire Line
 	1850 6600 1750 6600
@@
 	1850 7200 1750 7200
 Wire Wire Line
-	3150 5500 3050 5500
+	1850 7300 1750 7300
 Wire Wire Line
-	3050 5600 3150 5600
+	3150 5600 3050 5600
 Wire Wire Line
-	3150 5700 3050 5700
+	3050 5700 3150 5700
 Wire Wire Line
 	3150 5800 3050 5800
@@
 	3150 6200 3050 6200
 Wire Wire Line
-	3150 6500 3050 6500
+	3150 6300 3050 6300
 Wire Wire Line
 	3150 6600 3050 6600
@@
 	3150 6700 3050 6700
 Wire Wire Line
-	3150 6900 3050 6900
-Wire Wire Line
 	3150 6800 3050 6800
 Wire Wire Line
 	3150 7000 3050 7000
 Wire Wire Line
+	3150 6900 3050 6900
+Wire Wire Line
 	3150 7100 3050 7100
 Wire Wire Line
 	3150 7200 3050 7200
-Text Label 1750 5500 0    39   ~ 0
-C0
+Wire Wire Line
+	3150 7300 3050 7300
 Text Label 1750 5600 0    39   ~ 0
-C1
+C0
 Text Label 1750 5700 0    39   ~ 0
-C2
+C1
 Text Label 1750 5800 0    39   ~ 0
-C3
+C2
 Text Label 1750 5900 0    39   ~ 0
-C4
+C3
 Text Label 1750 6000 0    39   ~ 0
-C5
+C4
 Text Label 1750 6100 0    39   ~ 0
-C6
+C5
 Text Label 1750 6200 0    39   ~ 0
+C6
+Text Label 1750 6300 0    39   ~ 0
 C7
-Text Label 1750 6500 0    39   ~ 0
-C8
 Text Label 1750 6600 0    39   ~ 0
-C9
+C8
 Text Label 1750 6700 0    39   ~ 0
-C10
+C9
 Text Label 1750 6800 0    39   ~ 0
-C11
+C10
 Text Label 1750 6900 0    39   ~ 0
-C12
+C11
 Text Label 1750 7000 0    39   ~ 0
-C13
+C12
 Text Label 1750 7100 0    39   ~ 0
-C14
+C13
 Text Label 1750 7200 0    39   ~ 0
+C14
+Text Label 1750 7300 0    39   ~ 0
 C15
-Text Label 3050 5500 0    39   ~ 0
-C16
 Text Label 3050 5600 0    39   ~ 0
-C17
+C16
 Text Label 3050 5700 0    39   ~ 0
-C18
+C17
 Text Label 3050 5800 0    39   ~ 0
-C19
+C18
 Text Label 3050 5900 0    39   ~ 0
-C20
+C19
 Text Label 3050 6000 0    39   ~ 0
-C21
+C20
 Text Label 3050 6100 0    39   ~ 0
-C22
+C21
 Text Label 3050 6200 0    39   ~ 0
+C22
+Text Label 3050 6300 0    39   ~ 0
 C23
-Text Label 3050 6500 0    39   ~ 0
-C24
 Text Label 3050 6600 0    39   ~ 0
-C25
+C24
 Text Label 3050 6700 0    39   ~ 0
-C26
+C25
 Text Label 3050 6800 0    39   ~ 0
-C27
+C26
 Text Label 3050 6900 0    39   ~ 0
-C28
+C27
 Text Label 3050 7000 0    39   ~ 0
-C29
+C28
 Text Label 3050 7100 0    39   ~ 0
-C30
+C29
 Text Label 3050 7200 0    39   ~ 0
+C30
+Text Label 3050 7300 0    39   ~ 0
 C31
 Entry Wire Line
-	2100 4850 2200 4750
+	2100 4650 2200 4550
 Entry Wire Line
-	2200 4850 2300 4750
+	2200 4650 2300 4550
 Entry Wire Line
-	2300 4850 2400 4750
+	2300 4650 2400 4550
 Entry Wire Line
-	2400 4850 2500 4750
+	2400 4650 2500 4550
 Entry Wire Line
-	2500 4850 2600 4750
+	2500 4650 2600 4550
 Entry Wire Line
-	2600 4850 2700 4750
+	2600 4650 2700 4550
 Entry Wire Line
-	2700 4850 2800 4750
+	2700 4650 2800 4550
 Entry Wire Line
-	2800 4850 2900 4750
+	2800 4650 2900 4550
 Wire Bus Line
-	2050 4750 3000 4750
+	2050 4550 3000 4550
 Wire Bus Line
-	2050 4750 2050 4650
+	2050 4550 2050 4450
 Wire Bus Line
-	2050 4650 1950 4650
-Text HLabel 1950 4650 0    39   Input ~ 0
+	2050 4450 1950 4450
+Text HLabel 1950 4450 0    39   Input ~ 0
 ROW[0:7]
 Wire Wire Line
-	2100 4850 2100 4950
+	2100 4650 2100 4750
 Wire Wire Line
-	2200 4850 2200 4950
+	2200 4650 2200 4750
 Wire Wire Line
-	2300 4850 2300 4950
+	2300 4650 2300 4750
 Wire Wire Line
-	2400 4850 2400 4950
+	2400 4650 2400 4750
 Wire Wire Line
-	2500 4850 2500 4950
+	2500 4650 2500 4750
 Wire Wire Line
-	2600 4850 2600 4950
+	2600 4650 2600 4750
 Wire Wire Line
-	2700 4850 2700 4950
+	2700 4650 2700 4750
 Wire Wire Line
-	2800 4850 2800 4950
+	2800 4650 2800 4750
 Wire Notes Line
 	500  4400 11200 4400
-Text Label 2100 4950 1    39   ~ 0
+Text Label 2100 4750 1    39   ~ 0
 R0
-Text Label 2200 4950 1    39   ~ 0
+Text Label 2200 4750 1    39   ~ 0
 R1
-Text Label 2300 4950 1    39   ~ 0
+Text Label 2300 4750 1    39   ~ 0
 R2
-Text Label 2400 4950 1    39   ~ 0
+Text Label 2400 4750 1    39   ~ 0
 R3
-Text Label 2500 4950 1    39   ~ 0
+Text Label 2500 4750 1    39   ~ 0
 R4
-Text Label 2600 4950 1    39   ~ 0
+Text Label 2600 4750 1    39   ~ 0
 R5
-Text Label 2700 4950 1    39   ~ 0
+Text Label 2700 4750 1    39   ~ 0
 R6
-Text Label 2800 4950 1    39   ~ 0
+Text Label 2800 4750 1    39   ~ 0
 R7
 Text Notes 2350 4500 0    60   ~ 0
@@
 L MATRIX M?
 U 1 1 58ED21AF
-P 2950 6350
+P 2950 6450
 AR Path="/58ED21AF" Ref="M?"  Part="1"
 AR Path="/58E75CFC/58ED21AF" Ref="M?"  Part="1"
-F 0 "M?" V 4130 6850 60  0000 C CNN
-F 1 "MATRIX" V 4236 6850 60  0000 C CNN
-F 2 "pochi:Dot_matrix_CC_2088-AS" H 3050 6850 60  0001 C CNN
-F 3 "" H 2250 6800 60  0001 C CNN
-	1    2950 6350
+F 0 "M?" V 4130 6950 60  0000 C CNN
+F 1 "MATRIX" V 4236 6950 60  0000 C CNN
+F 2 "pochi:Dot_matrix_CC_2088-AS" H 3050 6950 60  0001 C CNN
+F 3 "" H 2250 6900 60  0001 C CNN
+	1    2950 6450
 	0    -1   1    0
 $EndComp
+$Comp
+L R R?
+U 1 1 58ECF1A7
+P 2100 4900
+F 0 "R?" H 2050 4950 50  0000 L CNN
+F 1 "R" H 2050 4850 50  0000 L CNN
+F 2 "" V 2030 4900 50  0001 C CNN
+F 3 "" H 2100 4900 50  0001 C CNN
+	1    2100 4900
+	1    0    0    -1
+$EndComp
+$Comp
+L R R?
+U 1 1 58ECF2DF
+P 2200 4900
+F 0 "R?" H 2150 4950 50  0000 L CNN
+F 1 "R" H 2150 4850 50  0000 L CNN
+F 2 "" V 2130 4900 50  0001 C CNN
+F 3 "" H 2200 4900 50  0001 C CNN
+	1    2200 4900
+	1    0    0    -1
+$EndComp
+$Comp
+L R R?
+U 1 1 58ECF317
+P 2300 4900
+F 0 "R?" H 2250 4950 50  0000 L CNN
+F 1 "R" H 2250 4850 50  0000 L CNN
+F 2 "" V 2230 4900 50  0001 C CNN
+F 3 "" H 2300 4900 50  0001 C CNN
+	1    2300 4900
+	1    0    0    -1
+$EndComp
+$Comp
+L R R?
+U 1 1 58ECF349
+P 2400 4900
+F 0 "R?" H 2350 4950 50  0000 L CNN
+F 1 "R" H 2350 4850 50  0000 L CNN
+F 2 "" V 2330 4900 50  0001 C CNN
+F 3 "" H 2400 4900 50  0001 C CNN
+	1    2400 4900
+	1    0    0    -1
+$EndComp
+$Comp
+L R R?
+U 1 1 58ECF37D
+P 2500 4900
+F 0 "R?" H 2450 4950 50  0000 L CNN
+F 1 "R" H 2450 4850 50  0000 L CNN
+F 2 "" V 2430 4900 50  0001 C CNN
+F 3 "" H 2500 4900 50  0001 C CNN
+	1    2500 4900
+	1    0    0    -1
+$EndComp
+$Comp
+L R R?
+U 1 1 58ECF3B3
+P 2600 4900
+F 0 "R?" H 2550 4950 50  0000 L CNN
+F 1 "R" H 2550 4850 50  0000 L CNN
+F 2 "" V 2530 4900 50  0001 C CNN
+F 3 "" H 2600 4900 50  0001 C CNN
+	1    2600 4900
+	1    0    0    -1
+$EndComp
+$Comp
+L R R?
+U 1 1 58ECF3EB
+P 2700 4900
+F 0 "R?" H 2650 4950 50  0000 L CNN
+F 1 "R" H 2650 4850 50  0000 L CNN
+F 2 "" V 2630 4900 50  0001 C CNN
+F 3 "" H 2700 4900 50  0001 C CNN
+	1    2700 4900
+	1    0    0    -1
+$EndComp
+$Comp
+L R R?
+U 1 1 58ECF425
+P 2800 4900
+F 0 "R?" H 2750 4950 50  0000 L CNN
+F 1 "R" H 2750 4850 50  0000 L CNN
+F 2 "" V 2730 4900 50  0001 C CNN
+F 3 "" H 2800 4900 50  0001 C CNN
+	1    2800 4900
+	1    0    0    -1
+$EndComp
 $EndSCHEMATC

Commit message: Add protection resistors to external row driver connector
Parts:
- added R? (x8): R, symbol R
Connections:
- net R0: now also R?.2; no longer J4.1 (P1)
- net R1: now also R?.2; no longer J4.2 (P2)
- net R2: now also R?.2; no longer J4.3 (P3)
- net R3: now also R?.2; no longer J4.4 (P4)
- net R4: now also R?.2; no longer J4.5 (P5)
- net R5: now also R?.2; no longer J4.6 (P6)
- net R6: now also R?.2; no longer J4.7 (P7)
- net R7: now also R?.2; no longer J4.8 (P8)
- new net: J4.1 (P1), R?.1
- new net: J4.2 (P2), R?.1
- new net: J4.3 (P3), R?.1
- new net: J4.4 (P4), R?.1
- new net: J4.5 (P5), R?.1
- new net: J4.6 (P6), R?.1
- new net: J4.7 (P7), R?.1
- new net: J4.8 (P8), R?.1
Other:
- moved on the sheet: J4
Changed lines of the file:
@@
 L CONN_01X08 J4
 U 1 1 58E76DCC
-P 5800 1400
-F 0 "J4" H 5878 1441 50  0000 L CNN
-F 1 "CONN_01X08" H 5878 1350 50  0000 L CNN
-F 2 "" H 5800 1400 50  0001 C CNN
-F 3 "" H 5800 1400 50  0001 C CNN
-	1    5800 1400
+P 6150 1400
+F 0 "J4" H 6228 1441 50  0000 L CNN
+F 1 "CONN_01X08" H 6228 1350 50  0000 L CNN
+F 2 "" H 6150 1400 50  0001 C CNN
+F 3 "" H 6150 1400 50  0001 C CNN
+	1    6150 1400
 	1    0    0    -1
 $EndComp
@@
 	5400 900  5400 1800
 Wire Wire Line
-	5600 1050 5500 1050
+	5950 1050 5850 1050
 Wire Wire Line
-	5600 1150 5500 1150
+	5950 1150 5850 1150
 Wire Wire Line
-	5600 1250 5500 1250
+	5950 1250 5850 1250
 Wire Wire Line
-	5600 1350 5500 1350
+	5950 1350 5850 1350
 Wire Wire Line
-	5600 1450 5500 1450
+	5950 1450 5850 1450
 Wire Wire Line
-	5600 1550 5500 1550
+	5950 1550 5850 1550
 Wire Wire Line
-	5600 1650 5500 1650
+	5950 1650 5850 1650
 Wire Wire Line
-	5600 1750 5500 1750
+	5950 1750 5850 1750
 Wire Bus Line
 	1200 2400 1500 2400
@@
 	1    0    0    -1
 $EndComp
+$Comp
+L R R?
+U 1 1 58ED01A9
+P 5700 1050
+F 0 "R?" V 5700 1050 50  0000 C CNN
+F 1 "R" V 5650 1200 50  0000 C CNN
+F 2 "" V 5630 1050 50  0001 C CNN
+F 3 "" H 5700 1050 50  0001 C CNN
+	1    5700 1050
+	0    1    1    0
+$EndComp
+$Comp
+L R R?
+U 1 1 58ED07F9
+P 5700 1150
+F 0 "R?" V 5700 1150 50  0000 C CNN
+F 1 "R" V 5650 1300 50  0000 C CNN
+F 2 "" V 5630 1150 50  0001 C CNN
+F 3 "" H 5700 1150 50  0001 C CNN
+	1    5700 1150
+	0    1    1    0
+$EndComp
+$Comp
+L R R?
+U 1 1 58ED08C9
+P 5700 1250
+F 0 "R?" V 5700 1250 50  0000 C CNN
+F 1 "R" V 5650 1400 50  0000 C CNN
+F 2 "" V 5630 1250 50  0001 C CNN
+F 3 "" H 5700 1250 50  0001 C CNN
+	1    5700 1250
+	0    1    1    0
+$EndComp
+$Comp
+L R R?
+U 1 1 58ED090B
+P 5700 1350
+F 0 "R?" V 5700 1350 50  0000 C CNN
+F 1 "R" V 5650 1500 50  0000 C CNN
+F 2 "" V 5630 1350 50  0001 C CNN
+F 3 "" H 5700 1350 50  0001 C CNN
+	1    5700 1350
+	0    1    1    0
+$EndComp
+$Comp
+L R R?
+U 1 1 58ED094F
+P 5700 1450
+F 0 "R?" V 5700 1450 50  0000 C CNN
+F 1 "R" V 5650 1600 50  0000 C CNN
+F 2 "" V 5630 1450 50  0001 C CNN
+F 3 "" H 5700 1450 50  0001 C CNN
+	1    5700 1450
+	0    1    1    0
+$EndComp
+$Comp
+L R R?
+U 1 1 58ED09E6
+P 5700 1550
+F 0 "R?" V 5700 1550 50  0000 C CNN
+F 1 "R" V 5650 1700 50  0000 C CNN
+F 2 "" V 5630 1550 50  0001 C CNN
+F 3 "" H 5700 1550 50  0001 C CNN
+	1    5700 1550
+	0    1    1    0
+$EndComp
+$Comp
+L R R?
+U 1 1 58ED0A32
+P 5700 1650
+F 0 "R?" V 5700 1650 50  0000 C CNN
+F 1 "R" V 5650 1800 50  0000 C CNN
+F 2 "" V 5630 1650 50  0001 C CNN
+F 3 "" H 5700 1650 50  0001 C CNN
+	1    5700 1650
+	0    1    1    0
+$EndComp
+$Comp
+L R R?
+U 1 1 58ED0A7C
+P 5700 1750
+F 0 "R?" V 5700 1750 50  0000 C CNN
+F 1 "R" V 5650 1900 50  0000 C CNN
+F 2 "" V 5630 1750 50  0001 C CNN
+F 3 "" H 5700 1750 50  0001 C CNN
+	1    5700 1750
+	0    1    1    0
+$EndComp
+Wire Wire Line
+	5500 1050 5550 1050
+Wire Wire Line
+	5500 1150 5550 1150
+Wire Wire Line
+	5500 1250 5550 1250
+Wire Wire Line
+	5500 1350 5550 1350
+Wire Wire Line
+	5500 1450 5550 1450
+Wire Wire Line
+	5500 1550 5550 1550
+Wire Wire Line
+	5500 1750 5550 1750
+Wire Wire Line
+	5500 1650 5550 1650
 $EndSCHEMATC

Commit message: semicomplete design
Parts:
- removed R? (x16): R, symbol R
- added J17, J18, J19, J20, J21, J22, J23, J24, J25, J26, J27, J28, J29, J30, J31, J32: GS2, Connectors:GS2, symbol GS2
- J10, J11, J12, J13, J14, J15, J16, J4, J5, J6, J7, J8, J9: footprint (none) -> Connectors_Molex:Molex_KK-6410-08_08x2.54mm_Straight
- gave numbers to parts that had none: 1
Connections:
- net R0: now also J17.2 (G2), J18.2 (G2)
- net R1: now also J19.2 (G2), J20.2 (G2)
- net R2: now also J21.2 (G2), J22.2 (G2)
- net R3: now also J23.2 (G2), J24.2 (G2)
- net R4: now also J25.2 (G2), J26.2 (G2)
- net R5: now also J27.2 (G2), J28.2 (G2)
- net R6: now also J29.2 (G2), J30.2 (G2)
- net R7: now also J31.2 (G2), J32.2 (G2)
- net EXT_R0: now reaches J4.1 (P1)
- net EXT_R0: now also J18.1 (G1)
- net EXT_R1: now reaches J4.2 (P2)
- net EXT_R1: now also J20.1 (G1)
- net EXT_R2: now reaches J4.3 (P3)
- net EXT_R2: now also J22.1 (G1)
- net EXT_R3: now reaches J4.4 (P4)
- net EXT_R3: now also J24.1 (G1)
- net EXT_R4: now reaches J4.5 (P5)
- net EXT_R4: now also J26.1 (G1)
- net EXT_R5: now reaches J4.6 (P6)
- net EXT_R5: now also J28.1 (G1)
- net EXT_R6: now reaches J4.7 (P7)
- net EXT_R6: now also J30.1 (G1)
- net EXT_R7: now reaches J4.8 (P8)
- net EXT_R7: now also J32.1 (G1)
- net INT_R0: now reaches M1.r0 (ROW0)
- net INT_R0: now also J17.1 (G1)
- net INT_R1: now reaches M1.r1 (ROW1)
- net INT_R1: now also J19.1 (G1)
- net INT_R2: now reaches M1.r2 (ROW2)
- net INT_R2: now also J21.1 (G1)
- net INT_R3: now reaches M1.r3 (ROW3)
- net INT_R3: now also J23.1 (G1)
- net INT_R4: now reaches M1.r4 (ROW4)
- net INT_R4: now also J25.1 (G1)
- net INT_R5: now reaches M1.r5 (ROW5)
- net INT_R5: now also J27.1 (G1)
- net INT_R6: now reaches M1.r6 (ROW6)
- net INT_R6: now also J29.1 (G1)
- net INT_R7: now reaches M1.r7 (ROW7)
- net INT_R7: now also J31.1 (G1)
Other:
- note added: "BYPASS SOLDER JUMPERS"
- moved on the sheet: J10, J11, J12, J13, J14, J15, J16, J4, J5, J6, J7, J8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
