File: drivers/ND-01/ND-01.kicad_pcb (KiCad board)
At the start: 4 copper layers, 232.4 x 49.5 mm, 76 parts, among them J1 CONN_01X02, J10 CONN_01X08, J11 CONN_01X08, J12 CONN_01X08, J13 CONN_01X08, J14 CONN_01X08, J15 CONN_01X08, J16 CONN_01X08, J17 GS2, J18 GS2, J19 GS2, J2 HIROSE-USB-MICROB, J20 GS2, J21 GS2, J22 GS2, J23 GS2, J24 GS2, J25 GS2, J26 GS2, J27 GS2, J28 GS2, J29 GS2, J3 CONN_01X08, J30 GS2, J31 GS2, J32 GS2, J33 GS2, J34 GS2, J35 GS2, J36 GS2, J37 GS2, J38 GS2, J39 GS2, J4 CONN_01X08, J40 GS3, J41 GS3, J5 CONN_01X08, J6 CONN_01X08, J7 CONN_01X08, J8 CONN_01X08, J9 CONN_01X08, M1 MATRIX, U1 ULN2803A, U10 74HC595, U11 74HC595, U12 74HC595, U13 74HC595, U14 74HC595, U2 4017, U3 74HC595, U4 74HC595, U5 74HC595, U6 74HC595, U7 74HC595, U8 74HC595, U9 74HC595

Commit message: complete initial prototype pcb design
Connections:
- J1 pad 1: GND -> /ND01 power/TEST
- J1 pad 2: /ND01 power/TEST -> GND
Routing:
- net VCC: track 19.5 -> 334.4 mm, vias 0 -> 8
- net /ND01 control/C10: track 81.0 -> 262.5 mm, vias 9 -> 12
- net /ND01 control/C34: track 0.00 -> 156.6 mm, vias 0 -> 5
- net /ND01 control/C11: track 71.9 -> 202.7 mm
- net /ND01 control/C12: track 52.5 -> 174.0 mm
- net /ND01 control/C15: track 74.7 -> 189.3 mm, vias 8 -> 10
- net /ND01 control/C14: track 78.9 -> 187.2 mm, vias 12 -> 13
- net /ND01 control/C35: track 0.00 -> 106.1 mm, vias 0 -> 6
- net /ND01 control/C33: track 0.00 -> 105.3 mm, vias 0 -> 4
- net /ND01 control/C32: track 0.00 -> 99.9 mm, vias 0 -> 3
- net /ND01 control/C37: track 0.00 -> 96.6 mm, vias 0 -> 1
- net /ND01 control/C36: track 0.00 -> 95.5 mm, vias 0 -> 3
- net /ND01 control/C40: track 0.00 -> 92.9 mm, vias 0 -> 2
- net /ND01 control/C39: track 0.00 -> 92.4 mm, vias 0 -> 3
- net /ND01 control/C38: track 0.00 -> 89.5 mm, vias 0 -> 1
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- added copper zone on B.Cu, net GND
- added copper zone on power.plane, net VCC
Other:
- net class Power-interconnect added: clearance 0.2, trace_width 0.2794, via_dia 0.8, via_drill 0.4
