File: drivers/ND-01/ND01 MCU INTERFACE.sch (KiCad schematic (older format))
At the start: 1 part, among them J3 CONN_01X08

Commit message: Add separate driver uses to schematic
Other:
- note added: "CONNECTOR"
- moved on the sheet: J3

Commit message: semicomplete design
Parts:
- J3: footprint (none) -> Connectors_Molex:Molex_KK-6410-08_08x2.54mm_Straight
Connections:
- net COL-DATA: now also J3.4 (P4); no longer J3.3 (P3)
- net COL-RCK: now also J3.6 (P6); no longer J3.5 (P5)
- net COL-SRCLK: now also J3.5 (P5); no longer J3.4 (P4)
- net GND: no longer J3.6 (P6)
- net ROW_CLK: now also J3.3 (P3); no longer J3.2 (P2)
- net ROW_RST: now also J3.2 (P2); no longer J3.1 (P1)
- new net VCC: J3.1 (P1)
Changed lines of the file:
@@
 Comment4 ""
 $EndDescr
-Text HLabel 5700 1000 2    39   Output ~ 0
-ROW_RST
 Text HLabel 5700 1100 2    39   Output ~ 0
-ROW_CLK
+ROW_RST
 Text HLabel 5700 1200 2    39   Output ~ 0
-COL-DATA
+ROW_CLK
 Text HLabel 5700 1300 2    39   Output ~ 0
-COL-SRCLK
+COL-DATA
 Text HLabel 5700 1400 2    39   Output ~ 0
+COL-SRCLK
+Text HLabel 5700 1500 2    39   Output ~ 0
 COL-RCK
 $Comp
@@
 F 0 "J3" H 5428 1391 50  0000 L CNN
 F 1 "CONN_01X08" H 5428 1300 50  0000 L CNN
-F 2 "" H 5350 1350 50  0001 C CNN
+F 2 "Connectors_Molex:Molex_KK-6410-08_08x2.54mm_Straight" H 5350 1350 50  0001 C CNN
 F 3 "" H 5350 1350 50  0001 C CNN
 	1    5350 1350
@@
 $EndComp
 Wire Wire Line
-	5700 1000 5550 1000
-Wire Wire Line
 	5700 1100 5550 1100
 Wire Wire Line
@@
 Wire Wire Line
 	5700 1400 5550 1400
+Wire Wire Line
+	5700 1500 5550 1500
 $Comp
-L GND #PWR5
+L GND #PWR7
 U 1 1 58E79E5E
 P 5700 1800
-F 0 "#PWR5" H 5700 1550 50  0001 C CNN
+F 0 "#PWR7" H 5700 1550 50  0001 C CNN
 F 1 "GND" H 5705 1627 50  0000 C CNN
 F 2 "" H 5700 1800 50  0001 C CNN
@@
 $EndComp
 Wire Wire Line
-	5700 1800 5700 1500
-Wire Wire Line
-	5700 1500 5550 1500
-Wire Wire Line
 	5700 1600 5550 1600
 Connection ~ 5700 1600
@@
 Wire Notes Line
 	650  2250 11200 2250
+Wire Wire Line
+	5700 1800 5700 1600
+Text GLabel 5700 1000 2    39   Input ~ 0
+VCC
+Wire Wire Line
+	5700 1000 5550 1000
 $EndSCHEMATC

Commit message: complete initial prototype pcb design
Changed lines of the file:
@@
 	5700 1500 5550 1500
 $Comp
-L GND #PWR7
+L GND #PWR07
 U 1 1 58E79E5E
 P 5700 1800
-F 0 "#PWR7" H 5700 1550 50  0001 C CNN
+F 0 "#PWR07" H 5700 1550 50  0001 C CNN
 F 1 "GND" H 5705 1627 50  0000 C CNN
 F 2 "" H 5700 1800 50  0001 C CNN
@@
 Wire Wire Line
 	5700 1600 5550 1600
-Connection ~ 5700 1600
 Wire Wire Line
 	5700 1700 5550 1700
