File: drivers/ND-01/ND01 control.sch (KiCad schematic (older format))
At the start: 14 parts

Commit message: complete preliminary ND01 system
Parts:
- gave numbers to parts that had none: 14
Connections:
- net COL_RCK renamed COL-RCK
- net ROW_CLK renamed ROW-CLK
- net ROW_RST renamed ROW-RST
Changed lines of the file:
@@
 $Descr A4 11693 8268
 encoding utf-8
-Sheet 3 3
+Sheet 4 5
 Title ""
 Date ""
@@
 $EndDescr
 $Comp
-L 4017 U?
+L 4017 U2
 U 1 1 58E5FFE3
 P 4800 1350
-F 0 "U?" H 4800 2166 50  0000 C CNN
+F 0 "U2" H 4800 2166 50  0000 C CNN
 F 1 "4017" H 4800 2075 50  0000 C CNN
 F 2 "" H 4800 1350 60  0001 C CNN
@@
 $EndComp
 $Comp
-L ULN2803A U?
+L ULN2803A U1
 U 1 1 58E60148
 P 7250 1200
-F 0 "U?" H 7250 1767 50  0000 C CNN
+F 0 "U1" H 7250 1767 50  0000 C CNN
 F 1 "ULN2803A" H 7250 1676 50  0000 C CNN
 F 2 "" H 7300 550 50  0001 L CNN
@@
 VCC
 $Comp
-L GND #PWR?
+L GND #PWR10
 U 1 1 58E61237
 P 1150 3300
-F 0 "#PWR?" H 1150 3050 50  0001 C CNN
+F 0 "#PWR10" H 1150 3050 50  0001 C CNN
 F 1 "GND" H 1155 3127 50  0000 C CNN
 F 2 "" H 1150 3300 50  0001 C CNN
@@
 $EndComp
 $Comp
-L GND #PWR?
+L GND #PWR6
 U 1 1 58E61370
 P 3750 900
-F 0 "#PWR?" H 3750 650 50  0001 C CNN
+F 0 "#PWR6" H 3750 650 50  0001 C CNN
 F 1 "GND" H 3650 800 50  0000 C CNN
 F 2 "" H 3750 900 50  0001 C CNN
@@
 COL-SRCLK
 Text HLabel 3800 800  0    60   Input ~ 0
-ROW_CLK
+ROW-CLK
 Text HLabel 3800 1100 0    60   Input ~ 0
-ROW_RST
+ROW-RST
 Text HLabel 1100 2600 0    39   Input ~ 0
 COL-DATA
 Text HLabel 1050 3100 0    39   Input ~ 0
-COL_RCK
+COL-RCK
 Text Label 1350 3100 2    39   ~ 0
 RCK
@@
 SRCLK
 $Comp
-L 74HC595 U?
+L 74HC595 U4
 U 1 1 58E62971
 P 4650 3000
-F 0 "U?" H 4650 3766 50  0000 C CNN
+F 0 "U4" H 4650 3766 50  0000 C CNN
 F 1 "74HC595" H 4650 3675 50  0000 C CNN
 F 2 "" H 4650 3000 50  0001 C CNN
@@
 VCC
 $Comp
-L GND #PWR?
+L GND #PWR8
 U 1 1 58E62979
 P 3750 3250
-F 0 "#PWR?" H 3750 3000 50  0001 C CNN
+F 0 "#PWR8" H 3750 3000 50  0001 C CNN
 F 1 "GND" H 3755 3077 50  0000 C CNN
 F 2 "" H 3750 3250 50  0001 C CNN
@@
 C15
 $Comp
-L 74HC595 U?
+L 74HC595 U5
 U 1 1 58E62FF1
 P 7000 3000
-F 0 "U?" H 7000 3766 50  0000 C CNN
+F 0 "U5" H 7000 3766 50  0000 C CNN
 F 1 "74HC595" H 7000 3675 50  0000 C CNN
 F 2 "" H 7000 3000 50  0001 C CNN
@@
 VCC
 $Comp
-L GND #PWR?
+L GND #PWR9
 U 1 1 58E62FF9
 P 6100 3250
-F 0 "#PWR?" H 6100 3000 50  0001 C CNN
+F 0 "#PWR9" H 6100 3000 50  0001 C CNN
 F 1 "GND" H 6105 3077 50  0000 C CNN
 F 2 "" H 6100 3250 50  0001 C CNN
@@
 LINK-2
 $Comp
-L 74HC595 U?
+L 74HC595 U3
 U 1 1 58E634B7
 P 9300 2950
-F 0 "U?" H 9300 3716 50  0000 C CNN
+F 0 "U3" H 9300 3716 50  0000 C CNN
 F 1 "74HC595" H 9300 3625 50  0000 C CNN
 F 2 "" H 9300 2950 50  0001 C CNN
@@
 COL[24:31]
 $Comp
-L 74HC595 U?
+L 74HC595 U7
 U 1 1 58E636AC
 P 2050 4400
-F 0 "U?" H 2050 5100 50  0000 C CNN
+F 0 "U7" H 2050 5100 50  0000 C CNN
 F 1 "74HC595" H 2050 5000 50  0000 C CNN
 F 2 "" H 2050 4400 50  0001 C CNN
@@
 COL[32:39]
 $Comp
-L 74HC595 U?
+L 74HC595 U8
 U 1 1 58E63760
 P 4650 4400
-F 0 "U?" H 4650 5100 50  0000 C CNN
+F 0 "U8" H 4650 5100 50  0000 C CNN
 F 1 "74HC595" H 4650 5000 50  0000 C CNN
 F 2 "" H 4650 4400 50  0001 C CNN
@@
 COL[40:47]
 $Comp
-L 74HC595 U?
+L 74HC595 U9
 U 1 1 58E638B8
 P 7000 4400
-F 0 "U?" H 7000 5100 50  0000 C CNN
+F 0 "U9" H 7000 5100 50  0000 C CNN
 F 1 "74HC595" H 7000 5000 50  0000 C CNN
 F 2 "" H 7000 4400 50  0001 C CNN
@@
 COL[48:55]
 $Comp
-L 74HC595 U?
+L 74HC595 U10
 U 1 1 58E63956
 P 9300 4400
-F 0 "U?" H 9300 5100 50  0000 C CNN
+F 0 "U10" H 9300 5100 50  0000 C CNN
 F 1 "74HC595" H 9300 5000 50  0000 C CNN
 F 2 "" H 9300 4400 50  0001 C CNN
@@
 COL[56:63]
 $Comp
-L 74HC595 U?
+L 74HC595 U6
 U 1 1 58E6101F
 P 2050 3050
-F 0 "U?" H 2050 3816 50  0000 C CNN
+F 0 "U6" H 2050 3816 50  0000 C CNN
 F 1 "74HC595" H 2050 3725 50  0000 C CNN
 F 2 "" H 2050 3050 50  0001 C CNN
@@
 $EndComp
 $Comp
-L 74HC595 U?
+L 74HC595 U11
 U 1 1 58E647FF
 P 2100 5700
-F 0 "U?" H 2100 6400 50  0000 C CNN
+F 0 "U11" H 2100 6400 50  0000 C CNN
 F 1 "74HC595" H 2100 6300 50  0000 C CNN
 F 2 "" H 2100 5700 50  0001 C CNN
@@
 COL[64:71]
 $Comp
-L 74HC595 U?
+L 74HC595 U12
 U 1 1 58E64821
 P 4700 5700
-F 0 "U?" H 4700 6400 50  0000 C CNN
+F 0 "U12" H 4700 6400 50  0000 C CNN
 F 1 "74HC595" H 4700 6300 50  0000 C CNN
 F 2 "" H 4700 5700 50  0001 C CNN
@@
 COL[72:79]
 $Comp
-L 74HC595 U?
+L 74HC595 U13
 U 1 1 58E64843
 P 7050 5700
-F 0 "U?" H 7050 6400 50  0000 C CNN
+F 0 "U13" H 7050 6400 50  0000 C CNN
 F 1 "74HC595" H 7050 6300 50  0000 C CNN
 F 2 "" H 7050 5700 50  0001 C CNN
@@
 COL[80:87]
 $Comp
-L 74HC595 U?
+L 74HC595 U14
 U 1 1 58E64865
 P 9350 5700
-F 0 "U?" H 9350 6400 50  0000 C CNN
+F 0 "U14" H 9350 6400 50  0000 C CNN
 F 1 "74HC595" H 9350 6300 50  0000 C CNN
 F 2 "" H 9350 5700 50  0001 C CNN
@@
 LINK-3
 $Comp
-L GND #PWR?
+L GND #PWR7
 U 1 1 58E6734E
 P 8500 3200
-F 0 "#PWR?" H 8500 2950 50  0001 C CNN
+F 0 "#PWR7" H 8500 2950 50  0001 C CNN
 F 1 "GND" H 8505 3027 50  0000 C CNN
 F 2 "" H 8500 3200 50  0001 C CNN
@@
 LINK-4
 $Comp
-L GND #PWR?
+L GND #PWR13
 U 1 1 58E6AAB3
 P 6100 4600
-F 0 "#PWR?" H 6100 4350 50  0001 C CNN
+F 0 "#PWR13" H 6100 4350 50  0001 C CNN
 F 1 "GND" H 6105 4427 50  0000 C CNN
 F 2 "" H 6100 4600 50  0001 C CNN
@@
 $EndComp
 $Comp
-L GND #PWR?
+L GND #PWR12
 U 1 1 58E6ABE4
 P 3750 4600
-F 0 "#PWR?" H 3750 4350 50  0001 C CNN
+F 0 "#PWR12" H 3750 4350 50  0001 C CNN
 F 1 "GND" H 3755 4427 50  0000 C CNN
 F 2 "" H 3750 4600 50  0001 C CNN
@@
 $EndComp
 $Comp
-L GND #PWR?
+L GND #PWR11
 U 1 1 58E6AC51
 P 1200 4600
-F 0 "#PWR?" H 1200 4350 50  0001 C CNN
+F 0 "#PWR11" H 1200 4350 50  0001 C CNN
 F 1 "GND" H 1205 4427 50  0000 C CNN
 F 2 "" H 1200 4600 50  0001 C CNN
@@
 $EndComp
 $Comp
-L GND #PWR?
+L GND #PWR14
 U 1 1 58E6ADD6
 P 8450 4600
-F 0 "#PWR?" H 8450 4350 50  0001 C CNN
+F 0 "#PWR14" H 8450 4350 50  0001 C CNN
 F 1 "GND" H 8455 4427 50  0000 C CNN
 F 2 "" H 8450 4600 50  0001 C CNN
@@
 $EndComp
 $Comp
-L GND #PWR?
+L GND #PWR15
 U 1 1 58E6B505
 P 1200 5900
-F 0 "#PWR?" H 1200 5650 50  0001 C CNN
+F 0 "#PWR15" H 1200 5650 50  0001 C CNN
 F 1 "GND" H 1205 5727 50  0000 C CNN
 F 2 "" H 1200 5900 50  0001 C CNN
@@
 $EndComp
 $Comp
-L GND #PWR?
+L GND #PWR16
 U 1 1 58E6B75E
 P 3750 5900
-F 0 "#PWR?" H 3750 5650 50  0001 C CNN
+F 0 "#PWR16" H 3750 5650 50  0001 C CNN
 F 1 "GND" H 3755 5727 50  0000 C CNN
 F 2 "" H 3750 5900 50  0001 C CNN
@@
 $EndComp
 $Comp
-L GND #PWR?
+L GND #PWR17
 U 1 1 58E6BB5E
 P 6100 5900
-F 0 "#PWR?" H 6100 5650 50  0001 C CNN
+F 0 "#PWR17" H 6100 5650 50  0001 C CNN
 F 1 "GND" H 6105 5727 50  0000 C CNN
 F 2 "" H 6100 5900 50  0001 C CNN
@@
 $EndComp
 $Comp
-L GND #PWR?
+L GND #PWR18
 U 1 1 58E6BE20
 P 8350 5900
-F 0 "#PWR?" H 8350 5650 50  0001 C CNN
+F 0 "#PWR18" H 8350 5650 50  0001 C CNN
 F 1 "GND" H 8355 5727 50  0000 C CNN
 F 2 "" H 8350 5900 50  0001 C CNN

Commit message: semicomplete design
Parts:
- added C10, C11, C12, C13, C14, C15, C16, C17, C4, C5, C6, C7, C8, C9: C, Capacitors_THT:C_Disc_D3.4mm_W2.1mm_P2.50mm, symbol C
- added J33, J34, J35, J36, J37, J38, J39: GS2, Connectors:GS2, symbol GS2
- added J40: GS3, Connectors:GS3, symbol GS3
- U1: footprint (none) -> Housings_DIP:DIP-18_W7.62mm_LongPads
- U10, U11, U12, U13, U14, U2, U3, U4, U5, U6, U7, U8, U9: footprint (none) -> Housings_DIP:DIP-16_W7.62mm_LongPads
Connections:
- net VDD is gone; now on net VCC: U2.16 (VDD)
- net GND: now also C10.2, C11.2, C12.2, C13.2, C14.2, C15.2, C16.2, C17.2, C4.2, C5.2, C6.2, C7.2, C8.2, C9.2
- net Q0: now also J40.1 (G1); no longer U1.1 (I1)
- net Q1: now also J39.2 (G2); no longer U1.2 (I2)
- net Q2: now also J38.2 (G2); no longer U1.3 (I3)
- net Q3: now also J37.2 (G2); no longer U1.4 (I4)
- net Q4: now also J36.2 (G2); no longer U1.5 (I5)
- net Q5: now also J35.2 (G2); no longer U1.6 (I6)
- net Q6: now also J34.2 (G2); no longer U1.7 (I7)
- net Q7: now also J33.2 (G2); no longer U1.8 (I8)
- net VCC: now also C10.1, C11.1, C12.1, C13.1, C14.1, C15.1, C16.1, C17.1, C4.1, C5.1, C6.1, C7.1, C8.1, C9.1
- net Q8: now reaches U2.9 (Q8)
- net Q8: now also J40.3 (G3)
- net GNDA: now reaches U1.9 (GND)
- new net: J33.1 (G1), U1.1 (I1)
- new net: J34.1 (G1), U1.2 (I2)
- new net: J35.1 (G1), U1.3 (I3)
- new net: J36.1 (G1), U1.4 (I4)
- new net: J37.1 (G1), U1.5 (I5)
- new net: J38.1 (G1), U1.6 (I6)
- new net: J39.1 (G1), U1.7 (I7)
- new net: J40.2 (G2), U1.8 (I8)
- no-connect marks 3 -> 2
Other:
- note added: "DECOUPLING CAPACITORS"
- moved on the sheet: U1
