File: drivers/ND-01/ND01 power.sch (KiCad schematic (older format))
At the start: 6 parts

Commit message: complete preliminary ND01 system
Parts:
- gave numbers to parts that had none: 6
Changed lines of the file:
@@
 $Descr A4 11693 8268
 encoding utf-8
-Sheet 2 3
+Sheet 2 5
 Title ""
 Date ""
@@
 $EndDescr
 $Comp
-L HIROSE-USB-MICROB J?
+L HIROSE-USB-MICROB J2
 U 1 1 58E5E79F
 P 2100 4800
-F 0 "J?" H 2100 5397 60  0000 C CNN
+F 0 "J2" H 2100 5397 60  0000 C CNN
 F 1 "HIROSE-USB-MICROB" H 2100 5291 60  0000 C CNN
 F 2 "" H 2100 4800 60  0001 C CNN
@@
 $EndComp
 $Comp
-L GND #PWR?
+L GND #PWR4
 U 1 1 58E5EAD0
 P 2550 5400
-F 0 "#PWR?" H 2550 5150 50  0001 C CNN
+F 0 "#PWR4" H 2550 5150 50  0001 C CNN
 F 1 "GND" H 2555 5227 50  0000 C CNN
 F 2 "" H 2550 5400 50  0001 C CNN
@@
 GND
 $Comp
-L CONN_01X02 J?
+L CONN_01X02 J1
 U 1 1 58E5ED61
 P 2000 3450
-F 0 "J?" H 1919 3175 50  0000 C CNN
+F 0 "J1" H 1919 3175 50  0000 C CNN
 F 1 "CONN_01X02" H 1919 3266 50  0000 C CNN
 F 2 "" H 2000 3450 50  0001 C CNN
@@
 5V
 $Comp
-L D_Zener D?
+L D_Zener D1
 U 1 1 58E5F2D5
 P 5300 4400
-F 0 "D?" V 5250 4150 50  0000 L CNN
+F 0 "D1" V 5250 4150 50  0000 L CNN
 F 1 "D_Zener" V 5350 4000 50  0000 L CNN
 F 2 "" H 5300 4400 50  0001 C CNN
@@
 $EndComp
 $Comp
-L CP1 C?
+L CP1 C1
 U 1 1 58E5F3F0
 P 5750 4400
-F 0 "C?" H 5865 4446 50  0000 L CNN
+F 0 "C1" H 5865 4446 50  0000 L CNN
 F 1 "CP1" H 5865 4355 50  0000 L CNN
 F 2 "" H 5750 4400 50  0001 C CNN
@@
 $EndComp
 $Comp
-L GND #PWR?
+L GND #PWR2
 U 1 1 58E5F47E
 P 5750 4850
-F 0 "#PWR?" H 5750 4600 50  0001 C CNN
+F 0 "#PWR2" H 5750 4600 50  0001 C CNN
 F 1 "GND" H 5755 4677 50  0000 C CNN
 F 2 "" H 5750 4850 50  0001 C CNN
@@
 $EndComp
 $Comp
-L R R?
+L R R1
 U 1 1 58E5F57B
 P 6200 4300
-F 0 "R?" H 6270 4346 50  0000 L CNN
+F 0 "R1" H 6270 4346 50  0000 L CNN
 F 1 "R" H 6270 4255 50  0000 L CNN
 F 2 "" V 6130 4300 50  0001 C CNN
@@
 $EndComp
 $Comp
-L LED D?
+L LED D2
 U 1 1 58E5F5EF
 P 6200 4600
-F 0 "D?" V 6238 4483 50  0000 R CNN
+F 0 "D2" V 6238 4483 50  0000 R CNN
 F 1 "LED" V 6147 4483 50  0000 R CNN
 F 2 "" H 6200 4600 50  0001 C CNN
@@
 $EndComp
 $Comp
-L GND #PWR?
+L GND #PWR3
 U 1 1 58E5F794
 P 6200 4850
-F 0 "#PWR?" H 6200 4600 50  0001 C CNN
+F 0 "#PWR3" H 6200 4600 50  0001 C CNN
 F 1 "GND" H 6205 4677 50  0000 C CNN
 F 2 "" H 6200 4850 50  0001 C CNN
@@
 $EndComp
 $Comp
-L GND #PWR?
+L GND #PWR1
 U 1 1 58E5F7E1
 P 5300 4850
-F 0 "#PWR?" H 5300 4600 50  0001 C CNN
+F 0 "#PWR1" H 5300 4600 50  0001 C CNN
 F 1 "GND" H 5305 4677 50  0000 C CNN
 F 2 "" H 5300 4850 50  0001 C CNN

Commit message: Add separate driver uses to schematic
Other:
- moved on the sheet: C1, D1, D2, J1, J2, R1

Commit message: semicomplete design
Parts:
- added C1: 1000uF, Capacitors_THT:CP_Radial_D5.0mm_P2.50mm, symbol CP1
- added C2: 0.1uF, Capacitors_THT:CP_Radial_D5.0mm_P2.50mm, symbol CP1
- added J41: GS3, Connectors:GS3, symbol GS3
- C3: renamed from C1; value CP1 -> 10uF; footprint (none) -> Capacitors_THT:CP_Radial_D5.0mm_P2.50mm
- D1: footprint (none) -> Diodes_THT:D_A-405_P10.16mm_Horizontal
- D2: footprint (none) -> LEDs:LED_D5.0mm
- J1: footprint (none) -> Connectors:Banana_Jack_2Pin
- J2: footprint (none) -> pochi:Hirose_ZX62D_B_5PA830
- R1: footprint (none) -> Resistors_THT:R_Axial_DIN0309_L9.0mm_D3.2mm_P12.70mm_Horizontal
Connections:
- net GND: now also C1.2, C2.2
- net VCC: now also C1.1, C2.1, J41.2 (G2); no longer J1.2 (P2), J2.1 (VBUS)
- new net 5V: J2.1 (VBUS), J41.3 (G3)
- new net TEST: J1.2 (P2), J41.1 (G1)
Other:
- note added: "POWER SELECTOR"
- moved on the sheet: C3, D1, D2, R1
Changed lines of the file:
@@
 F 0 "J2" H 1450 3297 60  0000 C CNN
 F 1 "HIROSE-USB-MICROB" H 1450 3191 60  0000 C CNN
-F 2 "" H 1450 2700 60  0001 C CNN
+F 2 "pochi:Hirose_ZX62D_B_5PA830" H 1450 2700 60  0001 C CNN
 F 3 "" H 1450 2700 60  0001 C CNN
 	1    1450 2700
@@
 $EndComp
 $Comp
-L GND #PWR4
+L GND #PWR6
 U 1 1 58E5EAD0
 P 1900 3300
-F 0 "#PWR4" H 1900 3050 50  0001 C CNN
+F 0 "#PWR6" H 1900 3050 50  0001 C CNN
 F 1 "GND" H 1905 3127 50  0000 C CNN
 F 2 "" H 1900 3300 50  0001 C CNN
@@
 F 0 "J1" H 1319 1075 50  0000 C CNN
 F 1 "CONN_01X02" H 1319 1166 50  0000 C CNN
-F 2 "" H 1400 1350 50  0001 C CNN
+F 2 "Connectors:Banana_Jack_2Pin" H 1400 1350 50  0001 C CNN
 F 3 "" H 1400 1350 50  0001 C CNN
 	1    1400 1350
@@
 GND
 Text Label 1700 1300 0    39   ~ 0
-5V
+TEST
 Text Notes 1900 600  0    60   ~ 0
 TEST POWER INPUT
@@
 L D_Zener D1
 U 1 1 58E5F2D5
-P 6350 2000
-F 0 "D1" V 6300 1750 50  0000 L CNN
-F 1 "D_Zener" V 6400 1600 50  0000 L CNN
-F 2 "" H 6350 2000 50  0001 C CNN
-F 3 "" H 6350 2000 50  0001 C CNN
-	1    6350 2000
+P 7950 1900
+F 0 "D1" V 7900 1650 50  0000 L CNN
+F 1 "D_Zener" V 8000 1500 50  0000 L CNN
+F 2 "Diodes_THT:D_A-405_P10.16mm_Horizontal" H 7950 1900 50  0001 C CNN
+F 3 "" H 7950 1900 50  0001 C CNN
+	1    7950 1900
 	0    1    1    0
 $EndComp
 $Comp
-L CP1 C1
+L CP1 C3
 U 1 1 58E5F3F0
-P 6800 2000
-F 0 "C1" H 6915 2046 50  0000 L CNN
-F 1 "CP1" H 6915 1955 50  0000 L CNN
-F 2 "" H 6800 2000 50  0001 C CNN
-F 3 "" H 6800 2000 50  0001 C CNN
-	1    6800 2000
+P 9150 1900
+F 0 "C3" H 9265 1946 50  0000 L CNN
+F 1 "10uF" H 9200 1750 50  0000 L CNN
+F 2 "Capacitors_THT:CP_Radial_D5.0mm_P2.50mm" H 9150 1900 50  0001 C CNN
+F 3 "" H 9150 1900 50  0001 C CNN
+	1    9150 1900
 	1    0    0    -1
 $EndComp
 $Comp
-L GND #PWR2
+L GND #PWR4
 U 1 1 58E5F47E
-P 6800 2450
-F 0 "#PWR2" H 6800 2200 50  0001 C CNN
-F 1 "GND" H 6805 2277 50  0000 C CNN
-F 2 "" H 6800 2450 50  0001 C CNN
-F 3 "" H 6800 2450 50  0001 C CNN
-	1    6800 2450
+P 9150 2350
+F 0 "#PWR4" H 9150 2100 50  0001 C CNN
+F 1 "GND" H 9155 2177 50  0000 C CNN
+F 2 "" H 9150 2350 50  0001 C CNN
+F 3 "" H 9150 2350 50  0001 C CNN
+	1    9150 2350
 	1    0    0    -1
 $EndComp
@@
 L R R1
 U 1 1 58E5F57B
-P 7250 1900
-F 0 "R1" H 7320 1946 50  0000 L CNN
-F 1 "R" H 7320 1855 50  0000 L CNN
-F 2 "" V 7180 1900 50  0001 C CNN
-F 3 "" H 7250 1900 50  0001 C CNN
-	1    7250 1900
+P 9600 1800
+F 0 "R1" H 9670 1846 50  0000 L CNN
+F 1 "R" H 9670 1755 50  0000 L CNN
+F 2 "Resistors_THT:R_Axial_DIN0309_L9.0mm_D3.2mm_P12.70mm_Horizontal" V 9530 1800 50  0001 C CNN
+F 3 "" H 9600 1800 50  0001 C CNN
+	1    9600 1800
 	1    0    0    -1
 $EndComp
@@
 L LED D2
 U 1 1 58E5F5EF
-P 7250 2200
-F 0 "D2" V 7288 2083 50  0000 R CNN
-F 1 "LED" V 7197 2083 50  0000 R CNN
-F 2 "" H 7250 2200 50  0001 C CNN
-F 3 "" H 7250 2200 50  0001 C CNN
-	1    7250 2200
+P 9600 2100
+F 0 "D2" V 9638 1983 50  0000 R CNN
+F 1 "LED" V 9547 1983 50  0000 R CNN
+F 2 "LEDs:LED_D5.0mm" H 9600 2100 50  0001 C CNN
+F 3 "" H 9600 2100 50  0001 C CNN
+	1    9600 2100
 	0    -1   -1   0
 $EndComp
 $Comp
-L GND #PWR3
+L GND #PWR5
 U 1 1 58E5F794
-P 7250 2450
-F 0 "#PWR3" H 7250 2200 50  0001 C CNN
-F 1 "GND" H 7255 2277 50  0000 C CNN
-F 2 "" H 7250 2450 50  0001 C CNN
-F 3 "" H 7250 2450 50  0001 C CNN
-	1    7250 2450
+P 9600 2350
+F 0 "#PWR5" H 9600 2100 50  0001 C CNN
+F 1 "GND" H 9605 2177 50  0000 C CNN
+F 2 "" H 9600 2350 50  0001 C CNN
+F 3 "" H 9600 2350 50  0001 C CNN
+	1    9600 2350
 	1    0    0    -1
 $EndComp
@@
 L GND #PWR1
 U 1 1 58E5F7E1
-P 6350 2450
-F 0 "#PWR1" H 6350 2200 50  0001 C CNN
-F 1 "GND" H 6355 2277 50  0000 C CNN
-F 2 "" H 6350 2450 50  0001 C CNN
-F 3 "" H 6350 2450 50  0001 C CNN
-	1    6350 2450
+P 7950 2350
+F 0 "#PWR1" H 7950 2100 50  0001 C CNN
+F 1 "GND" H 7955 2177 50  0000 C CNN
+F 2 "" H 7950 2350 50  0001 C CNN
+F 3 "" H 7950 2350 50  0001 C CNN
+	1    7950 2350
 	1    0    0    -1
 $EndComp
-Text GLabel 7850 1600 2    39   Output ~ 0
+Text GLabel 10200 1500 2    39   Output ~ 0
 VCC
 Text Notes 11200 600  2    60   ~ 0
 POWER CONDITIONING
-Wire Wire Line
-	900  2700 1050 2700
-Wire Wire Line
-	1850 3100 1900 3100
-Wire Wire Line
-	1900 3100 1900 3300
-Wire Wire Line
-	1850 2350 1950 2350
-Wire Wire Line
-	1600 1400 1700 1400
-Wire Wire Line
-	1600 1300 1700 1300
-Wire Wire Line
-	6350 1600 6350 1850
-Wire Wire Line
-	6800 1600 6800 1850
-Connection ~ 6350 1600
-Wire Wire Line
-	6350 2150 6350 2450
-Wire Wire Line
-	6800 2150 6800 2450
-Wire Wire Line
-	7250 1600 7250 1750
-Connection ~ 6800 1600
-Wire Wire Line
-	7250 2450 7250 2350
-Connection ~ 7250 1600
-Wire Wire Line
-	5950 1600 7850 1600
-Text Label 5950 1600 2    39   ~ 0
-5V
+Text Label 7600 1500 2    39   ~ 0
+VCC_SEL
 $Bitmap
 Pos 10250 6800
@@
 EndData
 $EndBitmap
+$Comp
+L CP1 C2
+U 1 1 58F30929
+P 8750 1900
+F 0 "C2" H 8865 1946 50  0000 L CNN
+F 1 "0.1uF" H 8800 1750 50  0000 L CNN
+F 2 "Capacitors_THT:CP_Radial_D5.0mm_P2.50mm" H 8750 1900 50  0001 C CNN
+F 3 "" H 8750 1900 50  0001 C CNN
+	1    8750 1900
+	1    0    0    -1
+$EndComp
+$Comp
+L GND #PWR3
+U 1 1 58F3092F
+P 8750 2350
+F 0 "#PWR3" H 8750 2100 50  0001 C CNN
+F 1 "GND" H 8755 2177 50  0000 C CNN
+F 2 "" H 8750 2350 50  0001 C CNN
+F 3 "" H 8750 2350 50  0001 C CNN
+	1    8750 2350
+	1    0    0    -1
+$EndComp
+$Comp
+L CP1 C1
+U 1 1 58F30A1C
+P 8350 1900
+F 0 "C1" H 8465 1946 50  0000 L CNN
+F 1 "1000uF" H 8400 1750 50  0000 L CNN
+F 2 "Capacitors_THT:CP_Radial_D5.0mm_P2.50mm" H 8350 1900 50  0001 C CNN
+F 3 "" H 8350 1900 50  0001 C CNN
+	1    8350 1900
+	1    0    0    -1
+$EndComp
+$Comp
+L GND #PWR2
+U 1 1 58F30A22
+P 8350 2350
+F 0 "#PWR2" H 8350 2100 50  0001 C CNN
+F 1 "GND" H 8355 2177 50  0000 C CNN
+F 2 "" H 8350 2350 50  0001 C CNN
+F 3 "" H 8350 2350 50  0001 C CNN
+	1    8350 2350
+	1    0    0    -1
+$EndComp
+Wire Wire Line
+	900  2700 1050 2700
+Wire Wire Line
+	1850 3100 1900 3100
+Wire Wire Line
+	1900 3100 1900 3300
+Wire Wire Line
+	1850 2350 1950 2350
+Wire Wire Line
+	1600 1400 1700 1400
+Wire Wire Line
+	1600 1300 1700 1300
+Wire Wire Line
+	7950 1500 7950 1750
+Wire Wire Line
+	9150 1500 9150 1750
+Wire Wire Line
+	7950 2050 7950 2350
+Wire Wire Line
+	9150 2050 9150 2350
+Wire Wire Line
+	9600 1500 9600 1650
+Connection ~ 9150 1500
+Wire Wire Line
+	9600 2350 9600 2250
+Connection ~ 9600 1500
+Wire Wire Line
+	7600 1500 10200 1500
 Wire Notes Line
 	500  1850 2800 1850
@@
 Wire Notes Line
 	500  3600 11200 3600
+Wire Wire Line
+	8750 1500 8750 1750
+Wire Wire Line
+	8750 2050 8750 2350
+Connection ~ 8750 1500
+Wire Wire Line
+	8350 1500 8350 1750
+Wire Wire Line
+	8350 2050 8350 2350
+Connection ~ 8350 1500
+Connection ~ 7950 1500
+Wire Wire Line
+	4450 1850 4750 1850
+Wire Wire Line
+	3900 1750 4150 1750
+Wire Wire Line
+	3900 1950 4150 1950
+Wire Notes Line
+	6200 500  6200 3600
+Text Label 4750 1850 0    39   ~ 0
+VCC_SEL
+Text Label 3900 1750 2    39   ~ 0
+TEST
+Text Label 3900 1950 2    39   ~ 0
+5V
+Text Notes 6150 650  2    60   ~ 0
+POWER SELECTOR
+$Comp
+L GS3 J41
+U 1 1 58FBB40E
+P 4300 1850
+F 0 "J41" H 4300 2155 50  0000 C CNN
+F 1 "GS3" H 4300 2064 50  0000 C CNN
+F 2 "Connectors:GS3" V 4388 1776 50  0001 C CNN
+F 3 "" H 4300 1850 50  0001 C CNN
+	1    4300 1850
+	1    0    0    -1
+$EndComp
 $EndSCHEMATC

Commit message: complete initial prototype pcb design
Connections:
- net GND: now also J1.2 (P2); no longer J1.1 (P1)
- net TEST: now also J1.1 (P1); no longer J1.2 (P2)
Changed lines of the file:
@@
 $EndComp
 $Comp
-L GND #PWR6
+L GND #PWR01
 U 1 1 58E5EAD0
 P 1900 3300
-F 0 "#PWR6" H 1900 3050 50  0001 C CNN
+F 0 "#PWR01" H 1900 3050 50  0001 C CNN
 F 1 "GND" H 1905 3127 50  0000 C CNN
 F 2 "" H 1900 3300 50  0001 C CNN
@@
 F 3 "" H 1400 1350 50  0001 C CNN
 	1    1400 1350
-	-1   0    0    1
+	-1   0    0    -1
 $EndComp
-Text Label 1700 1400 0    39   ~ 0
-GND
-Text Label 1700 1300 0    39   ~ 0
-TEST
 Text Notes 1900 600  0    60   ~ 0
 TEST POWER INPUT
@@
 $EndComp
 $Comp
-L GND #PWR4
+L GND #PWR02
 U 1 1 58E5F47E
 P 9150 2350
-F 0 "#PWR4" H 9150 2100 50  0001 C CNN
+F 0 "#PWR02" H 9150 2100 50  0001 C CNN
 F 1 "GND" H 9155 2177 50  0000 C CNN
 F 2 "" H 9150 2350 50  0001 C CNN
@@
 $EndComp
 $Comp
-L GND #PWR5
+L GND #PWR03
 U 1 1 58E5F794
 P 9600 2350
-F 0 "#PWR5" H 9600 2100 50  0001 C CNN
+F 0 "#PWR03" H 9600 2100 50  0001 C CNN
 F 1 "GND" H 9605 2177 50  0000 C CNN
 F 2 "" H 9600 2350 50  0001 C CNN
@@
 $EndComp
 $Comp
-L GND #PWR1
+L GND #PWR04
 U 1 1 58E5F7E1
 P 7950 2350
-F 0 "#PWR1" H 7950 2100 50  0001 C CNN
+F 0 "#PWR04" H 7950 2100 50  0001 C CNN
 F 1 "GND" H 7955 2177 50  0000 C CNN
 F 2 "" H 7950 2350 50  0001 C CNN
@@
 $EndComp
 $Comp
-L GND #PWR3
+L GND #PWR05
 U 1 1 58F3092F
 P 8750 2350
-F 0 "#PWR3" H 8750 2100 50  0001 C CNN
+F 0 "#PWR05" H 8750 2100 50  0001 C CNN
 F 1 "GND" H 8755 2177 50  0000 C CNN
 F 2 "" H 8750 2350 50  0001 C CNN
@@
 $EndComp
 $Comp
-L GND #PWR2
+L GND #PWR06
 U 1 1 58F30A22
 P 8350 2350
-F 0 "#PWR2" H 8350 2100 50  0001 C CNN
+F 0 "#PWR06" H 8350 2100 50  0001 C CNN
 F 1 "GND" H 8355 2177 50  0000 C CNN
 F 2 "" H 8350 2350 50  0001 C CNN
@@
 	1    0    0    -1
 $EndComp
+Text Label 1700 1300 0    39   ~ 0
+TEST
+Text Label 1700 1400 0    39   ~ 0
+GND
 $EndSCHEMATC
