File: hardware/Bitsoko-ESP32-module/ESP32-MODULE.sch (KiCad schematic (older format))
At the start: 7 parts

Commit message: Semicomplete Bitsoko ESP32 module
Parts:
- removed C?: C, symbol C
- added C6: 0.1uF, Capacitors_SMD:C_0805_HandSoldering, symbol C
- added R4: 5k, Resistors_SMD:R_0805_HandSoldering, symbol R
- C3, C4: renamed from C?; value C -> 1nF; footprint (none) -> Capacitors_SMD:C_0805_HandSoldering
- C5: renamed from C?; value C -> 10uF; footprint (none) -> Capacitors_SMD:C_0805_HandSoldering
- R2, R3: renamed from R?; value R -> 12k; footprint (none) -> Resistors_SMD:R_0805_HandSoldering
- gave numbers to parts that had none: 1
Connections:
- net VDD_33 is gone; now on net 3v3: R2.1, R3.1
- net 3v3: now also C5.1, C6.1
- net GND: now also C6.2, R4.2
- net IO2: now also R4.1
- net IO23: no longer U2.32 (GPIO20)
- no-connect marks 0 -> 1
Other:
- note added: "Boot mode control IO0\n1 Normal SPI flash boot control after reset\n2. Download boot after reset"
- note added: "Boot mode control IO2:\n0 on download boot\nDont care(X) on SPI boot"
- note added: "Reset control EN.\n0 - Reset state\n1 - Normal operation"
- moved on the sheet: C3, C4, C5, R2, R3
