File: hardware/Bitsoko-ESP32-module/power_supply.sch (KiCad schematic (older format))
At the start: 3 parts

Commit message: Semicomplete Bitsoko ESP32 module
Parts:
- added D1: LED, LEDs:LED_0805, symbol LED
- added R1: 1k, Resistors_SMD:R_0805_HandSoldering, symbol R
- C1: renamed from C?; footprint (none) -> Capacitors_SMD:C_0805_HandSoldering
- C2: renamed from C?; value 22uF -> 10uF; footprint (none) -> Capacitors_SMD:C_0805_HandSoldering
- gave numbers to parts that had none: 1
Connections:
- net EXT_5V: now also D1.2 (A)
- net GND: now also R1.2
- new net: D1.1 (K), R1.1
Changed lines of the file:
@@
 $EndDescr
 $Comp
-L NCP1117-3.3_SOT223 U?
+L NCP1117-3.3_SOT223 U1
 U 1 1 59513A80
 P 5665 3015
-F 0 "U?" H 5665 3257 50  0000 C CNN
+AR Path="/59510B2B/59513A80" Ref="U1"  Part="1"
+AR Path="/59531D77/59540E02/59513A80" Ref="U1"  Part="1"
+AR Path="/5955264F/59513A80" Ref="U1"  Part="1"
+F 0 "U1" H 5665 3257 50  0000 C CNN
 F 1 "NCP1117-3.3_SOT223" H 5665 3166 50  0000 C CNN
 F 2 "TO_SOT_Packages_SMD:SOT-223" H 5665 3215 50  0001 C CNN
@@
 $EndComp
 $Comp
-L GND #PWR?
+L GND #PWR01
 U 1 1 59513C5C
 P 5665 3765
-F 0 "#PWR?" H 5665 3515 50  0001 C CNN
+AR Path="/59510B2B/59513C5C" Ref="#PWR01"  Part="1"
+AR Path="/59531D77/59540E02/59513C5C" Ref="#PWR01"  Part="1"
+AR Path="/5955264F/59513C5C" Ref="#PWR01"  Part="1"
+F 0 "#PWR01" H 5665 3515 50  0001 C CNN
 F 1 "GND" H 5670 3592 50  0000 C CNN
 F 2 "" H 5665 3765 50  0001 C CNN
@@
 $EndComp
 $Comp
-L C C?
+L C C1
 U 1 1 59513D7D
 P 4665 3365
-F 0 "C?" H 4780 3411 50  0000 L CNN
+AR Path="/59510B2B/59513D7D" Ref="C1"  Part="1"
+AR Path="/59531D77/59540E02/59513D7D" Ref="C1"  Part="1"
+AR Path="/5955264F/59513D7D" Ref="C1"  Part="1"
+F 0 "C1" H 4780 3411 50  0000 L CNN
 F 1 "10uF" H 4780 3320 50  0000 L CNN
-F 2 "" H 4703 3215 50  0001 C CNN
+F 2 "Capacitors_SMD:C_0805_HandSoldering" H 4703 3215 50  0001 C CNN
 F 3 "" H 4665 3365 50  0001 C CNN
 	1    4665 3365
@@
 $EndComp
 $Comp
-L GND #PWR?
+L GND #PWR02
 U 1 1 59513DB7
 P 4665 3765
-F 0 "#PWR?" H 4665 3515 50  0001 C CNN
+AR Path="/59510B2B/59513DB7" Ref="#PWR02"  Part="1"
+AR Path="/59531D77/59540E02/59513DB7" Ref="#PWR02"  Part="1"
+AR Path="/5955264F/59513DB7" Ref="#PWR02"  Part="1"
+F 0 "#PWR02" H 4665 3515 50  0001 C CNN
 F 1 "GND" H 4670 3592 50  0000 C CNN
 F 2 "" H 4665 3765 50  0001 C CNN
@@
 $EndComp
 $Comp
-L GND #PWR?
+L GND #PWR03
 U 1 1 59513EDC
 P 6765 3765
-F 0 "#PWR?" H 6765 3515 50  0001 C CNN
+AR Path="/59510B2B/59513EDC" Ref="#PWR03"  Part="1"
+AR Path="/59531D77/59540E02/59513EDC" Ref="#PWR03"  Part="1"
+AR Path="/5955264F/59513EDC" Ref="#PWR03"  Part="1"
+F 0 "#PWR03" H 6765 3515 50  0001 C CNN
 F 1 "GND" H 6770 3592 50  0000 C CNN
 F 2 "" H 6765 3765 50  0001 C CNN
@@
 	6765 3765 6765 3515
 $Comp
-L C C?
+L C C2
 U 1 1 59513E27
 P 6765 3365
-F 0 "C?" H 6880 3411 50  0000 L CNN
-F 1 "22uF" H 6880 3320 50  0000 L CNN
-F 2 "" H 6803 3215 50  0001 C CNN
+AR Path="/59510B2B/59513E27" Ref="C2"  Part="1"
+AR Path="/59531D77/59540E02/59513E27" Ref="C2"  Part="1"
+AR Path="/5955264F/59513E27" Ref="C2"  Part="1"
+F 0 "C2" H 6880 3411 50  0000 L CNN
+F 1 "10uF" H 6880 3320 50  0000 L CNN
+F 2 "Capacitors_SMD:C_0805_HandSoldering" H 6803 3215 50  0001 C CNN
 F 3 "" H 6765 3365 50  0001 C CNN
 	1    6765 3365
@@
 	6765 3215 6765 3015
 Wire Wire Line
-	5965 3015 7015 3015
+	5965 3015 7615 3015
 Connection ~ 6765 3015
 Connection ~ 4665 3015
@@
 Text HLabel 4465 3015 0    60   Input ~ 0
 EXT_5V
-Text GLabel 7015 3015 2    60   Input ~ 0
+Text GLabel 7615 3015 2    60   Input ~ 0
 3v3
 Text Notes 10280 4330 0    60   ~ 0
 3v3 Linear regulator
+$Comp
+L R R1
+U 1 1 5955D47B
+P 5100 3650
+AR Path="/59510B2B/5955D47B" Ref="R1"  Part="1"
+AR Path="/59531D77/59540E02/5955D47B" Ref="R1"  Part="1"
+AR Path="/5955264F/5955D47B" Ref="R1"  Part="1"
+F 0 "R1" H 5170 3696 50  0000 L CNN
+F 1 "1k" H 5170 3605 50  0000 L CNN
+F 2 "Resistors_SMD:R_0805_HandSoldering" V 5030 3650 50  0001 C CNN
+F 3 "" H 5100 3650 50  0001 C CNN
+	1    5100 3650
+	1    0    0    -1
+$EndComp
+$Comp
+L LED D1
+U 1 1 5955D529
+P 5100 3300
+AR Path="/59510B2B/5955D529" Ref="D1"  Part="1"
+AR Path="/59531D77/59540E02/5955D529" Ref="D1"  Part="1"
+AR Path="/5955264F/5955D529" Ref="D1"  Part="1"
+F 0 "D1" V 5138 3183 50  0000 R CNN
+F 1 "LED" V 5047 3183 50  0000 R CNN
+F 2 "LEDs:LED_0805" H 5100 3300 50  0001 C CNN
+F 3 "" H 5100 3300 50  0001 C CNN
+	1    5100 3300
+	0    -1   -1   0
+$EndComp
+Wire Wire Line
+	5100 3450 5100 3500
+$Comp
+L GND #PWR04
+U 1 1 5955D5CA
+P 5100 3800
+AR Path="/59510B2B/5955D5CA" Ref="#PWR04"  Part="1"
+AR Path="/59531D77/59540E02/5955D5CA" Ref="#PWR04"  Part="1"
+AR Path="/5955264F/5955D5CA" Ref="#PWR04"  Part="1"
+F 0 "#PWR04" H 5100 3550 50  0001 C CNN
+F 1 "GND" H 5105 3627 50  0000 C CNN
+F 2 "" H 5100 3800 50  0001 C CNN
+F 3 "" H 5100 3800 50  0001 C CNN
+	1    5100 3800
+	1    0    0    -1
+$EndComp
+Wire Wire Line
+	5100 3150 5100 3015
+Connection ~ 5100 3015
 $EndSCHEMATC
