File: hardware/Bitsoko-ESP32-module/Connector_A.sch (KiCad schematic (older format))
At the start: 1 part

Commit message: Semicomplete Bitsoko ESP32 module
Parts:
- J2: renamed from J?; footprint (none) -> Pin_Headers:Pin_Header_Straight_1x20_Pitch2.54mm
Changed lines of the file:
@@
 $EndDescr
 $Comp
-L CONN_01X20 J?
+L CONN_01X20 J2
 U 1 1 59513823
 P 5650 3700
-F 0 "J?" V 5728 3741 50  0000 L CNN
+AR Path="/59510B3D/59513823" Ref="J2"  Part="1"
+AR Path="/59531D77/59540EC0/59513823" Ref="J2"  Part="1"
+AR Path="/5955270D/59513823" Ref="J2"  Part="1"
+F 0 "J2" H 5728 3741 50  0000 L CNN
 F 1 "CONN_01X20" H 5728 3650 50  0000 L CNN
-F 2 "" H 5650 3700 50  0001 C CNN
+F 2 "Pin_Headers:Pin_Header_Straight_1x20_Pitch2.54mm" H 5650 3700 50  0001 C CNN
 F 3 "" H 5650 3700 50  0001 C CNN
 	1    5650 3700
@@
 	475  5185 11220 5185
 $Comp
-L GND #PWR?
+L GND #PWR014
 U 1 1 59542B62
 P 5000 2750
-F 0 "#PWR?" H 5000 2500 50  0001 C CNN
+AR Path="/59510B3D/59542B62" Ref="#PWR014"  Part="1"
+AR Path="/59531D77/59540EC0/59542B62" Ref="#PWR014"  Part="1"
+AR Path="/5955270D/59542B62" Ref="#PWR014"  Part="1"
+F 0 "#PWR014" H 5000 2500 50  0001 C CNN
 F 1 "GND" H 4850 2700 50  0000 C CNN
 F 2 "" H 5000 2750 50  0001 C CNN
@@
 EN_EXT
 $Comp
-L GND #PWR?
+L GND #PWR015
 U 1 1 5954CB1B
 P 5200 4750
-F 0 "#PWR?" H 5200 4500 50  0001 C CNN
+AR Path="/59510B3D/5954CB1B" Ref="#PWR015"  Part="1"
+AR Path="/59531D77/59540EC0/5954CB1B" Ref="#PWR015"  Part="1"
+AR Path="/5955270D/5954CB1B" Ref="#PWR015"  Part="1"
+F 0 "#PWR015" H 5200 4500 50  0001 C CNN
 F 1 "GND" H 5205 4577 50  0000 C CNN
 F 2 "" H 5200 4750 50  0001 C CNN

Commit message: complete Bitsoko ESP32 module design
Parts:
- J2: footprint Pin_Headers:Pin_Header_Straight_1x20_Pitch2.54mm -> narra:Pin_Header_5mil_staggered_1x20_2.54mm
Changed lines of the file:
@@
 F 0 "J2" H 5728 3741 50  0000 L CNN
 F 1 "CONN_01X20" H 5728 3650 50  0000 L CNN
-F 2 "Pin_Headers:Pin_Header_Straight_1x20_Pitch2.54mm" H 5650 3700 50  0001 C CNN
+F 2 "narra:Pin_Header_5mil_staggered_1x20_2.54mm" H 5650 3700 50  0001 C CNN
 F 3 "" H 5650 3700 50  0001 C CNN
 	1    5650 3700
