File: hardware/Bitsoko-ESP32-module/connector_B.sch (KiCad schematic (older format))
At the start: 1 part

Commit message: Semicomplete Bitsoko ESP32 module
Parts:
- J3: renamed from J?; footprint (none) -> Pin_Headers:Pin_Header_Straight_1x20_Pitch2.54mm
Connections:
- net 3v3: now also J3.5 (P5); no longer J3.18 (P18)
- net EXT_5v: now also J3.7 (P7); no longer J3.20 (P20)
- net SENSOR_VN: now also J3.19 (P19); no longer J3.14 (P14)
- net SENSOR_VP: now also J3.20 (P20); no longer J3.15 (P15)
- net CLK: now reaches J3.1 (P1)
- net IO12: now reaches J3.10 (P10)
- net IO14: now reaches J3.11 (P11)
- net IO27: now reaches J3.12 (P12)
- net IO26: now reaches J3.13 (P13)
- net IO32: now reaches J3.16 (P16)
- net IO35: now reaches J3.17 (P17)
- net CMD: now reaches J3.2 (P2)
- net SD3: now reaches J3.3 (P3)
- net SD2: now reaches J3.4 (P4)
- net IO13: now reaches J3.9 (P9)
- new net IO25: J3.14 (P14)
- new net IO33: J3.15 (P15)
- new net IO34: J3.18 (P18)
- no-connect marks 0 -> 2
Other:
- moved on the sheet: J3
Changed lines of the file:
@@
 $EndDescr
 $Comp
-L CONN_01X20 J?
+L CONN_01X20 J3
 U 1 1 5951391D
-P 5600 3700
-F 0 "J?" H 5678 3741 50  0000 L CNN
-F 1 "CONN_01X20" H 5678 3650 50  0000 L CNN
-F 2 "" H 5600 3700 50  0001 C CNN
-F 3 "" H 5600 3700 50  0001 C CNN
-	1    5600 3700
+P 5450 3650
+AR Path="/59510C04/5951391D" Ref="J3"  Part="1"
+AR Path="/59531D77/59540F06/5951391D" Ref="J3"  Part="1"
+AR Path="/59552753/5951391D" Ref="J3"  Part="1"
+F 0 "J3" H 5528 3691 50  0000 L CNN
+F 1 "CONN_01X20" H 5528 3600 50  0000 L CNN
+F 2 "Pin_Headers:Pin_Header_Straight_1x20_Pitch2.54mm" H 5450 3650 50  0001 C CNN
+F 3 "" H 5450 3650 50  0001 C CNN
+	1    5450 3650
 	-1   0    0    1
 $EndComp
@@
 Wire Notes Line
 	475  2365 11220 2365
-Text HLabel 5800 2750 2    60   Input ~ 0
+Text HLabel 5650 4000 2    60   Input ~ 0
 EXT_5v
-Text HLabel 5800 3250 2    60   BiDi ~ 0
+Text HLabel 5650 2700 2    60   BiDi ~ 0
 SENSOR_VP
-Text HLabel 5800 3350 2    60   BiDi ~ 0
+Text HLabel 5650 2800 2    60   BiDi ~ 0
 SENSOR_VN
-Text GLabel 5800 2950 2    60   Input ~ 0
+Text GLabel 5650 4200 2    60   Input ~ 0
 3v3
+Text HLabel 5650 2900 2    60   BiDi ~ 0
+IO34
+Text HLabel 5650 3000 2    60   BiDi ~ 0
+IO35
+Text HLabel 5650 3100 2    60   BiDi ~ 0
+IO32
+Text HLabel 5650 3200 2    60   BiDi ~ 0
+IO33
+Text HLabel 5650 3300 2    60   BiDi ~ 0
+IO25
+Text HLabel 5650 3400 2    60   BiDi ~ 0
+IO26
+Text HLabel 5650 3500 2    60   BiDi ~ 0
+IO27
+Text HLabel 5650 3600 2    60   BiDi ~ 0
+IO14
+Text HLabel 5650 3700 2    60   BiDi ~ 0
+IO12
+Text HLabel 5650 3800 2    60   BiDi ~ 0
+IO13
+Text HLabel 5650 4300 2    60   BiDi ~ 0
+SD2
+Text HLabel 5650 4400 2    60   BiDi ~ 0
+SD3
+Text HLabel 5650 4500 2    60   BiDi ~ 0
+CMD
+Text HLabel 5650 4600 2    60   BiDi ~ 0
+CLK
+NoConn ~ 5650 3900
+NoConn ~ 5650 4100
 $EndSCHEMATC

Commit message: complete Bitsoko ESP32 module design
Parts:
- J3: footprint Pin_Headers:Pin_Header_Straight_1x20_Pitch2.54mm -> narra:Pin_Header_5mil_staggered_1x20_2.54mm
Changed lines of the file:
@@
 F 0 "J3" H 5528 3691 50  0000 L CNN
 F 1 "CONN_01X20" H 5528 3600 50  0000 L CNN
-F 2 "Pin_Headers:Pin_Header_Straight_1x20_Pitch2.54mm" H 5450 3650 50  0001 C CNN
+F 2 "narra:Pin_Header_5mil_staggered_1x20_2.54mm" H 5450 3650 50  0001 C CNN
 F 3 "" H 5450 3650 50  0001 C CNN
 	1    5450 3650
