File: hardware/Bitsoko-ESP32-module/Bitsoko-ESP32-module.kicad_pcb (KiCad board)
At the start: 2 copper layers, 39.4 x 53.3 mm, 17 parts, among them J1 CONN_01X06, J2 CONN_01X20, J3 CONN_01X20, U1 NCP1117-3.3_SOT223, U2 ESP32-WROOM32-MODULE

Commit message: complete Bitsoko ESP32 module design
Parts:
- removed REF***: ESD-Logo_8.9x8mm_SilkScreen, Symbols:ESD-Logo_8.9x8mm_SilkScreen
- J1: footprint Pin_Headers:Pin_Header_Straight_1x06_Pitch2.54mm -> narra:Pin_header_5mil_staggered_1x06_2.54mm
- J2, J3: footprint Pin_Headers:Pin_Header_Straight_1x20_Pitch2.54mm -> narra:Pin_Header_5mil_staggered_1x20_2.54mm
Routing:
- net 3v3: track 5.29 -> 105.9 mm, vias 0 -> 10
- net GND: track 33.4 -> 62.9 mm, vias 7 -> 21
- net /sheet59552648/EXT_5V: track 0.00 -> 12.4 mm
Other:
- net class 5v power added: clearance 0.2, trace_width 0.508, via_dia 0.8, via_drill 0.4

Commit message: correct UART connections
Connections:
- J1 pad 2: /sheet59552649/EN_EXT -> /sheet59552649/RX
- J1 pad 3: /sheet59552649/IO0_EXT -> /sheet59552649/TX
- J2 pad 13: /sheet59552649/EN -> /sheet59552649/RX
- J2 pad 14: /sheet59552649/IO0 -> /sheet59552649/TX
- J2 pad 15: /sheet59552649/IO0_EXT -> /sheet59552649/IO0
- J2 pad 16: /sheet59552649/EN_EXT -> /sheet59552649/EN
- U2 pad 34: /sheet59552649/EN_EXT -> /sheet59552649/RX
- U2 pad 35: /sheet59552649/IO0_EXT -> /sheet59552649/TX
Routing:
- net /sheet59552649/IO0_EXT: track 61.5 -> 0.00 mm, vias 3 -> 0
- net /sheet59552649/TX: track 0.00 -> 60.7 mm, vias 0 -> 6
- net /sheet59552649/EN_EXT: track 57.8 -> 0.00 mm, vias 3 -> 0
- net /sheet59552649/RX: track 0.00 -> 57.6 mm, vias 0 -> 4
- net /sheet59552649/EN: track 79.3 -> 92.3 mm
- net /sheet59552649/IO0: track 57.1 -> 53.8 mm
