File: hardware/Bitsoko-ESP32-module/USB-UART.sch (KiCad schematic (older format))
At the start: 1 part

Commit message: Semicomplete Bitsoko ESP32 module
Parts:
- J1: renamed from J?; footprint (none) -> Pin_Headers:Pin_Header_Straight_1x06_Pitch2.54mm
Changed lines of the file:
@@
 $EndDescr
 $Comp
-L CONN_01X06 J?
+L CONN_01X06 J1
 U 1 1 5951994E
 P 5680 3525
-F 0 "J?" H 5758 3566 50  0000 L CNN
+AR Path="/59510B33/5951994E" Ref="J1"  Part="1"
+AR Path="/59531D77/59540E0F/5951994E" Ref="J1"  Part="1"
+AR Path="/5955265C/5951994E" Ref="J1"  Part="1"
+F 0 "J1" H 5758 3566 50  0000 L CNN
 F 1 "CONN_01X06" H 5758 3475 50  0000 L CNN
-F 2 "" H 5680 3525 50  0001 C CNN
+F 2 "Pin_Headers:Pin_Header_Straight_1x06_Pitch2.54mm" H 5680 3525 50  0001 C CNN
 F 3 "" H 5680 3525 50  0001 C CNN
 	1    5680 3525
@@
 3v3
 $Comp
-L GND #PWR?
+L GND #PWR05
 U 1 1 595199D1
 P 5230 3875
-F 0 "#PWR?" H 5230 3625 50  0001 C CNN
+AR Path="/59510B33/595199D1" Ref="#PWR05"  Part="1"
+AR Path="/59531D77/59540E0F/595199D1" Ref="#PWR05"  Part="1"
+AR Path="/5955265C/595199D1" Ref="#PWR05"  Part="1"
+F 0 "#PWR05" H 5230 3625 50  0001 C CNN
 F 1 "GND" H 5235 3702 50  0000 C CNN
 F 2 "" H 5230 3875 50  0001 C CNN

Commit message: complete Bitsoko ESP32 module design
Parts:
- J1: footprint Pin_Headers:Pin_Header_Straight_1x06_Pitch2.54mm -> narra:Pin_header_5mil_staggered_1x06_2.54mm
Changed lines of the file:
@@
 F 0 "J1" H 5758 3566 50  0000 L CNN
 F 1 "CONN_01X06" H 5758 3475 50  0000 L CNN
-F 2 "Pin_Headers:Pin_Header_Straight_1x06_Pitch2.54mm" H 5680 3525 50  0001 C CNN
+F 2 "narra:Pin_header_5mil_staggered_1x06_2.54mm" H 5680 3525 50  0001 C CNN
 F 3 "" H 5680 3525 50  0001 C CNN
 	1    5680 3525

Commit message: correct UART connections
Connections:
- net EN_EXT renamed RX
- net IO0_EXT renamed TX
Changed lines of the file:
@@
 Connection ~ 5455 3675
 Text HLabel 5190 2590 1    40   Output ~ 0
+EN_EXT
+Text HLabel 5275 2720 1    40   Input ~ 0
+IO0_EXT
+Text HLabel 5370 2990 1    40   Output ~ 0
+TX_EXT
+Text HLabel 5430 3225 1    40   Output ~ 0
 RX_EXT
-Text HLabel 5275 2720 1    40   Input ~ 0
-TX_EXT
-Text HLabel 5370 2990 1    40   Output ~ 0
-IO0_EXT
-Text HLabel 5430 3225 1    40   Output ~ 0
-EN_EXT
 Wire Wire Line
 	5280 3500 5225 3440
