File: hardware/Bitsoko-ESP32-module-v2/Bitsoko-ESP32-module-v2.kicad_pcb (KiCad board)
At the start: 2 copper layers, 40.6 x 27.9 mm, 3 parts, among them J1 CONN_02X10, J2 CONN_02X10, U1 ESP32-WROOM32-MODULE

Commit message: Modify ESP32 module design
1. Add 22uF 1210, 2x0.1uF 0805 decoupling capacitors.
2. Add via fence on ground under the ESP32 WROOM 32 for a solid ground connection.
Parts:
- added C1: 0.1uF, Capacitors_SMD:C_0805_HandSoldering, B.Cu at (129.3, 82.5)
- added C2: 22uF, Capacitors_SMD:C_1210_HandSoldering, B.Cu at (129.3, 79.5)
- added C3: 0.1uF, Capacitors_SMD:C_0805_HandSoldering, B.Cu at (129.3, 85.1)
Connections:
- net /GND renamed GND
Routing:
- net /EN: track 8.75 -> 17.4 mm
- net /3V3: track 5.76 -> 12.1 mm
- net GND: vias 22 -> 59
