File: hardware/Bitsoko-ESP32-module-v2/Bitsoko-ESP32-module-v2.sch (KiCad schematic (older format))
At the start: 3 parts, among them J1 CONN_02X10, J2 CONN_02X10, U1 ESP32-WROOM32-MODULE

Commit message: Replaced pin headers with offset staggered headers from a friction fit without soldering
Parts:
- J1, J2: footprint (none) -> narra:Pin_Header_Straight_2x10_Pitch2.54mm_staggered
Changed lines of the file:
@@
 LIBS:valves
 LIBS:narra
+LIBS:Bitsoko-ESP32-module-v2-cache
 EELAYER 26 0
 EELAYER END
@@
 F 0 "J2" H 2950 3765 50  0000 C CNN
 F 1 "CONN_02X10" H 2950 3674 50  0000 C CNN
-F 2 "" H 2950 1900 50  0001 C CNN
+F 2 "narra:Pin_Header_Straight_2x10_Pitch2.54mm_staggered" H 2950 1900 50  0001 C CNN
 F 3 "" H 2950 1900 50  0001 C CNN
 	1    2950 3100
@@
 F 0 "J1" H 7700 3715 50  0000 C CNN
 F 1 "CONN_02X10" H 7700 3624 50  0000 C CNN
-F 2 "" H 7700 1850 50  0001 C CNN
+F 2 "narra:Pin_Header_Straight_2x10_Pitch2.54mm_staggered" H 7700 1850 50  0001 C CNN
 F 3 "" H 7700 1850 50  0001 C CNN
 	1    7700 3050
