File: hardware/Bitsoko-ESP32-module-v2/_saved_Bitsoko-ESP32-module-v2.sch (KiCad schematic (older format))
At the start: 6 parts, among them J1 CONN_02X10, J2 CONN_02X10, U1 ESP32-WROOM32-MODULE

Commit message: Modify ESP32 module design
1. Add 22uF 1210, 2x0.1uF 0805 decoupling capacitors.
2. Add via fence on ground under the ESP32 WROOM 32 for a solid ground connection.
Parts:
- removed C2: 100uF, Capacitors_THT:CP_Radial_D5.0mm_P2.50mm, symbol CP
- added C2: 22uF, Capacitors_SMD:C_1210_HandSoldering, symbol C
- C1: value 1uF -> 0.1uF; footprint (none) -> Capacitors_SMD:C_0805_HandSoldering
- C3: value C -> 0.1uF; footprint (none) -> Capacitors_SMD:C_0805_HandSoldering
Connections:
- net 3V3: now also C2.1
- net GND: now also C2.2
Changed lines of the file:
@@
 P 9895 5375
 F 0 "C1" H 10010 5421 50  0000 L CNN
-F 1 "1uF" H 10010 5330 50  0000 L CNN
-F 2 "" H 9933 5225 50  0001 C CNN
+F 1 "0.1uF" H 10010 5330 50  0000 L CNN
+F 2 "Capacitors_SMD:C_0805_HandSoldering" H 9933 5225 50  0001 C CNN
 F 3 "" H 9895 5375 50  0001 C CNN
 	1    9895 5375
-	1    0    0    -1
-$EndComp
-$Comp
-L CP C2
-U 1 1 59A51876
-P 10250 5375
-F 0 "C2" H 10368 5421 50  0000 L CNN
-F 1 "100uF" H 10368 5330 50  0000 L CNN
-F 2 "Capacitors_THT:CP_Radial_D5.0mm_P2.50mm" H 10288 5225 50  0001 C CNN
-F 3 "" H 10250 5375 50  0001 C CNN
-	1    10250 5375
 	1    0    0    -1
 $EndComp
@@
 P 7415 5390
 F 0 "C3" H 7530 5436 50  0000 L CNN
-F 1 "C" H 7530 5345 50  0000 L CNN
-F 2 "" H 7453 5240 50  0001 C CNN
+F 1 "0.1uF" H 7530 5345 50  0000 L CNN
+F 2 "Capacitors_SMD:C_0805_HandSoldering" H 7453 5240 50  0001 C CNN
 F 3 "" H 7415 5390 50  0001 C CNN
 	1    7415 5390
@@
 Wire Wire Line
 	10250 5555 10250 5525
+$Comp
+L C C2
+U 1 1 59A51BF7
+P 10250 5375
+F 0 "C2" H 10365 5421 50  0000 L CNN
+F 1 "22uF" H 10365 5330 50  0000 L CNN
+F 2 "Capacitors_SMD:C_1210_HandSoldering" H 10288 5225 50  0001 C CNN
+F 3 "" H 10250 5375 50  0001 C CNN
+	1    10250 5375
+	1    0    0    -1
+$EndComp
 $EndSCHEMATC
