File: hardware/ESP-32-programmer/ESP-32-programmer.kicad_pcb (KiCad board)
At the start: 2 copper layers, 100 x 45 mm, 17 parts, among them J1 GS2, J2 CONN_01X06, J3 CONN_02X10, J4 CONN_02X10, J5 CONN_02X10, J6 CONN_01X06, J7 GS2, SW1 SW_DIP_x02, SW2 SW_Push, U1 LD1117S33TR_SOT223, U2 ESP-32-module

Commit message: Change module in ESP32 programmer
Routing:
- net /TMS: track 86.8 -> 86.2 mm

Commit message: Design rule chcker pass
1.DRC pass for ESP32 module and no unconnected nets.
2.DRC pass for ESP32 programmer and no unconnected nets.
Routing:
- net /TMS: track 86.2 -> 87.1 mm
- net /TCK: track 85.4 -> 86.1 mm
Other:
- board text added: "BOOT MODE SEL"
- board text added: "CP210x"
- board text added: "FTDI 232RL"
- board text added: "JTAG"
- board text added: "NORMAL"
- board text added: "PROG"
- board text added: "RESET"
Changed lines of the file:
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@@
   (general
     (thickness 1.6)
-    (drawings 8)
-    (tracks 381)
+    (drawings 20)
+    (tracks 386)
     (zones 0)
     (modules 17)
@@
       (rotate (xyz 0 0 90))
     )
+  )
+  (gr_text "FTDI 232RL" (at 114.808 87.884) (layer F.SilkS)
+    (effects (font (size 1.5 1.5) (thickness 0.3)))
+  )
+  (gr_text CP210x (at 150.368 87.63) (layer F.SilkS)
+    (effects (font (size 1.5 1.5) (thickness 0.3)))
+  )
+  (gr_text NORMAL (at 179.324 50.546) (layer F.SilkS)
+    (effects (font (size 0.762 0.762) (thickness 0.127)))
+  )
+  (gr_text PROG (at 179.324 57.912) (layer F.SilkS)
+    (effects (font (size 0.762 0.762) (thickness 0.127)))
+  )
+  (gr_line (start 180.086 56.642) (end 180.086 56.388) (layer F.SilkS) (width 0.2))
+  (gr_line (start 179.578 57.15) (end 180.086 56.642) (layer F.SilkS) (width 0.2))
+  (gr_line (start 179.07 56.388) (end 179.07 56.642) (layer F.SilkS) (width 0.2))
+  (gr_line (start 179.578 57.15) (end 179.07 56.642) (layer F.SilkS) (width 0.2))
+  (gr_line (start 179.578 51.562) (end 179.578 57.15) (layer F.SilkS) (width 0.2))
+  (gr_text "BOOT\nMODE\nSEL" (at 177.8 54.102) (layer F.SilkS)
+    (effects (font (size 0.762 0.762) (thickness 0.127)))
+  )
+  (gr_text RESET (at 183.388 70.358) (layer F.SilkS)
+    (effects (font (size 0.762 0.762) (thickness 0.127)))
+  )
+  (gr_text JTAG (at 186.182 87.376) (layer F.SilkS)
+    (effects (font (size 1.5 1.5) (thickness 0.3)))
   )
   (dimension 100 (width 0.3) (layer Dwgs.User)
@@
   (segment (start 116.90959 67.62) (end 117.234 67.62) (width 0.25) (layer F.Cu) (net 12))
   (segment (start 99.92 67.78) (end 101.095001 68.955001) (width 0.25) (layer F.Cu) (net 12))
+  (segment (start 127.465 71.839) (end 120.706 65.08) (width 0.25) (layer F.Cu) (net 13))
+  (segment (start 120.706 65.08) (end 119.4438 65.08) (width 0.25) (layer F.Cu) (net 13))
+  (segment (start 127.465 73.025) (end 127.465 71.839) (width 0.25) (layer F.Cu) (net 13))
   (segment (start 102.206 65.24) (end 114.846 65.24) (width 0.25) (layer F.Cu) (net 13))
   (segment (start 114.846 65.24) (end 116.332 63.754) (width 0.25) (layer F.Cu) (net 13))
+  (segment (start 116.332 63.754) (end 118.1178 63.754) (width 0.25) (layer F.Cu) (net 13))
+  (segment (start 118.1178 63.754) (end 119.4438 65.08) (width 0.25) (layer F.Cu) (net 13))
   (segment (start 146.431 73.025) (end 147.955 74.549) (width 0.25) (layer F.Cu) (net 13))
-  (segment (start 116.332 63.754) (end 118.194 63.754) (width 0.25) (layer F.Cu) (net 13))
   (segment (start 168.656 88.646) (end 172.72 84.582) (width 0.25) (layer F.Cu) (net 13))
-  (segment (start 118.194 63.754) (end 127.465 73.025) (width 0.25) (layer F.Cu) (net 13))
   (segment (start 127.465 73.025) (end 146.431 73.025) (width 0.25) (layer F.Cu) (net 13))
   (segment (start 147.955 74.549) (end 147.955 78.486) (width 0.25) (layer F.Cu) (net 13))
@@
   (segment (start 158.568998 87.249) (end 164.973 87.249) (width 0.25) (layer F.Cu) (net 14))
   (segment (start 164.973 87.249) (end 167.64 84.582) (width 0.25) (layer F.Cu) (net 14))
-  (segment (start 166.878 88.138) (end 169.330001 85.685999) (width 0.25) (layer F.Cu) (net 15))
-  (segment (start 153.67 77.47282) (end 153.67 83.439) (width 0.25) (layer F.Cu) (net 15))
-  (segment (start 124.968001 63.627001) (end 133.731 72.39) (width 0.25) (layer F.Cu) (net 15))
-  (segment (start 120.502201 63.627001) (end 124.968001 63.627001) (width 0.25) (layer F.Cu) (net 15))
-  (segment (start 133.731 72.39) (end 148.58718 72.39) (width 0.25) (layer F.Cu) (net 15))
-  (segment (start 119.286199 63.715001) (end 120.414201 63.715001) (width 0.25) (layer F.Cu) (net 15))
-  (segment (start 120.414201 63.715001) (end 120.502201 63.627001) (width 0.25) (layer F.Cu) (net 15))
-  (segment (start 148.58718 72.39) (end 153.67 77.47282) (width 0.25) (layer F.Cu) (net 15))
-  (segment (start 118.875187 63.303989) (end 119.286199 63.715001) (width 0.25) (layer F.Cu) (net 15))
+  (segment (start 116.1456 62.9244) (end 116.53 62.54) (width 0.25) (layer F.Cu) (net 15))
+  (segment (start 116.53 62.54) (end 117.3102 62.54) (width 0.25) (layer F.Cu) (net 15))
+  (segment (start 116.1456 63.303989) (end 116.1456 62.9244) (width 0.25) (layer F.Cu) (net 15))
+  (segment (start 170.18 84.836) (end 166.878 88.138) (width 0.25) (layer F.Cu) (net 15))
+  (segment (start 166.878 88.138) (end 158.369 88.138) (width 0.25) (layer F.Cu) (net 15))
+  (segment (start 124.968001 63.627001) (end 120.502201 63.627001) (width 0.25) (layer F.Cu) (net 15))
+  (segment (start 158.369 88.138) (end 153.67 83.439) (width 0.25) (layer F.Cu) (net 15))
+  (segment (start 120.414201 63.715001) (end 119.286199 63.715001) (width 0.25) (layer F.Cu) (net 15))
+  (segment (start 118.111198 62.54) (end 117.3102 62.54) (width 0.25) (layer F.Cu) (net 15))
+  (segment (start 153.67 83.439) (end 153.67 77.47282) (width 0.25) (layer F.Cu) (net 15))
+  (segment (start 148.58718 72.39) (end 133.731 72.39) (width 0.25) (layer F.Cu) (net 15))
+  (segment (start 153.67 77.47282) (end 148.58718 72.39) (width 0.25) (layer F.Cu) (net 15))
+  (segment (start 133.731 72.39) (end 124.968001 63.627001) (width 0.25) (layer F.Cu) (net 15))
+  (segment (start 120.502201 63.627001) (end 120.414201 63.715001) (width 0.25) (layer F.Cu) (net 15))
+  (segment (start 119.286199 63.715001) (end 118.111198 62.54) (width 0.25) (layer F.Cu) (net 15))
   (segment (start 101.095001 63.875001) (end 115.574589 63.875001) (width 0.25) (layer F.Cu) (net 15))
-  (segment (start 116.1456 63.303989) (end 118.875187 63.303989) (width 0.25) (layer F.Cu) (net 15))
   (segment (start 115.574589 63.875001) (end 116.1456 63.303989) (width 0.25) (layer F.Cu) (net 15))
-  (segment (start 158.369 88.138) (end 166.878 88.138) (width 0.25) (layer F.Cu) (net 15))
-  (segment (start 169.330001 85.685999) (end 170.18 84.836) (width 0.25) (layer F.Cu) (net 15))
   (segment (start 99.92 62.7) (end 101.095001 63.875001) (width 0.25) (layer F.Cu) (net 15))
-  (segment (start 153.67 83.439) (end 158.369 88.138) (width 0.25) (layer F.Cu) (net 15))
   (segment (start 114.846 60.16) (end 116.332 58.674) (width 0.25) (layer F.Cu) (net 16))
   (segment (start 102.206 60.16) (end 114.846 60.16) (width 0.25) (layer F.Cu) (net 16))
