File: hardware/ESP-32-programmer/ESP-32-programmer.kicad_pcb (KiCad board)
At the start: 2 copper layers, 100 x 45 mm, 17 parts, among them J1 GS2, J2 CONN_01X06, J3 CONN_02X10, J4 CONN_02X10, J5 CONN_02X10, J6 CONN_01X06, J7 GS2, SW1 SW_DIP_x02, SW2 SW_Push, U1 LD1117S33TR_SOT223, U2 ESP-32-module

Commit message: Correct ESP-32 design based on tests
1. TXD of the ESP32 was connected to TXD of the FTDI programmer. This was corrected RXD<=>TXD and vice versa.
2. The DTR programmer line was connected to the EN line of the ESP32. This allows use of the DIP switch or tactile button to set boot mode.
Parts:
- added J8: GS2, Connectors:GS2, B.Cu at (131.7, 85.1)
Connections:
- J1 pad 2: /EN -> /DTR
- J2 pad 1: Net-(J2-Pad1) -> /DTR
- J2 pad 4: /5v -> /3v3
- J5 pad 3: /EN -> /DTR
- J6 pad 1: /5v -> Net-(J6-Pad1)
- J6 pad 5: Net-(J6-Pad5) -> /DTR
- R2 pad 2: /EN -> /DTR
- SW2 pad 1: /EN -> /IO0
- U2 pad 24: /TXD -> /RXD
- U2 pad 25: /RXD -> /TXD
- U2 pad 3: /EN -> /DTR
Routing:
- net /DTR: track 0.00 -> 164.7 mm, vias 0 -> 4
- net /EN: track 128.8 -> 0.00 mm, vias 3 -> 0
- net /5v: track 107.3 -> 83.4 mm, vias 5 -> 4
- net /IO0: track 49.2 -> 66.6 mm
- net /3v3: track 169.7 -> 177.2 mm
- net /RXD: track 106.8 -> 112.5 mm, vias 2 -> 4
- net /TXD: track 105.9 -> 108.7 mm, vias 0 -> 2
- net Net-(J6-Pad1): track 0.00 -> 2.68 mm
- net GND: vias 0 -> 52
- net (no net): vias 0 -> 1

Commit message: Move solder bridge on CP2012 programmer header
1. Move the solder bridge on the CP2012 header from 5v line to 3.3v line to prevent voltage fed to LDO(5v) output(3v3) from feeding back to the CP2102 3v3 output. This would allow unwanted currents to flow between the supplies.
Parts:
- moved J8 15.5 mm to (146.6, 80.8), turned to 0 degrees
Connections:
- J6 pad 1: Net-(J6-Pad1) -> /5v
- J6 pad 6: /3v3 -> Net-(J6-Pad6)
- J8 pad 1: Net-(J6-Pad1) -> Net-(J6-Pad6)
- J8 pad 2: /5v -> /3v3
Routing:
- net /3v3: track 177.2 -> 183.7 mm
- net Net-(J6-Pad6): track 0.00 -> 3.95 mm
- net Net-(J6-Pad1): track 2.68 -> 0.00 mm
- net /5v: track 83.4 -> 84.6 mm
- net (no net): vias 1 -> 0
