File: hardware/ESP-32-programmer/ESP-32-programmer.kicad_pcb (KiCad board)
At the start: 2 copper layers, 100 x 45 mm, 18 parts, among them J1 GS2, J2 CONN_01X06, J3 CONN_02X10, J4 CONN_02X10, J5 CONN_02X10, J6 CONN_01X06, J7 GS2, J8 GS2, SW1 SW_DIP_x02, SW2 SW_Push, U1 LD1117S33TR_SOT223, U2 ESP-32-module

Commit message: Rotate CP210x programming header 180 deg
1. Correct design error for cp210x programming header by rotating it 180 degrees and reconnecting.
2. Noticed after PCB fabrication.
Parts:
- moved J6 11.1 mm to (146.1, 85.0), turned to 270 degrees
Routing:
- net Net-(J6-Pad6): track 3.95 -> 21.4 mm
- net GND: track 18.4 -> 33.7 mm, vias 52 -> 54
- net /DTR: track 164.7 -> 175.4 mm
- net /5v: track 84.6 -> 93.1 mm
- net /TXD: track 108.7 -> 111.2 mm, vias 2 -> 3
- net /RXD: track 112.5 -> 114.1 mm, vias 4 -> 6
- net /TCK: track 86.1 -> 87.5 mm
- net /TDO: track 70.9 -> 71.5 mm
