File: hardware/ESP-32-programmer/ESP-32-programmer.sch (KiCad schematic (older format))
At the start: 17 parts, among them J1 GS2, J2 CONN_01X06, J3 CONN_02X10, J4 CONN_02X10, J5 CONN_02X10, J6 CONN_01X06, J7 GS2, SW1 SW_DIP_x02, SW2 SW_Push, U1 LD1117S33TR_SOT223, U2 ESP-32-module

Commit message: Correct ESP-32 design based on tests
1. TXD of the ESP32 was connected to TXD of the FTDI programmer. This was corrected RXD<=>TXD and vice versa.
2. The DTR programmer line was connected to the EN line of the ESP32. This allows use of the DIP switch or tactile button to set boot mode.
Parts:
- added J8: GS2, Connectors:GS2, symbol GS2
Connections:
- net 3v3: now also J2.4 (P4)
- net 5v: now also J8.2 (G2); no longer J2.4 (P4), J6.1 (P1)
- net DTR: now also J1.2 (G2), J2.1 (P1), J5.3 (P3), J6.5 (P5), R2.2, U2.3 (EN)
- net IO0: now also SW2.1
- net RXD: now also U2.24 (TXD); no longer U2.25 (RXD)
- net TXD: now also U2.25 (RXD); no longer U2.24 (TXD)
- removed net EN: J1.2 (G2), J5.3 (P3), R2.2, SW2.1, U2.3 (EN)
- new net: J6.1 (P1), J8.1 (G1)
- no-connect marks 10 -> 8
Changed lines of the file:
@@
 	1    0    0    -1
 $EndComp
-Text Label 9600 1200 2    60   ~ 0
+Text Label 9610 1200 2    60   ~ 0
 DTR
 Text Label 9600 1300 2    60   ~ 0
@@
 TXD
 Text Label 9600 1500 2    60   ~ 0
-5v
+3v3
 Text Label 9600 1600 2    60   ~ 0
 CTS
@@
 Text Label 7560 3210 0    60   ~ 0
 IO22
-Text Label 7560 3310 0    60   ~ 0
+Text Label 7560 3410 0    60   ~ 0
 TXD
-Text Label 7560 3410 0    60   ~ 0
-RXD
 Text Label 7560 3510 0    60   ~ 0
 IO21
@@
 	1    0    0    -1
 $EndComp
-Text Label 9600 5580 2    60   ~ 0
+Text Label 9140 5580 2    60   ~ 0
 5v
 Text Label 9600 5780 2    60   ~ 0
@@
 Text Notes 8270 6530 2    60   ~ 0
 SYSTEM_RESET
-Text Notes 4660 6530 2    60   ~ 0
-BOOT MODE SELECTION(PU-SPI BOOT, PD-DOWNLOAD BOOT)
 $Bitmap
 Pos 7180 6720
@@
 EndData
 $EndBitmap
-Text Label 2150 5850 2    60   ~ 0
-IO0
-$Comp
-L GND #PWR015
-U 1 1 59977E1F
-P 3300 5950
-F 0 "#PWR015" H 3300 5700 50  0001 C CNN
-F 1 "GND" H 3305 5777 50  0000 C CNN
-F 2 "" H 3300 5950 50  0001 C CNN
-F 3 "" H 3300 5950 50  0001 C CNN
-	1    3300 5950
-	1    0    0    -1
-$EndComp
-$Comp
-L SW_DIP_x02 SW1
-U 1 1 59977E12
-P 2650 5900
-F 0 "SW1" H 2650 6267 50  0000 C CNN
-F 1 "SW_DIP_x02" H 2650 6176 50  0000 C CNN
-F 2 "Buttons_Switches_THT:SW_DIP_x2_W7.62mm_Slide_LowProfile" H 2650 5900 50  0001 C CNN
-F 3 "" H 2650 5900 50  0001 C CNN
-	1    2650 5900
-	1    0    0    -1
-$EndComp
 Wire Wire Line
 	5260 3010 5710 3010
@@
 	8270 5220 8270 6540
 Wire Wire Line
-	9700 5580 9600 5580
+	9570 5580 9700 5580
 Wire Wire Line
 	9160 5680 9700 5680
@@
 	4660 5190 4660 6535
 Wire Wire Line
-	2350 5800 2350 5900
-Wire Wire Line
-	2350 5850 2150 5850
-Connection ~ 2350 5850
-Wire Wire Line
-	2950 5800 2950 5900
-Wire Wire Line
-	2950 5850 3300 5850
-Connection ~ 2950 5850
-Wire Wire Line
-	3300 5850 3300 5950
-Wire Wire Line
 	7200 5850 7200 5950
 Wire Wire Line
 	6720 5850 7200 5850
-Text Label 6050 5850 2    60   ~ 0
-EN
 Wire Wire Line
 	6050 5850 6320 5850
@@
 	0    -1   -1   0
 $EndComp
-NoConn ~ 9700 5980
-NoConn ~ 9700 1200
 NoConn ~ 9700 1600
 Text Label 9600 5980 2    60   ~ 0
@@
 	1    0    0    -1
 $EndComp
+Text Label 6050 5850 2    60   ~ 0
+IO0
+Text Notes 4660 6530 2    60   ~ 0
+BOOT MODE SELECTION(PU-SPI BOOT, PD-DOWNLOAD BOOT)
+$Comp
+L GND #PWR015
+U 1 1 59977E1F
+P 3300 5950
+F 0 "#PWR015" H 3300 5700 50  0001 C CNN
+F 1 "GND" H 3305 5777 50  0000 C CNN
+F 2 "" H 3300 5950 50  0001 C CNN
+F 3 "" H 3300 5950 50  0001 C CNN
+	1    3300 5950
+	1    0    0    -1
+$EndComp
+$Comp
+L SW_DIP_x02 SW1
+U 1 1 59977E12
+P 2650 5900
+F 0 "SW1" H 2650 6267 50  0000 C CNN
+F 1 "SW_DIP_x02" H 2650 6176 50  0000 C CNN
+F 2 "Buttons_Switches_THT:SW_DIP_x2_W7.62mm_Slide_LowProfile" H 2650 5900 50  0001 C CNN
+F 3 "" H 2650 5900 50  0001 C CNN
+	1    2650 5900
+	1    0    0    -1
+$EndComp
+Wire Wire Line
+	2350 5800 2350 5900
+Wire Wire Line
+	2350 5850 2150 5850
+Connection ~ 2350 5850
+Wire Wire Line
+	2950 5800 2950 5900
+Wire Wire Line
+	2950 5850 3300 5850
+Connection ~ 2950 5850
+Wire Wire Line
+	3300 5850 3300 5950
+Text Label 2150 5850 2    60   ~ 0
+IO0
+Wire Wire Line
+	9700 5980 9600 5980
+Wire Wire Line
+	9700 1200 9610 1200
+Wire Wire Line
+	4690 2990 4850 2990
+Wire Wire Line
+	4850 2990 4850 3210
+Connection ~ 4850 3210
+Text Label 4690 2990 0    60   ~ 0
+DTR
+$Comp
+L GS2 J8
+U 1 1 59A5D683
+P 9370 5580
+F 0 "J8" V 9165 5580 50  0000 C CNN
+F 1 "GS2" V 9256 5580 50  0000 C CNN
+F 2 "Connectors:GS2" V 9444 5580 50  0001 C CNN
+F 3 "" H 9370 5580 50  0001 C CNN
+	1    9370 5580
+	0    1    1    0
+$EndComp
+Wire Wire Line
+	9140 5580 9170 5580
+Text Label 7560 3310 0    60   ~ 0
+RXD
 $EndSCHEMATC

Commit message: Move solder bridge on CP2012 programmer header
1. Move the solder bridge on the CP2012 header from 5v line to 3.3v line to prevent voltage fed to LDO(5v) output(3v3) from feeding back to the CP2102 3v3 output. This would allow unwanted currents to flow between the supplies.
Connections:
- net 3v3: now also J8.2 (G2); no longer J6.6 (P6)
- net 5v: now also J6.1 (P1); no longer J8.2 (G2)
- net at J8.1 (G1): now also J6.6 (P6); no longer J6.1 (P1)
Other:
- moved on the sheet: J8
Changed lines of the file:
@@
 	1    0    0    -1
 $EndComp
-Text Label 9140 5580 2    60   ~ 0
+Text Label 9540 5580 2    60   ~ 0
 5v
 Text Label 9600 5780 2    60   ~ 0
@@
 Text Label 9600 5880 2    60   ~ 0
 RXD
-Text Label 9600 6080 2    60   ~ 0
-3v3
 $Comp
 L GS2 J1
@@
 	8270 5220 8270 6540
 Wire Wire Line
-	9570 5580 9700 5580
+	9540 5580 9700 5580
 Wire Wire Line
 	9160 5680 9700 5680
@@
 	9160 5760 9160 5680
 Wire Wire Line
-	9700 6080 9600 6080
+	9550 6080 9700 6080
 Wire Wire Line
 	1850 1250 1590 1250
@@
 L GS2 J8
 U 1 1 59A5D683
-P 9370 5580
-F 0 "J8" V 9165 5580 50  0000 C CNN
-F 1 "GS2" V 9256 5580 50  0000 C CNN
-F 2 "Connectors:GS2" V 9444 5580 50  0001 C CNN
-F 3 "" H 9370 5580 50  0001 C CNN
-	1    9370 5580
+P 9350 6080
+F 0 "J8" V 9145 6080 50  0000 C CNN
+F 1 "GS2" V 9236 6080 50  0000 C CNN
+F 2 "Connectors:GS2" V 9424 6080 50  0001 C CNN
+F 3 "" H 9350 6080 50  0001 C CNN
+	1    9350 6080
 	0    1    1    0
 $EndComp
-Wire Wire Line
-	9140 5580 9170 5580
 Text Label 7560 3310 0    60   ~ 0
 RXD
+Wire Wire Line
+	9150 6080 9050 6080
+Text Label 9050 6080 2    60   ~ 0
+3v3
 $EndSCHEMATC
