File: hardware/drivers/ND-03/ND-03.kicad_pcb (KiCad board)
At the start: 2 copper layers, 155.6 x 134.7 mm, 113 parts, among them J1 Screw_Terminal_1x02, J10 Screw_Terminal_1x02, J11 Screw_Terminal_1x02, J12 Screw_Terminal_1x02, J13 Screw_Terminal_1x02, J14 Screw_Terminal_1x02, J15 Screw_Terminal_1x02, J16 Screw_Terminal_1x02, J17 Screw_Terminal_1x02, J18 Screw_Terminal_1x02, J19 Screw_Terminal_1x02, J2 Screw_Terminal_1x02, J20 Screw_Terminal_1x02, J21 Screw_Terminal_1x02, J22 Screw_Terminal_1x02, J23 Screw_Terminal_1x02, J24 Screw_Terminal_1x02, J25 Screw_Terminal_1x02, J26 Screw_Terminal_1x02, J27 Screw_Terminal_1x02, J28 Screw_Terminal_1x02, J29 Screw_Terminal_1x02, J3 Screw_Terminal_1x02, J30 Screw_Terminal_1x02, J31 Screw_Terminal_1x02, J32 Screw_Terminal_1x02, J33 Screw_Terminal_1x02, J34 Screw_Terminal_1x02, J35 Screw_Terminal_1x02, J36 Screw_Terminal_1x02, J37 Screw_Terminal_1x02, J38 Screw_Terminal_1x02, J39 Screw_Terminal_1x02, J4 Screw_Terminal_1x02, J40 Screw_Terminal_1x02, J41 Screw_Terminal_1x02, J42 Screw_Terminal_1x02, J43 Screw_Terminal_1x02, J44 Screw_Terminal_1x02, J45 Screw_Terminal_1x02, J46 Screw_Terminal_1x02, J47 Screw_Terminal_1x02, J48 Screw_Terminal_1x02, J49 Screw_Terminal_1x02, J5 Screw_Terminal_1x02, J50 Screw_Terminal_1x02, J51 Screw_Terminal_1x02, J52 Screw_Terminal_1x02, J53 Screw_Terminal_1x02, J54 Screw_Terminal_1x02, J55 Screw_Terminal_1x02, J56 Screw_Terminal_1x02, J57 Screw_Terminal_1x02, J58 Screw_Terminal_1x02, J59 Screw_Terminal_1x02, J6 Screw_Terminal_1x02, J60 Screw_Terminal_1x02, J61 Screw_Terminal_1x02, J62 Screw_Terminal_1x02, J63 Screw_Terminal_1x02, J64 Screw_Terminal_1x02, J65 Screw_Terminal_1x02, J66 Screw_Terminal_1x02, J67 Screw_Terminal_1x02, J68 GS3, J69 Screw_Terminal_1x02, J7 Screw_Terminal_1x02, J70 Screw_Terminal_1x02, J71 Screw_Terminal_1x02, J72 Screw_Terminal_1x02, J8 Screw_Terminal_1x02, J9 Screw_Terminal_1x02, U1 ESP-32-module, U10 74HC595, U11 74HC595, U12 74HC595, U13 74HC595, U14 74HC595, U15 74HC595, U16 74HC595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

Commit message: Update PCB driver design
Parts:
- removed J58: Screw_Terminal_1x02, Connectors_Terminal_Blocks:TerminalBlock_Pheonix_MKDS1.5-2pol
- moved J69 47.4 mm to (117.2, 37.2)
- moved J70 47.4 mm to (127.2, 37.3)
- moved J71 47.4 mm to (107.2, 37.3)
- moved J72 47.4 mm to (97.2, 37.1)
- moved R1 47.4 mm to (43.9, 85.3)
- moved U11 47.4 mm to (49.0, 99.3)
- moved U12 47.4 mm to (49.0, 141.2)
- moved U15 47.4 mm to (49.0, 155.2)
- moved U16 47.4 mm to (49.0, 113.3)
- moved U19 47.4 mm to (49.0, 127.2)
- moved U4 47.4 mm to (49.0, 57.4)
- moved U7 47.4 mm to (49.0, 71.4)
- moved U8 47.4 mm to (49.0, 85.3)
- moved C10 47.4 mm to (64.2, 131.1)
- moved C11 47.4 mm to (64.2, 61.2)
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Routing:
- net /Sheet59972800/Sheet599739F6/C14: track 0.00 -> 69.1 mm, vias 0 -> 2
- net /Sheet59972800/Sheet599739F6/C25: track 0.00 -> 67.6 mm, vias 0 -> 1
- net /Sheet59972800/Sheet59973A04/C17: track 0.00 -> 63.5 mm, vias 0 -> 1
- net /Sheet59972800/Sheet599739F9/C25: track 0.00 -> 62.4 mm, vias 0 -> 1
- net /Sheet59972800/Sheet599739F9/C17: track 0.00 -> 61.9 mm, vias 0 -> 1
- net /Sheet59972800/Sheet599739F6/C17: track 0.00 -> 61.3 mm, vias 0 -> 1
- net /Sheet59972800/Sheet599739FF/C17: track 0.00 -> 61.0 mm
- net /Sheet59972800/Sheet59973A04/C25: track 0.00 -> 61.0 mm, vias 0 -> 1
- net /Sheet59972800/Sheet599739F6/C18: track 0.00 -> 60.9 mm, vias 0 -> 2
- net /Sheet59972800/Sheet599739F9/C18: track 0.00 -> 59.9 mm, vias 0 -> 3
- net /Sheet59972800/Sheet599739FF/C25: track 0.00 -> 59.7 mm
- net /Sheet59972800/Sheet599739FF/C18: track 0.00 -> 59.5 mm
- net /Sheet59972800/Sheet599739F9/C26: track 0.00 -> 58.3 mm, vias 0 -> 2
- net /Sheet59972800/Sheet599739FF/C26: track 0.00 -> 58.3 mm
- net /Sheet59972800/Sheet59973A04/C18: track 0.00 -> 57.6 mm, vias 0 -> 2
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Other:
- copper layers 2 -> 4
- net class Power added: clearance 0.2, trace_width 0.508, via_dia 0.8, via_drill 0.4

Commit message: Include missing terminal block in driver layout
Parts:
- added J58: Screw_Terminal_1x02, Connectors_Terminal_Blocks:TerminalBlock_Pheonix_MKDS1.5-2pol, F.Cu at (72.0, 110.0)
Routing:
- net /Sheet59972800/Sheet59973A04/C1: track 25.2 -> 26.8 mm
Changed lines of the file:
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@@
     (thickness 1.6)
     (drawings 10)
-    (tracks 2843)
+    (tracks 2842)
     (zones 0)
-    (modules 112)
+    (modules 113)
     (nets 209)
   )
@@
     (add_net VCC)
   )
+  (module Connectors_Terminal_Blocks:TerminalBlock_Pheonix_MKDS1.5-2pol (layer F.Cu)
+    (at 72.047 109.982)
+    (descr "2-way 5mm pitch terminal block, Phoenix MKDS series")
+    (fp_text reference J58 (at 2.5 5.9) (layer F.SilkS)
+      (effects (font (size 1 1) (thickness 0.15)))
+    )
+    (fp_text value Screw_Terminal_1x02 (at 2.5 -6.6) (layer F.Fab)
+      (effects (font (size 1 1) (thickness 0.15)))
+    )
+    (fp_line (start -2.7 -5.4) (end 7.7 -5.4) (layer F.CrtYd) (width 0.05))
+    (fp_line (start -2.7 4.8) (end -2.7 -5.4) (layer F.CrtYd) (width 0.05))
+    (fp_line (start 7.7 4.8) (end -2.7 4.8) (layer F.CrtYd) (width 0.05))
+    (fp_line (start 7.7 -5.4) (end 7.7 4.8) (layer F.CrtYd) (width 0.05))
+    (fp_line (start 2.5 4.1) (end 2.5 4.6) (layer F.SilkS) (width 0.15))
+    (fp_circle (center 5 0.1) (end 3 0.1) (layer F.SilkS) (width 0.15))
+    (fp_circle (center 0 0.1) (end 2 0.1) (layer F.SilkS) (width 0.15))
+    (fp_line (start -2.5 2.6) (end 7.5 2.6) (layer F.SilkS) (width 0.15))
+    (fp_line (start -2.5 -2.3) (end 7.5 -2.3) (layer F.SilkS) (width 0.15))
+    (fp_line (start -2.5 4.1) (end 7.5 4.1) (layer F.SilkS) (width 0.15))
+    (fp_line (start -2.5 4.6) (end 7.5 4.6) (layer F.SilkS) (width 0.15))
+    (fp_line (start 7.5 4.6) (end 7.5 -5.2) (layer F.SilkS) (width 0.15))
+    (fp_line (start 7.5 -5.2) (end -2.5 -5.2) (layer F.SilkS) (width 0.15))
+    (fp_line (start -2.5 -5.2) (end -2.5 4.6) (layer F.SilkS) (width 0.15))
+    (pad 1 thru_hole rect (at 0 0) (size 2.5 2.5) (drill 1.3) (layers *.Cu *.Mask)
+      (net 107 /Sheet59972800/Sheet59973A04/C1))
+    (pad 2 thru_hole circle (at 5 0) (size 2.5 2.5) (drill 1.3) (layers *.Cu *.Mask)
+      (net 98 /Sheet59972800/Sheet59973A04/C2))
+    (model Terminal_Blocks.3dshapes/TerminalBlock_Pheonix_MKDS1.5-2pol.wrl
+      (at (xyz 0.0984 0 0))
+      (scale (xyz 1 1 1))
+      (rotate (xyz 0 0 0))
+    )
+  )
   (module Housings_DIP:DIP-16_W7.62mm_LongPads (layer F.Cu)
     (at 112.226 71.36 90)
@@
   (segment (start 99.013 148.844) (end 70.866 148.844) (width 0.25) (layer F.Cu) (net 97))
   (segment (start 102.047 151.878) (end 99.013 148.844) (width 0.25) (layer F.Cu) (net 97))
-  (segment (start 70.765855 112.201842) (end 70.365856 112.601841) (width 0.25) (layer F.Cu) (net 98))
-  (segment (start 70.974685 111.993012) (end 70.765855 112.201842) (width 0.25) (layer F.Cu) (net 98))
-  (segment (start 77.047 109.968) (end 75.021988 111.993012) (width 0.25) (layer F.Cu) (net 98))
+  (segment (start 70.365856 112.601841) (end 70.974685 111.993012) (width 0.25) (layer F.Cu) (net 98))
+  (segment (start 70.974685 111.993012) (end 75.035988 111.993012) (width 0.25) (layer F.Cu) (net 98))
+  (segment (start 75.035988 111.993012) (end 77.047 109.982) (width 0.25) (layer F.Cu) (net 98))
   (segment (start 51.36 110.49) (end 68.254015 110.49) (width 0.25) (layer B.Cu) (net 98))
   (via (at 70.365856 112.601841) (size 0.8) (drill 0.4) (layers F.Cu B.Cu) (net 98))
@@
   (segment (start 48.98 112.87) (end 51.36 110.49) (width 0.25) (layer B.Cu) (net 98))
   (segment (start 48.98 113.27) (end 48.98 112.87) (width 0.25) (layer B.Cu) (net 98))
-  (segment (start 75.021988 111.993012) (end 70.974685 111.993012) (width 0.25) (layer F.Cu) (net 98))
   (segment (start 70.565904 101.121809) (end 70.565904 100.556124) (width 0.25) (layer F.Cu) (net 99))
   (segment (start 70.565904 102.794734) (end 70.565904 101.121809) (width 0.25) (layer F.Cu) (net 99))
@@
   (segment (start 64.22 113.27) (end 64.22 113.67) (width 0.25) (layer B.Cu) (net 106))
   (segment (start 64.22 113.67) (end 67.136 116.586) (width 0.25) (layer B.Cu) (net 106))
-  (segment (start 71.665998 108.204) (end 71.783 108.204) (width 0.25) (layer B.Cu) (net 107))
-  (segment (start 71.783 108.204) (end 72.047 108.468) (width 0.25) (layer B.Cu) (net 107))
-  (segment (start 72.047 108.468) (end 72.047 109.968) (width 0.25) (layer B.Cu) (net 107))
-  (segment (start 71.265999 107.804001) (end 71.665998 108.204) (width 0.25) (layer B.Cu) (net 107))
   (segment (start 69.342 108.204) (end 69.741999 107.804001) (width 0.25) (layer B.Cu) (net 107))
-  (segment (start 69.741999 107.804001) (end 71.265999 107.804001) (width 0.25) (layer B.Cu) (net 107))
+  (segment (start 69.741999 107.804001) (end 71.482001 107.804001) (width 0.25) (layer B.Cu) (net 107))
+  (segment (start 71.482001 107.804001) (end 72.047 108.369) (width 0.25) (layer B.Cu) (net 107))
+  (segment (start 72.047 108.369) (end 72.047 108.468) (width 0.25) (layer B.Cu) (net 107))
+  (segment (start 72.047 108.468) (end 72.047 109.982) (width 0.25) (layer B.Cu) (net 107))
+  (segment (start 72.047 108.468) (end 72.047 109.968) (width 0.25) (layer B.Cu) (net 107))
   (segment (start 55.47 110) (end 67.546 110) (width 0.25) (layer F.Cu) (net 107))
   (via (at 69.342 108.204) (size 0.8) (drill 0.4) (layers F.Cu B.Cu) (net 107))

Commit message: Multple commits enclosed in this commit.
1.Design passes all DRC tests.
2.Add PMOS reverse polarity protection on 5v direct input.
Parts:
- added D2: D_Zener, Diodes_THT:D_T-1_P5.08mm_Horizontal, F.Cu at (41.1, 103.1)
- added J73: GS2, Connectors:GS2, F.Cu at (42.2, 99.6)
- added J74: GS2, Connectors:GS2, F.Cu at (44.2, 99.6)
- added Q1: Q_PMOS_GDS, TO_SOT_Packages_THT:TO-220_Neutral123_Vertical_LargePads, F.Cu at (36.8, 96.5)
- added R10: 10k, Resistors_THT:R_Axial_DIN0207_L6.3mm_D2.5mm_P7.62mm_Horizontal, F.Cu at (38.1, 103.1)
- added R2: R, Resistors_THT:R_Axial_DIN0207_L6.3mm_D2.5mm_P7.62mm_Horizontal, F.Cu at (96.8, 33.5)
- added R3: R, Resistors_THT:R_Axial_DIN0207_L6.3mm_D2.5mm_P7.62mm_Horizontal, F.Cu at (101.3, 33.5)
- added R4: R, Resistors_THT:R_Axial_DIN0207_L6.3mm_D2.5mm_P7.62mm_Horizontal, F.Cu at (105.7, 33.5)
- added R5: R, Resistors_THT:R_Axial_DIN0207_L6.3mm_D2.5mm_P7.62mm_Horizontal, F.Cu at (110.2, 33.5)
- added R6: R, Resistors_THT:R_Axial_DIN0207_L6.3mm_D2.5mm_P7.62mm_Horizontal, F.Cu at (114.8, 33.5)
- added R7: R, Resistors_THT:R_Axial_DIN0207_L6.3mm_D2.5mm_P7.62mm_Horizontal, F.Cu at (119.4, 33.5)
- added R8: R, Resistors_THT:R_Axial_DIN0207_L6.3mm_D2.5mm_P7.62mm_Horizontal, F.Cu at (123.7, 33.5)
- added R9: R, Resistors_THT:R_Axial_DIN0207_L6.3mm_D2.5mm_P7.62mm_Horizontal, F.Cu at (128.0, 33.5)
- C10, C11, C12, C13, C14, C15, C16, C17, C18, C3, C4, C5, C6, C7, C8, C9: value C -> 10nF
- moved J70 37.8 mm to (165.1, 36.8)
- moved J71 37.8 mm to (145.1, 36.8)
- moved J69 37.8 mm to (155.1, 36.8)
- moved J72 37.8 mm to (135.1, 36.8)
- moved J3 8.69 mm to (29.8, 160.8)
- moved C18 1.06 mm to (127.5, 47.0)
Connections:
- J1 pad 1: 5v -> /INPUT_5V
- J2 pad 1: 5v -> /INPUT_5V
- J3 pad 2: Net-(J3-Pad2) -> GND
- U10 pad 16: VCC -> 5v
- U11 pad 16: VCC -> 5v
- U12 pad 16: VCC -> 5v
- U13 pad 16: VCC -> 5v
- U14 pad 16: VCC -> 5v
- U15 pad 16: VCC -> 5v
- U16 pad 16: VCC -> 5v
- U17 pad 16: VCC -> 5v
- U18 pad 16: VCC -> 5v
- U19 pad 16: VCC -> 5v
- U20 pad 11: /Sheet599728AA/R8 -> Net-(R9-Pad1)
- U20 pad 12: /Sheet599728AA/R7 -> Net-(R8-Pad1)
- U20 pad 13: /Sheet599728AA/R6 -> Net-(R7-Pad1)
- U20 pad 14: /Sheet599728AA/R5 -> Net-(R6-Pad1)
- U20 pad 15: /Sheet599728AA/R4 -> Net-(R5-Pad1)
- U20 pad 16: /Sheet599728AA/R3 -> Net-(R4-Pad1)
- U20 pad 17: /Sheet599728AA/R2 -> Net-(R3-Pad1)
- U20 pad 18: /Sheet599728AA/R1 -> Net-(R2-Pad1)
- U3 pad 2: Net-(J3-Pad2) -> GND
- U3 pad 3: 5v -> /INPUT_5V
- U4 pad 16: VCC -> 5v
- U5 pad 16: VCC -> 5v
- U6 pad 16: VCC -> 5v
- U7 pad 16: VCC -> 5v
- U8 pad 16: VCC -> 5v
- U9 pad 16: VCC -> 5v
Routing:
- net /INPUT_5V: track 0.00 -> 61.8 mm
- net Net-(R9-Pad1): track 0.00 -> 59.5 mm, vias 0 -> 3
- net Net-(R8-Pad1): track 0.00 -> 53.5 mm, vias 0 -> 2
- net /Sheet599728AA/R8: track 0.00 -> 48.8 mm
- net /Sheet599728AA/R5: track 0.00 -> 47.2 mm
- net /Sheet599728AA/R7: track 0.00 -> 46.6 mm, vias 0 -> 2
- net Net-(R6-Pad1): track 0.00 -> 46.6 mm
- net 5v: track 0.00 -> 46.3 mm
- net /Sheet599728AA/R1: track 0.00 -> 46.2 mm
- net /Sheet599728AA/R4: track 0.00 -> 46.1 mm
- net /Sheet599728AA/R3: track 0.00 -> 46.0 mm
- net /Sheet599728AA/R6: track 0.00 -> 45.8 mm, vias 0 -> 1
- net Net-(R7-Pad1): track 0.00 -> 44.7 mm, vias 0 -> 1
- net /Sheet599728AA/R2: track 0.00 -> 44.5 mm, vias 0 -> 1
- net Net-(R5-Pad1): track 0.00 -> 36.0 mm
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- added copper zone on VCC.Cu, net 5v
- added copper zone on GND.Cu, net GND
Other:
- board text added: "5v"
- board text added: "GND"
