File: hardware/drivers/ND-03/ND-03.kicad_pcb (KiCad board)
At the start: 4 copper layers, 155.6 x 134.7 mm, 126 parts, among them J1 Screw_Terminal_1x02, J10 Screw_Terminal_1x02, J11 Screw_Terminal_1x02, J12 Screw_Terminal_1x02, J13 Screw_Terminal_1x02, J14 Screw_Terminal_1x02, J15 Screw_Terminal_1x02, J16 Screw_Terminal_1x02, J17 Screw_Terminal_1x02, J18 Screw_Terminal_1x02, J19 Screw_Terminal_1x02, J2 Screw_Terminal_1x02, J20 Screw_Terminal_1x02, J21 Screw_Terminal_1x02, J22 Screw_Terminal_1x02, J23 Screw_Terminal_1x02, J24 Screw_Terminal_1x02, J25 Screw_Terminal_1x02, J26 Screw_Terminal_1x02, J27 Screw_Terminal_1x02, J28 Screw_Terminal_1x02, J29 Screw_Terminal_1x02, J3 Screw_Terminal_1x02, J30 Screw_Terminal_1x02, J31 Screw_Terminal_1x02, J32 Screw_Terminal_1x02, J33 Screw_Terminal_1x02, J34 Screw_Terminal_1x02, J35 Screw_Terminal_1x02, J36 Screw_Terminal_1x02, J37 Screw_Terminal_1x02, J38 Screw_Terminal_1x02, J39 Screw_Terminal_1x02, J4 Screw_Terminal_1x02, J40 Screw_Terminal_1x02, J41 Screw_Terminal_1x02, J42 Screw_Terminal_1x02, J43 Screw_Terminal_1x02, J44 Screw_Terminal_1x02, J45 Screw_Terminal_1x02, J46 Screw_Terminal_1x02, J47 Screw_Terminal_1x02, J48 Screw_Terminal_1x02, J49 Screw_Terminal_1x02, J5 Screw_Terminal_1x02, J50 Screw_Terminal_1x02, J51 Screw_Terminal_1x02, J52 Screw_Terminal_1x02, J53 Screw_Terminal_1x02, J54 Screw_Terminal_1x02, J55 Screw_Terminal_1x02, J56 Screw_Terminal_1x02, J57 Screw_Terminal_1x02, J58 Screw_Terminal_1x02, J59 Screw_Terminal_1x02, J6 Screw_Terminal_1x02, J60 Screw_Terminal_1x02, J61 Screw_Terminal_1x02, J62 Screw_Terminal_1x02, J63 Screw_Terminal_1x02, J64 Screw_Terminal_1x02, J65 Screw_Terminal_1x02, J66 Screw_Terminal_1x02, J67 Screw_Terminal_1x02, J68 GS3, J69 Screw_Terminal_1x02, J7 Screw_Terminal_1x02, J70 Screw_Terminal_1x02, J71 Screw_Terminal_1x02, J72 Screw_Terminal_1x02, J73 GS2, J74 GS2, J8 Screw_Terminal_1x02, J9 Screw_Terminal_1x02, Q1 Q_PMOS_GDS, U1 ESP-32-module, U10 74HC595, U11 74HC595, U12 74HC595, U13 74HC595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

Commit message: Add mounting holes
Parts:
- added REF**: MountingHole_3.2mm_M3_ISO7380, Mounting_Holes:MountingHole_3.2mm_M3_ISO7380, F.Cu at (169.0, 45.0)
- added REF**: MountingHole_3.2mm_M3_ISO7380, Mounting_Holes:MountingHole_3.2mm_M3_ISO7380, F.Cu at (169.0, 162.0)
- added REF**: MountingHole_3.2mm_M3_ISO7380, Mounting_Holes:MountingHole_3.2mm_M3_ISO7380, F.Cu at (22.5, 162.0)
Changed lines of the file:
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@@
     (tracks 3092)
     (zones 0)
-    (modules 126)
+    (modules 129)
     (nets 217)
   )
@@
     (add_net "Net-(R9-Pad1)")
   )
+  (module Mounting_Holes:MountingHole_3.2mm_M3_ISO7380 (layer F.Cu)
+    (at 169 45)
+    (descr "Mounting Hole 3.2mm, no annular, M3, ISO7380")
+    (tags "mounting hole 3.2mm no annular m3 iso7380")
+    (fp_text reference REF** (at 0 -3.85) (layer Dwgs.User)
+      (effects (font (size 1 1) (thickness 0.15)))
+    )
+    (fp_text value MountingHole_3.2mm_M3_ISO7380 (at 0 3.85) (layer F.Fab)
+      (effects (font (size 1 1) (thickness 0.15)))
+    )
+    (fp_circle (center 0 0) (end 3.1 0) (layer F.CrtYd) (width 0.05))
+    (fp_circle (center 0 0) (end 2.85 0) (layer Cmts.User) (width 0.15))
+    (pad 1 np_thru_hole circle (at 0 0) (size 3.2 3.2) (drill 3.2) (layers *.Cu *.Mask))
+  )
+  (module Mounting_Holes:MountingHole_3.2mm_M3_ISO7380 (layer F.Cu)
+    (at 169 162)
+    (descr "Mounting Hole 3.2mm, no annular, M3, ISO7380")
+    (tags "mounting hole 3.2mm no annular m3 iso7380")
+    (fp_text reference REF** (at 0 -3.85) (layer Dwgs.User)
+      (effects (font (size 1 1) (thickness 0.15)))
+    )
+    (fp_text value MountingHole_3.2mm_M3_ISO7380 (at 0 3.85) (layer F.Fab)
+      (effects (font (size 1 1) (thickness 0.15)))
+    )
+    (fp_circle (center 0 0) (end 3.1 0) (layer F.CrtYd) (width 0.05))
+    (fp_circle (center 0 0) (end 2.85 0) (layer Cmts.User) (width 0.15))
+    (pad 1 np_thru_hole circle (at 0 0) (size 3.2 3.2) (drill 3.2) (layers *.Cu *.Mask))
+  )
+  (module Mounting_Holes:MountingHole_3.2mm_M3_ISO7380 (layer F.Cu)
+    (at 22.5 162)
+    (descr "Mounting Hole 3.2mm, no annular, M3, ISO7380")
+    (tags "mounting hole 3.2mm no annular m3 iso7380")
+    (fp_text reference REF** (at 0 -3.85) (layer Dwgs.User) hide
+      (effects (font (size 1 1) (thickness 0.15)))
+    )
+    (fp_text value MountingHole_3.2mm_M3_ISO7380 (at 0 3.85) (layer F.Fab)
+      (effects (font (size 1 1) (thickness 0.15)))
+    )
+    (fp_circle (center 0 0) (end 3.1 0) (layer F.CrtYd) (width 0.05))
+    (fp_circle (center 0 0) (end 2.85 0) (layer Cmts.User) (width 0.15))
+    (pad 1 np_thru_hole circle (at 0 0) (size 3.2 3.2) (drill 3.2) (layers *.Cu *.Mask))
+  )
   (module Resistors_THT:R_Axial_DIN0207_L6.3mm_D2.5mm_P7.62mm_Horizontal (layer F.Cu)
     (at 38.1 103.124 180)
@@
     (at 29.798 160.782)
     (descr "2-way 5mm pitch terminal block, Phoenix MKDS series")
-    (fp_text reference J3 (at 2.5 5.9) (layer F.SilkS)
+    (fp_text reference J3 (at 9.202 3.218) (layer F.SilkS)
       (effects (font (size 1 1) (thickness 0.15)))
     )
@@
     )
   )
+  (gr_line (start 17.865 31.101) (end 17.865 165.848) (layer Edge.Cuts) (width 0.15))
   (gr_circle (center 20.32 63.5) (end 21.336 63.754) (layer F.SilkS) (width 0.2))
   (gr_line (start 34.798 159.258) (end 34.798 155.194) (layer F.SilkS) (width 0.2))
@@
     (effects (font (size 1.5 1.5) (thickness 0.3)))
   )
-  (gr_line (start 17.865 31.101) (end 17.865 165.848) (layer Edge.Cuts) (width 0.15))
   (dimension 134.747 (width 0.3) (layer Dwgs.User)
     (gr_text "134.747 mm" (at 185.585 98.4745 270) (layer Dwgs.User)

Commit message: Add ND-03 gerbers folder and zip
Parts:
- added G***: NARRA, logos:narra_logo, F.Cu at (30.5, 53.3)
Routing:
- net GND: vias 17 -> 262
- added copper zone on B.Cu, net GND
- added copper zone on F.Cu, net GND
