File: hardware/drivers/ND-03/ND-03.sch (KiCad schematic (older format))
At the start: 10 parts, among them J1 Screw_Terminal_1x02, J2 Screw_Terminal_1x02, J3 Screw_Terminal_1x02, U1 ESP-32-module, U2 LD1117S33TR_SOT223, U3 LM2596_MODULE

Commit message: Multple commits enclosed in this commit.
1.Design passes all DRC tests.
2.Add PMOS reverse polarity protection on 5v direct input.
Parts:
- added D2: D_Zener, Diodes_THT:D_T-1_P5.08mm_Horizontal, symbol D_Zener
- added J73, J74: GS2, Connectors:GS2, symbol GS2
- added Q1: Q_PMOS_GDS, TO_SOT_Packages_THT:TO-220_Neutral123_Vertical_LargePads, symbol Q_PMOS_GDS
- added R10: 10k, Resistors_THT:R_Axial_DIN0207_L6.3mm_D2.5mm_P7.62mm_Horizontal, symbol R
Connections:
- net 5v: now also D2.1 (K), J73.1 (G1), J74.1 (G1), Q1.3 (S); no longer J1.1, J2.1, U3.3 (OUT+)
- net GND: now also J3.2, U3.2 (IN-), R10.2
- new net: D2.2 (A), Q1.1 (G), R10.1
- new net INPUT_5V: J1.1, J2.1, J73.2 (G2), J74.2 (G2), Q1.2 (D), U3.3 (OUT+)
Other:
- note added: "REVERSE POLARITY \nPROTECTION FOR DIRECT \n5V CONNECTION"
Changed lines of the file:
@@
 	1    0    0    -1
 $EndComp
-Wire Notes Line
-	11220 3320 470  3320
-Wire Notes Line
-	11220 5050 470  5050
-Wire Wire Line
-	2870 1550 2960 1550
-Wire Wire Line
-	2870 1690 2960 1690
-Wire Wire Line
-	7460 1300 7290 1300
-Wire Wire Line
-	7460 1460 7300 1460
-Wire Wire Line
-	7460 1620 7310 1620
-Wire Wire Line
-	7130 3880 7850 3880
-Wire Wire Line
-	8450 3880 9000 3880
-Wire Wire Line
-	8150 4250 8150 4180
-Wire Wire Line
-	7600 4330 7600 4260
-Wire Wire Line
-	7600 4650 7600 4630
-Wire Wire Line
-	7600 3960 7600 3880
-Connection ~ 7600 3880
-Wire Wire Line
-	7300 3960 7300 3880
-Connection ~ 7300 3880
-Wire Wire Line
-	8750 3950 8750 3880
-Connection ~ 8750 3880
-Wire Wire Line
-	8750 4250 8750 4640
-Wire Wire Line
-	7300 4660 7300 4260
-Wire Wire Line
-	3860 900  4340 900
-Wire Wire Line
-	4090 2320 4090 2300
-Wire Wire Line
-	4090 2300 4340 2300
-Wire Wire Line
-	6440 910  6440 900
-Wire Wire Line
-	6440 900  6140 900
-Wire Notes Line
-	5310 3320 5310 5050
-Wire Wire Line
-	4160 1000 4340 1000
-Wire Wire Line
-	4340 1800 4280 1800
-Wire Wire Line
-	4340 1900 4280 1900
-Wire Wire Line
-	4340 2000 4280 2000
-Wire Wire Line
-	4340 2100 4280 2100
-Wire Wire Line
-	4340 2200 4280 2200
-Wire Notes Line
-	6970 6540 6970 5050
 Text Notes 11220 6540 2    60   ~ 0
 DC-DC converter
@@
 	0    -1   -1   0
 $EndComp
-Wire Wire Line
-	2160 4120 2160 4040
-Wire Wire Line
-	2360 3890 2360 4120
-Wire Wire Line
-	3580 3970 3580 4120
-Wire Wire Line
-	3780 3840 3780 4120
-Text GLabel 2160 4040 1    60   Input ~ 0
-5v
 $Comp
 L GND #PWR08
@@
 	1    0    0    -1
 $EndComp
-Wire Wire Line
-	2500 3890 2360 3890
-Text GLabel 3580 3970 1    60   Input ~ 0
-5v
 $Comp
 L GND #PWR09
@@
 	1    0    0    -1
 $EndComp
-Wire Wire Line
-	3990 3900 3990 3840
-Wire Wire Line
-	3990 3840 3780 3840
 Text Notes 5310 5050 2    60   ~ 0
 DIRECT 5V CONNECTION
@@
 	1    0    0    -1
 $EndComp
-Wire Wire Line
-	8090 5410 7840 5410
 $Comp
 L Screw_Terminal_1x02 J3
@@
 	1    0    0    -1
 $EndComp
-Wire Wire Line
-	7630 5610 7840 5610
-Wire Wire Line
-	7840 5610 7840 5410
-Wire Wire Line
-	7630 5810 7850 5810
-Wire Wire Line
-	7850 5810 7850 6010
-Wire Wire Line
-	7850 6010 8090 6010
-Wire Wire Line
-	10240 5410 10380 5410
-Text GLabel 10380 5410 2    60   Input ~ 0
-5v
 $Comp
 L GND #PWR010
@@
 	1    0    0    -1
 $EndComp
-Wire Wire Line
-	10400 6040 10400 6010
-Wire Wire Line
-	10400 6010 10240 6010
 Text GLabel 4160 1000 0    60   Input ~ 0
 3v3
@@
 NoConn ~ 6140 1100
 NoConn ~ 6140 1000
+$Comp
+L Q_PMOS_GDS Q1
+U 1 1 59A57239
+P 6240 5720
+F 0 "Q1" V 6210 5880 50  0000 C CNN
+F 1 "Q_PMOS_GDS" V 6120 5990 50  0000 C CNN
+F 2 "TO_SOT_Packages_THT:TO-220_Neutral123_Vertical_LargePads" H 6440 5820 50  0001 C CNN
+F 3 "" H 6240 5720 50  0001 C CNN
+	1    6240 5720
+	0    -1   -1   0
+$EndComp
+Text Label 3460 3840 2    60   ~ 0
+INPUT_5V
+Text Label 2050 3890 2    60   ~ 0
+INPUT_5V
+Text Label 5810 5620 2    60   ~ 0
+INPUT_5V
+Text Label 10380 5410 0    60   ~ 0
+INPUT_5V
+Text GLabel 6610 5620 2    60   Input ~ 0
+5v
+$Comp
+L GND #PWR011
+U 1 1 59A59685
+P 6240 6300
+F 0 "#PWR011" H 6240 6050 50  0001 C CNN
+F 1 "GND" H 6245 6127 50  0000 C CNN
+F 2 "" H 6240 6300 50  0001 C CNN
+F 3 "" H 6240 6300 50  0001 C CNN
+	1    6240 6300
+	1    0    0    -1
+$EndComp
+$Comp
+L R R10
+U 1 1 59A59F39
+P 6240 6090
+F 0 "R10" H 6310 6136 50  0000 L CNN
+F 1 "10k" H 6310 6045 50  0000 L CNN
+F 2 "Resistors_THT:R_Axial_DIN0207_L6.3mm_D2.5mm_P7.62mm_Horizontal" V 6170 6090 50  0001 C CNN
+F 3 "" H 6240 6090 50  0001 C CNN
+	1    6240 6090
+	1    0    0    -1
+$EndComp
+Text Notes 5310 6540 0    60   ~ 0
+REVERSE POLARITY \nPROTECTION FOR  DIRECT \n5V CONNECTION
+$Comp
+L D_Zener D2
+U 1 1 59A5BD86
+P 6520 5780
+F 0 "D2" V 6474 5859 50  0000 L CNN
+F 1 "D_Zener" V 6565 5859 50  0000 L CNN
+F 2 "Diodes_THT:D_T-1_P5.08mm_Horizontal" H 6520 5780 50  0001 C CNN
+F 3 "" H 6520 5780 50  0001 C CNN
+	1    6520 5780
+	0    1    1    0
+$EndComp
+$Comp
+L GS2 J73
+U 1 1 59A5DC35
+P 6240 5210
+F 0 "J73" V 6170 5360 50  0000 C CNN
+F 1 "GS2" V 6170 5030 50  0000 C CNN
+F 2 "Connectors:GS2" V 6314 5210 50  0001 C CNN
+F 3 "" H 6240 5210 50  0001 C CNN
+	1    6240 5210
+	0    1    1    0
+$EndComp
+$Comp
+L GS2 J74
+U 1 1 59A5DF25
+P 6240 5300
+F 0 "J74" V 6290 5450 50  0000 C CNN
+F 1 "GS2" V 6290 5120 50  0000 C CNN
+F 2 "Connectors:GS2" V 6314 5300 50  0001 C CNN
+F 3 "" H 6240 5300 50  0001 C CNN
+	1    6240 5300
+	0    1    1    0
+$EndComp
+$Comp
+L GND #PWR012
+U 1 1 59A60C96
+P 7660 5860
+F 0 "#PWR012" H 7660 5610 50  0001 C CNN
+F 1 "GND" H 7665 5687 50  0000 C CNN
+F 2 "" H 7660 5860 50  0001 C CNN
+F 3 "" H 7660 5860 50  0001 C CNN
+	1    7660 5860
+	1    0    0    -1
+$EndComp
+Wire Notes Line
+	11220 3320 470  3320
+Wire Notes Line
+	11220 5050 470  5050
+Wire Wire Line
+	2870 1550 2960 1550
+Wire Wire Line
+	2870 1690 2960 1690
+Wire Wire Line
+	7460 1300 7290 1300
+Wire Wire Line
+	7460 1460 7300 1460
+Wire Wire Line
+	7460 1620 7310 1620
+Wire Wire Line
+	7130 3880 7850 3880
+Wire Wire Line
+	8450 3880 9000 3880
+Wire Wire Line
+	8150 4250 8150 4180
+Wire Wire Line
+	7600 4330 7600 4260
+Wire Wire Line
+	7600 4650 7600 4630
+Wire Wire Line
+	7600 3960 7600 3880
+Connection ~ 7600 3880
+Wire Wire Line
+	7300 3960 7300 3880
+Connection ~ 7300 3880
+Wire Wire Line
+	8750 3950 8750 3880
+Connection ~ 8750 3880
+Wire Wire Line
+	8750 4250 8750 4640
+Wire Wire Line
+	7300 4660 7300 4260
+Wire Wire Line
+	3860 900  4340 900
+Wire Wire Line
+	4090 2320 4090 2300
+Wire Wire Line
+	4090 2300 4340 2300
+Wire Wire Line
+	6440 910  6440 900
+Wire Wire Line
+	6440 900  6140 900
+Wire Notes Line
+	5310 3320 5310 6540
+Wire Wire Line
+	4160 1000 4340 1000
+Wire Wire Line
+	4340 1800 4280 1800
+Wire Wire Line
+	4340 1900 4280 1900
+Wire Wire Line
+	4340 2000 4280 2000
+Wire Wire Line
+	4340 2100 4280 2100
+Wire Wire Line
+	4340 2200 4280 2200
+Wire Notes Line
+	6970 6540 6970 5050
+Wire Wire Line
+	2160 3890 2160 4120
+Wire Wire Line
+	2360 3890 2360 4120
+Wire Wire Line
+	3580 3840 3580 4120
+Wire Wire Line
+	3780 3840 3780 4120
+Wire Wire Line
+	2500 3890 2360 3890
+Wire Wire Line
+	3990 3900 3990 3840
+Wire Wire Line
+	3990 3840 3780 3840
+Wire Wire Line
+	8090 5410 7840 5410
+Wire Wire Line
+	7630 5610 7840 5610
+Wire Wire Line
+	7840 5610 7840 5410
+Wire Wire Line
+	7630 5810 7850 5810
+Wire Wire Line
+	7850 5810 7850 6010
+Wire Wire Line
+	7850 6010 8090 6010
+Wire Wire Line
+	10240 5410 10380 5410
+Wire Wire Line
+	10400 6040 10400 6010
+Wire Wire Line
+	10400 6010 10240 6010
+Wire Notes Line
+	6970 6540 470  6540
+Wire Wire Line
+	5810 5620 6040 5620
+Wire Wire Line
+	2160 3890 2050 3890
+Wire Wire Line
+	3580 3840 3460 3840
+Wire Wire Line
+	6240 5940 6240 5920
+Wire Wire Line
+	6240 6300 6240 6240
+Wire Wire Line
+	6520 5930 6240 5930
+Connection ~ 6240 5930
+Wire Wire Line
+	6520 5210 6520 5630
+Wire Wire Line
+	6040 5300 5960 5300
+Connection ~ 5960 5620
+Wire Wire Line
+	5960 5210 6040 5210
+Connection ~ 5960 5300
+Wire Wire Line
+	5960 5210 5960 5620
+Wire Wire Line
+	7660 5860 7660 5810
+Connection ~ 7660 5810
+Wire Wire Line
+	6440 5620 6610 5620
+Connection ~ 6520 5620
+Wire Wire Line
+	6440 5300 6520 5300
+Connection ~ 6520 5300
+Wire Wire Line
+	6440 5210 6520 5210
 $EndSCHEMATC
