File: hardware/drivers/ND-03/column1_32.sch (KiCad schematic (older format))
At the start: 24 parts, among them J10 Screw_Terminal_1x02, J11 Screw_Terminal_1x02, J12 Screw_Terminal_1x02, J13 Screw_Terminal_1x02, J14 Screw_Terminal_1x02, J15 Screw_Terminal_1x02, J16 Screw_Terminal_1x02, J17 Screw_Terminal_1x02, J18 Screw_Terminal_1x02, J19 Screw_Terminal_1x02, J4 Screw_Terminal_1x02, J5 Screw_Terminal_1x02, J6 Screw_Terminal_1x02, J7 Screw_Terminal_1x02, J8 Screw_Terminal_1x02, J9 Screw_Terminal_1x02, U4 74HC595, U5 74HC595, U6 74HC595, U7 74HC595

Commit message: Multple commits enclosed in this commit.
1.Design passes all DRC tests.
2.Add PMOS reverse polarity protection on 5v direct input.
Parts:
- C3, C4, C5, C6: value C -> 10nF
Connections:
- net 5v is gone; now on net VCC: C3.1, C4.1, C5.1, C6.1, U4.10 (SRCLR), U5.10 (SRCLR), U6.10 (SRCLR), U7.10 (SRCLR)
Changed lines of the file:
@@
 5v
 $Comp
-L GND #PWR011
+L GND #PWR013
 U 1 1 5998E76C
 P 1640 1800
-F 0 "#PWR011" H 1640 1550 50  0001 C CNN
+F 0 "#PWR013" H 1640 1550 50  0001 C CNN
 F 1 "GND" H 1645 1627 50  0000 C CNN
 F 2 "" H 1640 1800 50  0001 C CNN
@@
 $EndComp
 $Comp
-L GND #PWR012
+L GND #PWR014
 U 1 1 5998E84C
 P 3690 1810
-F 0 "#PWR012" H 3690 1560 50  0001 C CNN
+F 0 "#PWR014" H 3690 1560 50  0001 C CNN
 F 1 "GND" H 3695 1637 50  0000 C CNN
 F 2 "" H 3690 1810 50  0001 C CNN
@@
 $EndComp
 $Comp
-L GND #PWR013
+L GND #PWR015
 U 1 1 5998EAA8
 P 5840 1840
-F 0 "#PWR013" H 5840 1590 50  0001 C CNN
+F 0 "#PWR015" H 5840 1590 50  0001 C CNN
 F 1 "GND" H 5845 1667 50  0000 C CNN
 F 2 "" H 5840 1840 50  0001 C CNN
@@
 $EndComp
 $Comp
-L GND #PWR014
+L GND #PWR016
 U 1 1 5998ED65
 P 8100 1830
-F 0 "#PWR014" H 8100 1580 50  0001 C CNN
+F 0 "#PWR016" H 8100 1580 50  0001 C CNN
 F 1 "GND" H 8105 1657 50  0000 C CNN
 F 2 "" H 8100 1830 50  0001 C CNN
@@
 5v
 $Comp
-L C C3
-U 1 1 59996F55
-P 2950 7160
-F 0 "C3" H 3065 7206 50  0000 L CNN
-F 1 "C" H 3065 7115 50  0000 L CNN
-F 2 "Capacitors_THT:C_Disc_D3.4mm_W2.1mm_P2.50mm" H 2988 7010 50  0001 C CNN
-F 3 "" H 2950 7160 50  0001 C CNN
-	1    2950 7160
-	1    0    0    -1
-$EndComp
-$Comp
 L C C4
 U 1 1 59997009
 P 3250 7160
 F 0 "C4" H 3365 7206 50  0000 L CNN
-F 1 "C" H 3365 7115 50  0000 L CNN
+F 1 "10nF" H 3365 7115 50  0000 L CNN
 F 2 "Capacitors_THT:C_Disc_D3.4mm_W2.1mm_P2.50mm" H 3288 7010 50  0001 C CNN
 F 3 "" H 3250 7160 50  0001 C CNN
@@
 P 3560 7160
 F 0 "C5" H 3675 7206 50  0000 L CNN
-F 1 "C" H 3675 7115 50  0000 L CNN
+F 1 "10nF" H 3675 7115 50  0000 L CNN
 F 2 "Capacitors_THT:C_Disc_D3.4mm_W2.1mm_P2.50mm" H 3598 7010 50  0001 C CNN
 F 3 "" H 3560 7160 50  0001 C CNN
@@
 P 3880 7160
 F 0 "C6" H 3995 7206 50  0000 L CNN
-F 1 "C" H 3995 7115 50  0000 L CNN
+F 1 "10nF" H 3995 7115 50  0000 L CNN
 F 2 "Capacitors_THT:C_Disc_D3.4mm_W2.1mm_P2.50mm" H 3918 7010 50  0001 C CNN
 F 3 "" H 3880 7160 50  0001 C CNN
@@
 Wire Wire Line
 	3880 7010 2830 7010
-Connection ~ 2950 7010
 Connection ~ 3250 7010
 Connection ~ 3560 7010
@@
 5v
 $Comp
-L GND #PWR015
+L GND #PWR017
 U 1 1 599984DE
 P 2820 7310
-F 0 "#PWR015" H 2820 7060 50  0001 C CNN
+F 0 "#PWR017" H 2820 7060 50  0001 C CNN
 F 1 "GND" H 2825 7137 50  0000 C CNN
 F 2 "" H 2820 7310 50  0001 C CNN
@@
 DECOUPLING CAPS\n
 $Comp
-L PWR_FLAG #FLG016
-U 1 1 599B94F2
-P 2950 7010
-F 0 "#FLG016" H 2950 7085 50  0001 C CNN
-F 1 "PWR_FLAG" H 2950 7184 50  0000 C CNN
-F 2 "" H 2950 7010 50  0001 C CNN
-F 3 "" H 2950 7010 50  0001 C CNN
-	1    2950 7010
-	1    0    0    -1
-$EndComp
+L C C3
+U 1 1 59996F55
+P 2950 7160
+F 0 "C3" H 3065 7206 50  0000 L CNN
+F 1 "10nF" H 3065 7115 50  0000 L CNN
+F 2 "Capacitors_THT:C_Disc_D3.4mm_W2.1mm_P2.50mm" H 2988 7010 50  0001 C CNN
+F 3 "" H 2950 7160 50  0001 C CNN
+	1    2950 7160
+	1    0    0    -1
+$EndComp
+Wire Wire Line
+	2950 7010 2950 6960
+Connection ~ 2950 7010
+$Comp
+L VCC #PWR018
+U 1 1 59A69BDF
+P 2950 6960
+F 0 "#PWR018" H 2950 6810 50  0001 C CNN
+F 1 "VCC" H 2967 7133 50  0000 C CNN
+F 2 "" H 2950 6960 50  0001 C CNN
+F 3 "" H 2950 6960 50  0001 C CNN
+	1    2950 6960
+	1    0    0    -1
+$EndComp
