File: hardware/drivers/ND-03/column33_64.sch (KiCad schematic (older format))
At the start: 24 parts, among them J20 Screw_Terminal_1x02, J21 Screw_Terminal_1x02, J22 Screw_Terminal_1x02, J23 Screw_Terminal_1x02, J24 Screw_Terminal_1x02, J25 Screw_Terminal_1x02, J26 Screw_Terminal_1x02, J27 Screw_Terminal_1x02, J28 Screw_Terminal_1x02, J29 Screw_Terminal_1x02, J30 Screw_Terminal_1x02, J31 Screw_Terminal_1x02, J32 Screw_Terminal_1x02, J33 Screw_Terminal_1x02, J34 Screw_Terminal_1x02, J35 Screw_Terminal_1x02, U10 74HC595, U11 74HC595, U8 74HC595, U9 74HC595

Commit message: Multple commits enclosed in this commit.
1.Design passes all DRC tests.
2.Add PMOS reverse polarity protection on 5v direct input.
Parts:
- C10, C7, C8, C9: value C -> 10nF
Connections:
- net 5v is gone; now on net VCC: C10.1, C7.1, C8.1, C9.1, U10.10 (SRCLR), U11.10 (SRCLR), U8.10 (SRCLR), U9.10 (SRCLR)
Changed lines of the file:
@@
 5v
 $Comp
-L GND #PWR017
+L GND #PWR019
 U 1 1 59992539
 P 1660 1810
-F 0 "#PWR017" H 1660 1560 50  0001 C CNN
+F 0 "#PWR019" H 1660 1560 50  0001 C CNN
 F 1 "GND" H 1665 1637 50  0000 C CNN
 F 2 "" H 1660 1810 50  0001 C CNN
@@
 $EndComp
 $Comp
-L GND #PWR018
+L GND #PWR020
 U 1 1 5999253F
 P 3710 1820
-F 0 "#PWR018" H 3710 1570 50  0001 C CNN
+F 0 "#PWR020" H 3710 1570 50  0001 C CNN
 F 1 "GND" H 3715 1647 50  0000 C CNN
 F 2 "" H 3710 1820 50  0001 C CNN
@@
 $EndComp
 $Comp
-L GND #PWR019
+L GND #PWR021
 U 1 1 59992545
 P 5860 1850
-F 0 "#PWR019" H 5860 1600 50  0001 C CNN
+F 0 "#PWR021" H 5860 1600 50  0001 C CNN
 F 1 "GND" H 5865 1677 50  0000 C CNN
 F 2 "" H 5860 1850 50  0001 C CNN
@@
 $EndComp
 $Comp
-L GND #PWR020
+L GND #PWR022
 U 1 1 5999254B
 P 8120 1840
-F 0 "#PWR020" H 8120 1590 50  0001 C CNN
+F 0 "#PWR022" H 8120 1590 50  0001 C CNN
 F 1 "GND" H 8125 1667 50  0000 C CNN
 F 2 "" H 8120 1840 50  0001 C CNN
@@
 P 2950 7170
 F 0 "C7" H 3065 7216 50  0000 L CNN
-F 1 "C" H 3065 7125 50  0000 L CNN
+F 1 "10nF" H 3065 7125 50  0000 L CNN
 F 2 "Capacitors_THT:C_Disc_D3.4mm_W2.1mm_P2.50mm" H 2988 7020 50  0001 C CNN
 F 3 "" H 2950 7170 50  0001 C CNN
@@
 P 3250 7170
 F 0 "C8" H 3365 7216 50  0000 L CNN
-F 1 "C" H 3365 7125 50  0000 L CNN
+F 1 "10nF" H 3365 7125 50  0000 L CNN
 F 2 "Capacitors_THT:C_Disc_D3.4mm_W2.1mm_P2.50mm" H 3288 7020 50  0001 C CNN
 F 3 "" H 3250 7170 50  0001 C CNN
@@
 P 3560 7170
 F 0 "C9" H 3675 7216 50  0000 L CNN
-F 1 "C" H 3675 7125 50  0000 L CNN
+F 1 "10nF" H 3675 7125 50  0000 L CNN
 F 2 "Capacitors_THT:C_Disc_D3.4mm_W2.1mm_P2.50mm" H 3598 7020 50  0001 C CNN
 F 3 "" H 3560 7170 50  0001 C CNN
@@
 P 3880 7170
 F 0 "C10" H 3995 7216 50  0000 L CNN
-F 1 "C" H 3995 7125 50  0000 L CNN
+F 1 "10nF" H 3995 7125 50  0000 L CNN
 F 2 "Capacitors_THT:C_Disc_D3.4mm_W2.1mm_P2.50mm" H 3918 7020 50  0001 C CNN
 F 3 "" H 3880 7170 50  0001 C CNN
@@
 5v
 $Comp
-L GND #PWR021
+L GND #PWR023
 U 1 1 599998DA
 P 2820 7320
-F 0 "#PWR021" H 2820 7070 50  0001 C CNN
+F 0 "#PWR023" H 2820 7070 50  0001 C CNN
 F 1 "GND" H 2825 7147 50  0000 C CNN
 F 2 "" H 2820 7320 50  0001 C CNN
@@
 Text Notes 6970 7800 2    60   ~ 0
 DECOUPLING CAPS\n
+Wire Wire Line
+	2950 6990 2950 7020
+$Comp
+L VCC #PWR024
+U 1 1 59A69107
+P 2950 6990
+F 0 "#PWR024" H 2950 6840 50  0001 C CNN
+F 1 "VCC" H 2967 7163 50  0000 C CNN
+F 2 "" H 2950 6990 50  0001 C CNN
+F 3 "" H 2950 6990 50  0001 C CNN
+	1    2950 6990
+	1    0    0    -1
+$EndComp
 $EndSCHEMATC
