File: hardware/drivers/ND-03/column65_96.sch (KiCad schematic (older format))
At the start: 24 parts, among them J36 Screw_Terminal_1x02, J37 Screw_Terminal_1x02, J38 Screw_Terminal_1x02, J39 Screw_Terminal_1x02, J40 Screw_Terminal_1x02, J41 Screw_Terminal_1x02, J42 Screw_Terminal_1x02, J43 Screw_Terminal_1x02, J44 Screw_Terminal_1x02, J45 Screw_Terminal_1x02, J46 Screw_Terminal_1x02, J47 Screw_Terminal_1x02, J48 Screw_Terminal_1x02, J49 Screw_Terminal_1x02, J50 Screw_Terminal_1x02, J51 Screw_Terminal_1x02, U12 74HC595, U13 74HC595, U14 74HC595, U15 74HC595

Commit message: Multple commits enclosed in this commit.
1.Design passes all DRC tests.
2.Add PMOS reverse polarity protection on 5v direct input.
Parts:
- C11, C12, C13, C14: value C -> 10nF
Connections:
- net 5v is gone; now on net VCC: C11.1, C12.1, C13.1, C14.1, U12.10 (SRCLR), U13.10 (SRCLR), U14.10 (SRCLR), U15.10 (SRCLR)
Changed lines of the file:
@@
 5v
 $Comp
-L GND #PWR022
+L GND #PWR025
 U 1 1 599942BD
 P 1660 1810
-F 0 "#PWR022" H 1660 1560 50  0001 C CNN
+F 0 "#PWR025" H 1660 1560 50  0001 C CNN
 F 1 "GND" H 1665 1637 50  0000 C CNN
 F 2 "" H 1660 1810 50  0001 C CNN
@@
 $EndComp
 $Comp
-L GND #PWR023
+L GND #PWR026
 U 1 1 599942C3
 P 3710 1820
-F 0 "#PWR023" H 3710 1570 50  0001 C CNN
+F 0 "#PWR026" H 3710 1570 50  0001 C CNN
 F 1 "GND" H 3715 1647 50  0000 C CNN
 F 2 "" H 3710 1820 50  0001 C CNN
@@
 $EndComp
 $Comp
-L GND #PWR024
+L GND #PWR027
 U 1 1 599942C9
 P 5860 1850
-F 0 "#PWR024" H 5860 1600 50  0001 C CNN
+F 0 "#PWR027" H 5860 1600 50  0001 C CNN
 F 1 "GND" H 5865 1677 50  0000 C CNN
 F 2 "" H 5860 1850 50  0001 C CNN
@@
 $EndComp
 $Comp
-L GND #PWR025
+L GND #PWR028
 U 1 1 599942CF
 P 8120 1840
-F 0 "#PWR025" H 8120 1590 50  0001 C CNN
+F 0 "#PWR028" H 8120 1590 50  0001 C CNN
 F 1 "GND" H 8125 1667 50  0000 C CNN
 F 2 "" H 8120 1840 50  0001 C CNN
@@
 P 2950 7170
 F 0 "C11" H 3065 7216 50  0000 L CNN
-F 1 "C" H 3065 7125 50  0000 L CNN
+F 1 "10nF" H 3065 7125 50  0000 L CNN
 F 2 "Capacitors_THT:C_Disc_D3.4mm_W2.1mm_P2.50mm" H 2988 7020 50  0001 C CNN
 F 3 "" H 2950 7170 50  0001 C CNN
@@
 P 3250 7170
 F 0 "C12" H 3365 7216 50  0000 L CNN
-F 1 "C" H 3365 7125 50  0000 L CNN
+F 1 "10nF" H 3365 7125 50  0000 L CNN
 F 2 "Capacitors_THT:C_Disc_D3.4mm_W2.1mm_P2.50mm" H 3288 7020 50  0001 C CNN
 F 3 "" H 3250 7170 50  0001 C CNN
@@
 P 3560 7170
 F 0 "C13" H 3675 7216 50  0000 L CNN
-F 1 "C" H 3675 7125 50  0000 L CNN
+F 1 "10nF" H 3675 7125 50  0000 L CNN
 F 2 "Capacitors_THT:C_Disc_D3.4mm_W2.1mm_P2.50mm" H 3598 7020 50  0001 C CNN
 F 3 "" H 3560 7170 50  0001 C CNN
@@
 P 3880 7170
 F 0 "C14" H 3995 7216 50  0000 L CNN
-F 1 "C" H 3995 7125 50  0000 L CNN
+F 1 "10nF" H 3995 7125 50  0000 L CNN
 F 2 "Capacitors_THT:C_Disc_D3.4mm_W2.1mm_P2.50mm" H 3918 7020 50  0001 C CNN
 F 3 "" H 3880 7170 50  0001 C CNN
@@
 $EndComp
 Wire Wire Line
-	3880 7020 2830 7020
+	2830 7020 3880 7020
 Connection ~ 2950 7020
 Connection ~ 3250 7020
@@
 5v
 $Comp
-L GND #PWR026
+L GND #PWR029
 U 1 1 5999A733
 P 2820 7320
-F 0 "#PWR026" H 2820 7070 50  0001 C CNN
+F 0 "#PWR029" H 2820 7070 50  0001 C CNN
 F 1 "GND" H 2825 7147 50  0000 C CNN
 F 2 "" H 2820 7320 50  0001 C CNN
@@
 Text Notes 6970 7800 2    60   ~ 0
 DECOUPLING CAPS\n
+Wire Wire Line
+	2950 6980 2950 7020
+$Comp
+L VCC #PWR030
+U 1 1 59A68883
+P 2950 6980
+F 0 "#PWR030" H 2950 6830 50  0001 C CNN
+F 1 "VCC" H 2967 7153 50  0000 C CNN
+F 2 "" H 2950 6980 50  0001 C CNN
+F 3 "" H 2950 6980 50  0001 C CNN
+	1    2950 6980
+	1    0    0    -1
+$EndComp
 $EndSCHEMATC
