File: hardware/drivers/ND-03/row-driver.sch (KiCad schematic (older format))
At the start: 7 parts, among them J68 GS3, J69 Screw_Terminal_1x02, J70 Screw_Terminal_1x02, J71 Screw_Terminal_1x02, J72 Screw_Terminal_1x02, U20 ULN2803A, U21 CD4017

Commit message: Multple commits enclosed in this commit.
1.Design passes all DRC tests.
2.Add PMOS reverse polarity protection on 5v direct input.
Parts:
- added R2, R3, R4, R5, R6, R7, R8, R9: R, Resistors_THT:R_Axial_DIN0207_L6.3mm_D2.5mm_P7.62mm_Horizontal, symbol R
Connections:
- net R1: now also R2.2; no longer U20.18 (O1)
- net R2: now also R3.2; no longer U20.17 (O2)
- net R3: now also R4.2; no longer U20.16 (O3)
- net R4: now also R5.2; no longer U20.15 (O4)
- net R5: now also R6.2; no longer U20.14 (O5)
- net R6: now also R7.2; no longer U20.13 (O6)
- net R7: now also R8.2; no longer U20.12 (O7)
- net R8: now also R9.2; no longer U20.11 (O8)
- new net: R9.1, U20.11 (O8)
- new net: R8.1, U20.12 (O7)
- new net: R7.1, U20.13 (O6)
- new net: R6.1, U20.14 (O5)
- new net: R5.1, U20.15 (O4)
- new net: R4.1, U20.16 (O3)
- new net: R3.1, U20.17 (O2)
- new net: R2.1, U20.18 (O1)
Changed lines of the file:
@@
 $EndComp
 $Comp
-L GND #PWR032
+L GND #PWR037
 U 1 1 599A2812
 P 2910 1340
-F 0 "#PWR032" H 2910 1090 50  0001 C CNN
+F 0 "#PWR037" H 2910 1090 50  0001 C CNN
 F 1 "GND" H 2780 1250 50  0000 C CNN
 F 2 "" H 2910 1340 50  0001 C CNN
@@
 NoConn ~ 4640 2340
 $Comp
-L GND #PWR033
+L GND #PWR038
 U 1 1 599A3632
 P 6400 2280
-F 0 "#PWR033" H 6400 2030 50  0001 C CNN
+F 0 "#PWR038" H 6400 2030 50  0001 C CNN
 F 1 "GND" H 6405 2107 50  0000 C CNN
 F 2 "" H 6400 2280 50  0001 C CNN
@@
 Text Label 6000 1910 2    60   ~ 0
 JUMP
-Wire Notes Line
-	470  4590 11220 4590
-Wire Wire Line
-	3340 1240 3210 1240
-Wire Wire Line
-	2910 1340 3340 1340
-Wire Wire Line
-	3340 1540 3150 1540
-Wire Wire Line
-	4640 1240 4730 1240
-Wire Wire Line
-	4640 1340 4730 1340
-Wire Wire Line
-	4640 1440 4730 1440
-Wire Wire Line
-	4640 1540 4730 1540
-Wire Wire Line
-	4640 1640 4730 1640
-Wire Wire Line
-	4640 1740 4730 1740
-Wire Wire Line
-	4640 1840 4730 1840
-Wire Wire Line
-	4640 1940 4730 1940
-Wire Wire Line
-	4640 2040 4730 2040
-Wire Wire Line
-	6000 1210 5900 1210
-Wire Wire Line
-	6000 1310 5910 1310
-Wire Wire Line
-	6000 1410 5910 1410
-Wire Wire Line
-	6000 1510 5920 1510
-Wire Wire Line
-	6000 1610 5920 1610
-Wire Wire Line
-	6000 1710 5920 1710
-Wire Wire Line
-	6000 1810 5930 1810
-Wire Wire Line
-	5790 1910 6000 1910
-Wire Wire Line
-	5490 1810 5410 1810
-Wire Wire Line
-	5490 2010 5410 2010
-Wire Wire Line
-	6800 1210 6950 1210
-Wire Wire Line
-	6800 1310 6950 1310
-Wire Wire Line
-	6800 1410 6950 1410
-Wire Wire Line
-	6800 1510 6950 1510
-Wire Wire Line
-	6800 1610 6950 1610
-Wire Wire Line
-	6800 1710 6950 1710
-Wire Wire Line
-	6800 1810 6950 1810
-Wire Wire Line
-	6800 1910 6950 1910
-Wire Wire Line
-	6400 2280 6400 2210
-Wire Notes Line
-	11220 6530 470  6530
-Wire Wire Line
-	3060 5330 3060 5260
-Wire Wire Line
-	3260 5330 3260 5270
-Wire Wire Line
-	4310 5320 4310 5250
-Wire Wire Line
-	4510 5320 4510 5250
-Wire Wire Line
-	5520 5300 5520 5230
-Wire Wire Line
-	5720 5300 5720 5230
-Wire Wire Line
-	6760 5300 6760 5230
-Wire Wire Line
-	6960 5300 6960 5230
 Text Notes 11220 6530 2    60   ~ 0
 TERMINAL BLOCKS\n
@@
 Text Label 6960 5230 1    60   ~ 0
 R8
-Text Label 6950 1210 0    60   ~ 0
+Text Label 7310 1210 0    60   ~ 0
 R1
-Text Label 6950 1310 0    60   ~ 0
+Text Label 7310 1310 0    60   ~ 0
 R2
-Text Label 6950 1410 0    60   ~ 0
+Text Label 7310 1410 0    60   ~ 0
 R3
-Text Label 6950 1510 0    60   ~ 0
+Text Label 7310 1510 0    60   ~ 0
 R4
-Text Label 6950 1610 0    60   ~ 0
+Text Label 7310 1610 0    60   ~ 0
 R5
-Text Label 6950 1710 0    60   ~ 0
+Text Label 7310 1710 0    60   ~ 0
 R6
-Text Label 6950 1810 0    60   ~ 0
+Text Label 7310 1810 0    60   ~ 0
 R7
-Text Label 6950 1910 0    60   ~ 0
+Text Label 7310 1910 0    60   ~ 0
 R8
 NoConn ~ 6800 2010
-Wire Notes Line
-	475  2565 11220 2565
 $Comp
 L CD4017 U21
@@
 Text GLabel 3425 1035 0    60   Input ~ 0
 5v
-Wire Wire Line
-	3425 1035 3990 1035
-Wire Wire Line
-	3990 1035 3990 1190
-$Comp
-L GND #PWR034
+$Comp
+L GND #PWR039
 U 1 1 599C2C7A
 P 3990 2425
-F 0 "#PWR034" H 3990 2175 50  0001 C CNN
+F 0 "#PWR039" H 3990 2175 50  0001 C CNN
 F 1 "GND" H 4120 2335 50  0000 C CNN
 F 2 "" H 3990 2425 50  0001 C CNN
@@
 	1    0    0    -1
 $EndComp
+$Comp
+L R R2
+U 1 1 59A532E8
+P 7100 1210
+F 0 "R2" V 7140 1360 50  0000 C CNN
+F 1 "R" V 7100 1210 50  0000 C CNN
+F 2 "Resistors_THT:R_Axial_DIN0207_L6.3mm_D2.5mm_P7.62mm_Horizontal" V 7030 1210 50  0001 C CNN
+F 3 "" H 7100 1210 50  0001 C CNN
+	1    7100 1210
+	0    -1   -1   0
+$EndComp
+Wire Notes Line
+	470  4590 11220 4590
+Wire Wire Line
+	3340 1240 3210 1240
+Wire Wire Line
+	2910 1340 3340 1340
+Wire Wire Line
+	3340 1540 3150 1540
+Wire Wire Line
+	4640 1240 4730 1240
+Wire Wire Line
+	4640 1340 4730 1340
+Wire Wire Line
+	4640 1440 4730 1440
+Wire Wire Line
+	4640 1540 4730 1540
+Wire Wire Line
+	4640 1640 4730 1640
+Wire Wire Line
+	4640 1740 4730 1740
+Wire Wire Line
+	4640 1840 4730 1840
+Wire Wire Line
+	4640 1940 4730 1940
+Wire Wire Line
+	4640 2040 4730 2040
+Wire Wire Line
+	6000 1210 5900 1210
+Wire Wire Line
+	6000 1310 5910 1310
+Wire Wire Line
+	6000 1410 5910 1410
+Wire Wire Line
+	6000 1510 5920 1510
+Wire Wire Line
+	6000 1610 5920 1610
+Wire Wire Line
+	6000 1710 5920 1710
+Wire Wire Line
+	6000 1810 5930 1810
+Wire Wire Line
+	5790 1910 6000 1910
+Wire Wire Line
+	5490 1810 5410 1810
+Wire Wire Line
+	5490 2010 5410 2010
+Wire Wire Line
+	6800 1210 6950 1210
+Wire Wire Line
+	6800 1310 6950 1310
+Wire Wire Line
+	6800 1410 6950 1410
+Wire Wire Line
+	6800 1510 6950 1510
+Wire Wire Line
+	6800 1610 6950 1610
+Wire Wire Line
+	6800 1710 6950 1710
+Wire Wire Line
+	6800 1810 6950 1810
+Wire Wire Line
+	6800 1910 6950 1910
+Wire Wire Line
+	6400 2280 6400 2210
+Wire Notes Line
+	11220 6530 470  6530
+Wire Wire Line
+	3060 5330 3060 5260
+Wire Wire Line
+	3260 5330 3260 5270
+Wire Wire Line
+	4310 5320 4310 5250
+Wire Wire Line
+	4510 5320 4510 5250
+Wire Wire Line
+	5520 5300 5520 5230
+Wire Wire Line
+	5720 5300 5720 5230
+Wire Wire Line
+	6760 5300 6760 5230
+Wire Wire Line
+	6960 5300 6960 5230
+Wire Notes Line
+	475  2565 11220 2565
+Wire Wire Line
+	3425 1035 3990 1035
+Wire Wire Line
+	3990 1035 3990 1190
 Wire Wire Line
 	3990 2425 3990 2390
+$Comp
+L R R3
+U 1 1 59A53F67
+P 7100 1310
+F 0 "R3" V 7140 1460 50  0000 C CNN
+F 1 "R" V 7100 1310 50  0000 C CNN
+F 2 "Resistors_THT:R_Axial_DIN0207_L6.3mm_D2.5mm_P7.62mm_Horizontal" V 7030 1310 50  0001 C CNN
+F 3 "" H 7100 1310 50  0001 C CNN
+	1    7100 1310
+	0    -1   -1   0
+$EndComp
+$Comp
+L R R4
+U 1 1 59A53FF7
+P 7100 1410
+F 0 "R4" V 7140 1560 50  0000 C CNN
+F 1 "R" V 7100 1410 50  0000 C CNN
+F 2 "Resistors_THT:R_Axial_DIN0207_L6.3mm_D2.5mm_P7.62mm_Horizontal" V 7030 1410 50  0001 C CNN
+F 3 "" H 7100 1410 50  0001 C CNN
+	1    7100 1410
+	0    -1   -1   0
+$EndComp
+$Comp
+L R R5
+U 1 1 59A54063
+P 7100 1510
+F 0 "R5" V 7140 1660 50  0000 C CNN
+F 1 "R" V 7100 1510 50  0000 C CNN
+F 2 "Resistors_THT:R_Axial_DIN0207_L6.3mm_D2.5mm_P7.62mm_Horizontal" V 7030 1510 50  0001 C CNN
+F 3 "" H 7100 1510 50  0001 C CNN
+	1    7100 1510
+	0    -1   -1   0
+$EndComp
+$Comp
+L R R6
+U 1 1 59A5411A
+P 7100 1610
+F 0 "R6" V 7140 1760 50  0000 C CNN
+F 1 "R" V 7100 1610 50  0000 C CNN
+F 2 "Resistors_THT:R_Axial_DIN0207_L6.3mm_D2.5mm_P7.62mm_Horizontal" V 7030 1610 50  0001 C CNN
+F 3 "" H 7100 1610 50  0001 C CNN
+	1    7100 1610
+	0    -1   -1   0
+$EndComp
+$Comp
+L R R7
+U 1 1 59A54156
+P 7100 1710
+F 0 "R7" V 7140 1860 50  0000 C CNN
+F 1 "R" V 7100 1710 50  0000 C CNN
+F 2 "Resistors_THT:R_Axial_DIN0207_L6.3mm_D2.5mm_P7.62mm_Horizontal" V 7030 1710 50  0001 C CNN
+F 3 "" H 7100 1710 50  0001 C CNN
+	1    7100 1710
+	0    -1   -1   0
+$EndComp
+$Comp
+L R R8
+U 1 1 59A54223
+P 7100 1810
+F 0 "R8" V 7140 1960 50  0000 C CNN
+F 1 "R" V 7100 1810 50  0000 C CNN
+F 2 "Resistors_THT:R_Axial_DIN0207_L6.3mm_D2.5mm_P7.62mm_Horizontal" V 7030 1810 50  0001 C CNN
+F 3 "" H 7100 1810 50  0001 C CNN
+	1    7100 1810
+	0    -1   -1   0
+$EndComp
+$Comp
+L R R9
+U 1 1 59A54263
+P 7100 1910
+F 0 "R9" V 7140 2060 50  0000 C CNN
+F 1 "R" V 7100 1910 50  0000 C CNN
+F 2 "Resistors_THT:R_Axial_DIN0207_L6.3mm_D2.5mm_P7.62mm_Horizontal" V 7030 1910 50  0001 C CNN
+F 3 "" H 7100 1910 50  0001 C CNN
+	1    7100 1910
+	0    -1   -1   0
+$EndComp
+Wire Wire Line
+	7250 1210 7310 1210
+Wire Wire Line
+	7250 1310 7310 1310
+Wire Wire Line
+	7250 1410 7310 1410
+Wire Wire Line
+	7250 1510 7310 1510
+Wire Wire Line
+	7250 1610 7310 1610
+Wire Wire Line
+	7250 1710 7310 1710
+Wire Wire Line
+	7250 1810 7310 1810
+Wire Wire Line
+	7250 1910 7310 1910
 $EndSCHEMATC
