File: hardware/drivers/ND-01/ND01 MCU INTERFACE.sch (KiCad schematic (older format))
At the start: 1 part, among them J3 CONN_01X08

Commit message: Prepare release version
Parts:
- J3: symbol CONN_01X08 -> CONN_01X08-RESCUE-ND-01
Changed lines of the file:
@@
-EESchema Schematic File Version 2
-LIBS:power
-LIBS:device
-LIBS:transistors
-LIBS:conn
-LIBS:linear
-LIBS:regul
-LIBS:74xx
-LIBS:cmos4000
-LIBS:adc-dac
-LIBS:memory
-LIBS:xilinx
-LIBS:microcontrollers
-LIBS:dsp
-LIBS:microchip
-LIBS:analog_switches
-LIBS:motorola
-LIBS:texas
-LIBS:intel
-LIBS:audio
-LIBS:interface
-LIBS:digital-audio
-LIBS:philips
-LIBS:display
-LIBS:cypress
-LIBS:siliconi
-LIBS:opto
-LIBS:atmel
-LIBS:contrib
-LIBS:valves
-LIBS:pochi
-LIBS:narra
+EESchema Schematic File Version 4
 LIBS:ND-01-cache
 EELAYER 26 0
@@
 COL-RCK
 $Comp
-L CONN_01X08 J3
+L CONN_01X08-RESCUE-ND-01 J3
 U 1 1 58E79D53
 P 5350 1350
@@
 	5700 1500 5550 1500
 $Comp
-L GND #PWR07
+L GND-RESCUE-ND-01 #PWR07
 U 1 1 58E79E5E
 P 5700 1800
