File: hardware/drivers/ND-01/ND01 control.sch (KiCad schematic (older format))
At the start: 36 parts, among them J33 GS2, J34 GS2, J35 GS2, J36 GS2, J37 GS2, J38 GS2, J39 GS2, J40 GS3, U1 ULN2803A, U10 74HC595, U11 74HC595, U12 74HC595, U13 74HC595, U14 74HC595, U2 4017, U3 74HC595, U4 74HC595, U5 74HC595, U6 74HC595, U7 74HC595, U8 74HC595, U9 74HC595

Commit message: Prepare release version
Parts:
- C10, C11, C12, C13, C14, C15, C16, C17, C4, C5, C6, C7, C8, C9: symbol C -> C-RESCUE-ND-01
- J33, J34, J35, J36, J37, J38, J39: symbol GS2 -> GS2-RESCUE-ND-01
- J40: symbol GS3 -> GS3-RESCUE-ND-01
- U1: symbol ULN2803A -> ULN2803A-RESCUE-ND-01
- U10, U11, U12, U13, U14, U3, U4, U5, U6, U7, U8, U9: symbol 74HC595 -> 74HC595-RESCUE-ND-01
- U2: symbol 4017 -> 4017-RESCUE-ND-01
Changed lines of the file:
@@
-EESchema Schematic File Version 2
-LIBS:power
-LIBS:device
-LIBS:transistors
-LIBS:conn
-LIBS:linear
-LIBS:regul
-LIBS:74xx
-LIBS:cmos4000
-LIBS:adc-dac
-LIBS:memory
-LIBS:xilinx
-LIBS:microcontrollers
-LIBS:dsp
-LIBS:microchip
-LIBS:analog_switches
-LIBS:motorola
-LIBS:texas
-LIBS:intel
-LIBS:audio
-LIBS:interface
-LIBS:digital-audio
-LIBS:philips
-LIBS:display
-LIBS:cypress
-LIBS:siliconi
-LIBS:opto
-LIBS:atmel
-LIBS:contrib
-LIBS:valves
-LIBS:pochi
-LIBS:narra
+EESchema Schematic File Version 4
 LIBS:ND-01-cache
 EELAYER 26 0
@@
 $EndDescr
 $Comp
-L 4017 U2
+L 4017-RESCUE-ND-01 U2
 U 1 1 58E5FFE3
 P 4800 1350
@@
 $EndComp
 $Comp
-L ULN2803A U1
+L ULN2803A-RESCUE-ND-01 U1
 U 1 1 58E60148
 P 8150 1200
@@
 VCC
 $Comp
-L GND #PWR08
+L GND-RESCUE-ND-01 #PWR08
 U 1 1 58E61237
 P 1150 3300
@@
 $EndComp
 $Comp
-L GND #PWR09
+L GND-RESCUE-ND-01 #PWR09
 U 1 1 58E61370
 P 3750 900
@@
 SRCLK
 $Comp
-L 74HC595 U4
+L 74HC595-RESCUE-ND-01 U4
 U 1 1 58E62971
 P 4650 3000
@@
 VCC
 $Comp
-L GND #PWR010
+L GND-RESCUE-ND-01 #PWR010
 U 1 1 58E62979
 P 3750 3250
@@
 C15
 $Comp
-L 74HC595 U5
+L 74HC595-RESCUE-ND-01 U5
 U 1 1 58E62FF1
 P 7000 3000
@@
 VCC
 $Comp
-L GND #PWR011
+L GND-RESCUE-ND-01 #PWR011
 U 1 1 58E62FF9
 P 6100 3250
@@
 LINK-2
 $Comp
-L 74HC595 U3
+L 74HC595-RESCUE-ND-01 U3
 U 1 1 58E634B7
 P 9300 2950
@@
 C[24..31]
 $Comp
-L 74HC595 U7
+L 74HC595-RESCUE-ND-01 U7
 U 1 1 58E636AC
 P 2050 4400
@@
 C[32..39]
 $Comp
-L 74HC595 U8
+L 74HC595-RESCUE-ND-01 U8
 U 1 1 58E63760
 P 4650 4400
@@
 C[40..47]
 $Comp
-L 74HC595 U9
+L 74HC595-RESCUE-ND-01 U9
 U 1 1 58E638B8
 P 7000 4400
@@
 C[48..55]
 $Comp
-L 74HC595 U10
+L 74HC595-RESCUE-ND-01 U10
 U 1 1 58E63956
 P 9300 4400
@@
 C[56..63]
 $Comp
-L 74HC595 U6
+L 74HC595-RESCUE-ND-01 U6
 U 1 1 58E6101F
 P 2050 3050
@@
 $EndComp
 $Comp
-L 74HC595 U11
+L 74HC595-RESCUE-ND-01 U11
 U 1 1 58E647FF
 P 2100 5700
@@
 C[64..71]
 $Comp
-L 74HC595 U12
+L 74HC595-RESCUE-ND-01 U12
 U 1 1 58E64821
 P 4700 5700
@@
 C[72..79]
 $Comp
-L 74HC595 U13
+L 74HC595-RESCUE-ND-01 U13
 U 1 1 58E64843
 P 7050 5700
@@
 C[80..87]
 $Comp
-L 74HC595 U14
+L 74HC595-RESCUE-ND-01 U14
 U 1 1 58E64865
 P 9350 5700
@@
 LINK-3
 $Comp
-L GND #PWR012
+L GND-RESCUE-ND-01 #PWR012
 U 1 1 58E6734E
 P 8500 3200
@@
 LINK-4
 $Comp
-L GND #PWR013
+L GND-RESCUE-ND-01 #PWR013
 U 1 1 58E6AAB3
 P 6100 4600
@@
 $EndComp
 $Comp
-L GND #PWR014
+L GND-RESCUE-ND-01 #PWR014
 U 1 1 58E6ABE4
 P 3750 4600
@@
 $EndComp
 $Comp
-L GND #PWR015
+L GND-RESCUE-ND-01 #PWR015
 U 1 1 58E6AC51
 P 1200 4600
@@
 $EndComp
 $Comp
-L GND #PWR016
+L GND-RESCUE-ND-01 #PWR016
 U 1 1 58E6ADD6
 P 8450 4600
@@
 $EndComp
 $Comp
-L GND #PWR017
+L GND-RESCUE-ND-01 #PWR017
 U 1 1 58E6B505
 P 1200 5900
@@
 $EndComp
 $Comp
-L GND #PWR018
+L GND-RESCUE-ND-01 #PWR018
 U 1 1 58E6B75E
 P 3750 5900
@@
 $EndComp
 $Comp
-L GND #PWR019
+L GND-RESCUE-ND-01 #PWR019
 U 1 1 58E6BB5E
 P 6100 5900
@@
 $EndComp
 $Comp
-L GND #PWR020
+L GND-RESCUE-ND-01 #PWR020
 U 1 1 58E6BE20
 P 8350 5900
@@
 	6950 6550 450  6550
 $Comp
-L GNDA #PWR021
+L GNDA-RESCUE-ND-01 #PWR021
 U 1 1 58F1E870
 P 8150 1900
@@
 	800  7350 5600 7350
 $Comp
-L PWR_FLAG #FLG022
+L PWR_FLAG-RESCUE-ND-01 #FLG022
 U 1 1 58F1F6A8
 P 5600 6950
@@
 $EndComp
 $Comp
-L PWR_FLAG #FLG023
+L PWR_FLAG-RESCUE-ND-01 #FLG023
 U 1 1 58F1F70F
 P 5600 7350
@@
 $EndComp
 $Comp
-L C C4
+L C-RESCUE-ND-01 C4
 U 1 1 58F2029E
 P 1050 7150
@@
 Connection ~ 1050 7350
 $Comp
-L C C5
+L C-RESCUE-ND-01 C5
 U 1 1 58F20590
 P 1300 7150
@@
 Connection ~ 1300 7350
 $Comp
-L C C6
+L C-RESCUE-ND-01 C6
 U 1 1 58F2081C
 P 1550 7150
@@
 Connection ~ 1550 7350
 $Comp
-L C C7
+L C-RESCUE-ND-01 C7
 U 1 1 58F20CD0
 P 1850 7150
@@
 $EndComp
 $Comp
-L C C8
+L C-RESCUE-ND-01 C8
 U 1 1 58F20D34
 P 2150 7150
@@
 $EndComp
 $Comp
-L C C9
+L C-RESCUE-ND-01 C9
 U 1 1 58F20F28
 P 2450 7150
@@
 $EndComp
 $Comp
-L C C10
+L C-RESCUE-ND-01 C10
 U 1 1 58F20F7E
 P 2750 7150
@@
 $EndComp
 $Comp
-L C C11
+L C-RESCUE-ND-01 C11
 U 1 1 58F2100A
 P 3000 7150
@@
 $EndComp
 $Comp
-L C C12
+L C-RESCUE-ND-01 C12
 U 1 1 58F21B92
 P 3300 7150
@@
 $EndComp
 $Comp
-L C C13
+L C-RESCUE-ND-01 C13
 U 1 1 58F21C18
 P 3600 7150
@@
 $EndComp
 $Comp
-L C C14
+L C-RESCUE-ND-01 C14
 U 1 1 58F21D29
 P 3900 7150
@@
 $EndComp
 $Comp
-L C C15
+L C-RESCUE-ND-01 C15
 U 1 1 58F21F49
 P 4200 7150
@@
 Connection ~ 3900 7350
 $Comp
-L C C16
+L C-RESCUE-ND-01 C16
 U 1 1 58F24B28
 P 4550 7150
@@
 Connection ~ 4550 7350
 $Comp
-L C C17
+L C-RESCUE-ND-01 C17
 U 1 1 58F263E2
 P 4900 7150
@@
 DECOUPLING CAPACITORS
 $Comp
-L VDD #PWR024
+L VDD-RESCUE-ND-01 #PWR024
 U 1 1 58F2925C
 P 1050 6900
@@
 	5500 2550 5350 2550
 $Comp
-L GND #PWR025
+L GND-RESCUE-ND-01 #PWR025
 U 1 1 58F48E4F
 P 800 7375
@@
 C[0..7]
 $Comp
-L GS2 J33
+L GS2-RESCUE-ND-01 J33
 U 1 1 58F7661F
 P 7150 900
@@
 $EndComp
 $Comp
-L GS2 J35
+L GS2-RESCUE-ND-01 J35
 U 1 1 58F76BD5
 P 7150 1100
@@
 $EndComp
 $Comp
-L GS2 J34
+L GS2-RESCUE-ND-01 J34
 U 1 1 58F76CF1
 P 7150 1000
@@
 $EndComp
 $Comp
-L GS2 J36
+L GS2-RESCUE-ND-01 J36
 U 1 1 58F76D3F
 P 7150 1200
@@
 $EndComp
 $Comp
-L GS2 J37
+L GS2-RESCUE-ND-01 J37
 U 1 1 58F76D8F
 P 7150 1300
@@
 $EndComp
 $Comp
-L GS2 J38
+L GS2-RESCUE-ND-01 J38
 U 1 1 58F76DE1
 P 7150 1400
@@
 $EndComp
 $Comp
-L GS2 J39
+L GS2-RESCUE-ND-01 J39
 U 1 1 58F76E35
 P 7150 1500
@@
 $EndComp
 $Comp
-L GS3 J40
+L GS3-RESCUE-ND-01 J40
 U 1 1 58F78FCA
 P 7200 1750
