File: hardware/drivers/ND-01/ND01 output.sch (KiCad schematic (older format))
At the start: 30 parts, among them J10 CONN_01X08, J11 CONN_01X08, J12 CONN_01X08, J13 CONN_01X08, J14 CONN_01X08, J15 CONN_01X08, J16 CONN_01X08, J17 GS2, J18 GS2, J19 GS2, J20 GS2, J21 GS2, J22 GS2, J23 GS2, J24 GS2, J25 GS2, J26 GS2, J27 GS2, J28 GS2, J29 GS2, J30 GS2, J31 GS2, J32 GS2, J4 CONN_01X08, J5 CONN_01X08, J6 CONN_01X08, J7 CONN_01X08, J8 CONN_01X08, J9 CONN_01X08, M1 MATRIX

Commit message: Prepare release version
Parts:
- J10, J11, J12, J13, J14, J15, J16, J4, J5, J6, J7, J8, J9: symbol CONN_01X08 -> CONN_01X08-RESCUE-ND-01
- J17, J18, J19, J20, J21, J22, J23, J24, J25, J26, J27, J28, J29, J30, J31, J32: symbol GS2 -> GS2-RESCUE-ND-01
- M1: symbol MATRIX -> MATRIX-RESCUE-ND-01
Changed lines of the file:
@@
-EESchema Schematic File Version 2
-LIBS:power
-LIBS:device
-LIBS:transistors
-LIBS:conn
-LIBS:linear
-LIBS:regul
-LIBS:74xx
-LIBS:cmos4000
-LIBS:adc-dac
-LIBS:memory
-LIBS:xilinx
-LIBS:microcontrollers
-LIBS:dsp
-LIBS:microchip
-LIBS:analog_switches
-LIBS:motorola
-LIBS:texas
-LIBS:intel
-LIBS:audio
-LIBS:interface
-LIBS:digital-audio
-LIBS:philips
-LIBS:display
-LIBS:cypress
-LIBS:siliconi
-LIBS:opto
-LIBS:atmel
-LIBS:contrib
-LIBS:valves
-LIBS:pochi
-LIBS:narra
+EESchema Schematic File Version 4
 LIBS:ND-01-cache
 EELAYER 26 0
@@
 $EndDescr
 $Comp
-L CONN_01X08 J4
+L CONN_01X08-RESCUE-ND-01 J4
 U 1 1 58E76DCC
 P 6300 1075
@@
 C[88..95]
 $Comp
-L CONN_01X08 J5
+L CONN_01X08-RESCUE-ND-01 J5
 U 1 1 58E7B392
 P 1900 2400
@@
 	1500 2650 1600 2750
 $Comp
-L CONN_01X08 J6
+L CONN_01X08-RESCUE-ND-01 J6
 U 1 1 58E7B6D4
 P 3600 2400
@@
 	3200 2650 3300 2750
 $Comp
-L CONN_01X08 J7
+L CONN_01X08-RESCUE-ND-01 J7
 U 1 1 58E7B765
 P 5300 2400
@@
 	4900 2650 5000 2750
 $Comp
-L CONN_01X08 J8
+L CONN_01X08-RESCUE-ND-01 J8
 U 1 1 58E7B832
 P 6900 2400
@@
 	6500 2650 6600 2750
 $Comp
-L CONN_01X08 J9
+L CONN_01X08-RESCUE-ND-01 J9
 U 1 1 58E7B935
 P 8450 2400
@@
 	8050 2650 8150 2750
 $Comp
-L CONN_01X08 J10
+L CONN_01X08-RESCUE-ND-01 J10
 U 1 1 58E7BBF0
 P 10000 2400
@@
 	9600 2650 9700 2750
 $Comp
-L CONN_01X08 J11
+L CONN_01X08-RESCUE-ND-01 J11
 U 1 1 58E7C2E0
 P 1900 3400
@@
 	1500 3650 1600 3750
 $Comp
-L CONN_01X08 J12
+L CONN_01X08-RESCUE-ND-01 J12
 U 1 1 58E7C2F8
 P 3600 3400
@@
 	3200 3650 3300 3750
 $Comp
-L CONN_01X08 J13
+L CONN_01X08-RESCUE-ND-01 J13
 U 1 1 58E7C310
 P 5300 3400
@@
 	4900 3650 5000 3750
 $Comp
-L CONN_01X08 J14
+L CONN_01X08-RESCUE-ND-01 J14
 U 1 1 58E7C328
 P 6900 3400
@@
 	6500 3650 6600 3750
 $Comp
-L CONN_01X08 J15
+L CONN_01X08-RESCUE-ND-01 J15
 U 1 1 58E7C340
 P 8450 3400
@@
 	8050 3650 8150 3750
 $Comp
-L CONN_01X08 J16
+L CONN_01X08-RESCUE-ND-01 J16
 U 1 1 58E7C358
 P 10000 3400
@@
 $EndBitmap
 $Comp
-L MATRIX M1
+L MATRIX-RESCUE-ND-01 M1
 U 1 1 58ED21AF
 P 2950 6050
@@
 C[0..7]
 $Comp
-L GS2 J18
+L GS2-RESCUE-ND-01 J18
 U 1 1 58F71A14
 P 5200 4200
@@
 $EndComp
 $Comp
-L GS2 J20
+L GS2-RESCUE-ND-01 J20
 U 1 1 58F71FF4
 P 5200 4300
@@
 $EndComp
 $Comp
-L GS2 J22
+L GS2-RESCUE-ND-01 J22
 U 1 1 58F72028
 P 5200 4400
@@
 $EndComp
 $Comp
-L GS2 J24
+L GS2-RESCUE-ND-01 J24
 U 1 1 58F720D1
 P 5200 4500
@@
 $EndComp
 $Comp
-L GS2 J26
+L GS2-RESCUE-ND-01 J26
 U 1 1 58F72105
 P 5200 4600
@@
 $EndComp
 $Comp
-L GS2 J28
+L GS2-RESCUE-ND-01 J28
 U 1 1 58F7213B
 P 5200 4700
@@
 $EndComp
 $Comp
-L GS2 J30
+L GS2-RESCUE-ND-01 J30
 U 1 1 58F72173
 P 5200 4800
@@
 $EndComp
 $Comp
-L GS2 J32
+L GS2-RESCUE-ND-01 J32
 U 1 1 58F721AD
 P 5200 4900
@@
 $EndComp
 $Comp
-L GS2 J17
+L GS2-RESCUE-ND-01 J17
 U 1 1 58F722DF
 P 9055 4150
@@
 $EndComp
 $Comp
-L GS2 J19
+L GS2-RESCUE-ND-01 J19
 U 1 1 58F72759
 P 9050 4250
@@
 $EndComp
 $Comp
-L GS2 J21
+L GS2-RESCUE-ND-01 J21
 U 1 1 58F72799
 P 9050 4350
@@
 $EndComp
 $Comp
-L GS2 J23
+L GS2-RESCUE-ND-01 J23
 U 1 1 58F727E3
 P 9050 4450
@@
 $EndComp
 $Comp
-L GS2 J25
+L GS2-RESCUE-ND-01 J25
 U 1 1 58F72945
 P 9050 4550
@@
 $EndComp
 $Comp
-L GS2 J27
+L GS2-RESCUE-ND-01 J27
 U 1 1 58F7298B
 P 9050 4650
@@
 $EndComp
 $Comp
-L GS2 J29
+L GS2-RESCUE-ND-01 J29
 U 1 1 58F729D3
 P 9050 4750
@@
 $EndComp
 $Comp
-L GS2 J31
+L GS2-RESCUE-ND-01 J31
 U 1 1 58F72A1D
 P 9050 4850
