File: hardware/drivers/ND-01/ND01 power.sch (KiCad schematic (older format))
At the start: 9 parts, among them J1 CONN_01X02, J2 HIROSE-USB-MICROB, J41 GS3

Commit message: Prepare release version
Parts:
- C1, C2, C3: symbol CP1 -> CP1-RESCUE-ND-01
- D1: symbol D_Zener -> D_Zener-RESCUE-ND-01
- D2: symbol LED -> LED-RESCUE-ND-01
- J1: symbol CONN_01X02 -> CONN_01X02-RESCUE-ND-01
- J2: symbol HIROSE-USB-MICROB -> HIROSE-USB-MICROB-RESCUE-ND-01
- J41: symbol GS3 -> GS3-RESCUE-ND-01
- R1: symbol R -> R-RESCUE-ND-01
Changed lines of the file:
@@
-EESchema Schematic File Version 2
-LIBS:power
-LIBS:device
-LIBS:transistors
-LIBS:conn
-LIBS:linear
-LIBS:regul
-LIBS:74xx
-LIBS:cmos4000
-LIBS:adc-dac
-LIBS:memory
-LIBS:xilinx
-LIBS:microcontrollers
-LIBS:dsp
-LIBS:microchip
-LIBS:analog_switches
-LIBS:motorola
-LIBS:texas
-LIBS:intel
-LIBS:audio
-LIBS:interface
-LIBS:digital-audio
-LIBS:philips
-LIBS:display
-LIBS:cypress
-LIBS:siliconi
-LIBS:opto
-LIBS:atmel
-LIBS:contrib
-LIBS:valves
-LIBS:pochi
-LIBS:narra
+EESchema Schematic File Version 4
 LIBS:ND-01-cache
 EELAYER 26 0
@@
 $EndDescr
 $Comp
-L HIROSE-USB-MICROB J2
+L HIROSE-USB-MICROB-RESCUE-ND-01 J2
 U 1 1 58E5E79F
 P 1450 2700
@@
 $EndComp
 $Comp
-L GND #PWR01
+L GND-RESCUE-ND-01 #PWR01
 U 1 1 58E5EAD0
 P 1900 3300
@@
 GND
 $Comp
-L CONN_01X02 J1
+L CONN_01X02-RESCUE-ND-01 J1
 U 1 1 58E5ED61
 P 1400 1350
@@
 5V
 $Comp
-L D_Zener D1
+L D_Zener-RESCUE-ND-01 D1
 U 1 1 58E5F2D5
 P 7950 1900
@@
 $EndComp
 $Comp
-L CP1 C3
+L CP1-RESCUE-ND-01 C3
 U 1 1 58E5F3F0
 P 9150 1900
@@
 $EndComp
 $Comp
-L GND #PWR02
+L GND-RESCUE-ND-01 #PWR02
 U 1 1 58E5F47E
 P 9150 2350
@@
 $EndComp
 $Comp
-L R R1
+L R-RESCUE-ND-01 R1
 U 1 1 58E5F57B
 P 9600 1800
@@
 $EndComp
 $Comp
-L LED D2
+L LED-RESCUE-ND-01 D2
 U 1 1 58E5F5EF
 P 9600 2100
@@
 $EndComp
 $Comp
-L GND #PWR03
+L GND-RESCUE-ND-01 #PWR03
 U 1 1 58E5F794
 P 9600 2350
@@
 $EndComp
 $Comp
-L GND #PWR04
+L GND-RESCUE-ND-01 #PWR04
 U 1 1 58E5F7E1
 P 7950 2350
@@
 $EndBitmap
 $Comp
-L CP1 C2
+L CP1-RESCUE-ND-01 C2
 U 1 1 58F30929
 P 8750 1900
@@
 $EndComp
 $Comp
-L GND #PWR05
+L GND-RESCUE-ND-01 #PWR05
 U 1 1 58F3092F
 P 8750 2350
@@
 $EndComp
 $Comp
-L CP1 C1
+L CP1-RESCUE-ND-01 C1
 U 1 1 58F30A1C
 P 8350 1900
@@
 $EndComp
 $Comp
-L GND #PWR06
+L GND-RESCUE-ND-01 #PWR06
 U 1 1 58F30A22
 P 8350 2350
@@
 POWER SELECTOR
 $Comp
-L GS3 J41
+L GS3-RESCUE-ND-01 J41
 U 1 1 58FBB40E
 P 4300 1850
